Commit message: cleanup of human hand urdf

File: robot/human_hand_simple.urdf.xacro (robot description, xacro)
@@ -3,8 +3,4 @@
 	<xacro:include filename="$(find pisa_hand_description)/model/human_hand.urdf.xacro"/>
 	<link name="box">
-		<!-- <inertial>
-			<mass value="50.0"/>
-			<inertia  ixx="1" ixy="0.00"  ixz="0.00" iyy="1" iyz="0.00" izz="1" />
-		</inertial> -->
 		<visual>
 			<origin xyz="0 0 0.50" rpy="0 0 0"/>
@@ -13,38 +9,5 @@
 			</geometry>
 		</visual>
-		<!-- <collision>
-			<origin xyz="0 0 0.50" rpy="0 0 0"/>
-			<geometry>
-				<box size="1.0 1.0 1.0"/>
-			</geometry>
-		</collision> -->
 	</link>
-<!--
-	<joint name="box_wrist_left_joint" type="fixed">
-		<origin xyz="0 -0.2 1.02" rpy="0 0 0" />
-		<parent link="box"/>
-		<child link="wrist_left"/>
-	</joint>
-	<link name="wrist_left">
-		<inertial>
-			<mass value="1.0"/>
-			<inertia  ixx="0.01" ixy="0.00"  ixz="0.00" iyy="0.01" iyz="0.00" izz="0.01" />
-		</inertial>
-		<visual>
-			<geometry>
-				<mesh filename="package://pisa_hand_description/meshes/coman_coupler_left.stl" scale=" .001 .001 .001" />
-			</geometry>
-			<material name="SoftHand/LightBlue" />
-		</visual>
-		<collision>
-			<geometry>
-				<mesh filename="package://pisa_hand_description/meshes/coman_coupler_left.stl" scale=" .001 .001 .001" />
-			</geometry>
-		</collision>
-	</link>
-	<xacro:pisa_hand parent="wrist_left" name="pisa_hand_left" withAdaptiveTransmission="true" useMimicTag="$(arg use_mimic_tag)" left="true">
-		<origin xyz="0.002 -0.009 0.038" rpy="0 0 0"/>
-	</xacro:pisa_hand>
--->
 	<joint name="box_wrist_right_joint_1" type="revolute">
 		<origin xyz="0 0.2 1.02" rpy="0 0 0" />
@@ -76,19 +39,4 @@
 	</joint>
 	<link name="wrist_right">
-		<!-- <inertial>
-			<mass value="1.0"/>
-			<inertia  ixx="0.01" ixy="0.00"  ixz="0.00" iyy="0.01" iyz="0.00" izz="0.01" />
-		</inertial>
-		<visual>
-			<geometry>
-				<mesh filename="package://pisa_hand_description/meshes/coman_coupler_right.stl" scale=" .001 .001 .001"/>
-			</geometry>
-			<material name="SoftHand/LightBlue" />
-		</visual>
-		<collision>
-			<geometry>
-				<mesh filename="package://pisa_hand_description/meshes/coman_coupler_right.stl" scale=" .001 .001 .001" />
-			</geometry>
-		</collision> -->
 	</link>
 	<xacro:human_hand parent="wrist_right" name="pisa_hand_right" left="false">
