Commit message: Added a human hand model (from grabCAD) and created stl files and urdf out of it

File: model/materials.urdf.xacro (robot description, xacro)
@@ -25,3 +25,6 @@
 		<color rgba="0.0 0.0 0.0 1.0"/>
 	</material>
+  <material name="HumanHand/Skin">
+		<color rgba="0.802 0.732 0.673 1.0"/>
+	</material>
 </robot>

Commit message: removed wrist joints, renamed my_rviz.rviz -> display.rviz

File: model/materials.urdf.xacro (robot description, xacro)
@@ -1,5 +1,5 @@
 <?xml version="1.0"?>
 <robot>
-  <material name="HumanHand/Skin">
+	<material name="HumanHand/Skin">
 		<color rgba="0.802 0.732 0.673 1.0"/>
 	</material>

File: robot/human_hand_simple.urdf.xacro (robot description, xacro)
@@ -2,43 +2,6 @@
 <robot xmlns:xacro="http://www.ros.org/wiki/xacro" name="human_hand">
 	<xacro:include filename="$(find human_hand_description)/model/human_hand.urdf.xacro"/>
-	<link name="box">
-		<visual>
-			<origin xyz="0 0 0.50" rpy="0 0 0"/>
-			<geometry>
-				<box size="1.0 1.0 1.0"/>
-			</geometry>
-		</visual>
-	</link>
-	<joint name="box_wrist_right_joint_1" type="revolute">
-		<origin xyz="0 0.2 1.02" rpy="0 0 0" />
-		<parent link="box"/>
-		<child link="wrist_right_fake_1"/>
-				<axis xyz="1 0 0" />
-				<limit lower="${abd_lb *pi/180}" upper="${abd_ub *pi/180}" effort="${effort}" velocity="${velocity}"/>
-    	<dynamics damping="${damping}" friction="${friction}"/>
-	</joint>
-	<link name="wrist_right_fake_1">
-	</link>
-	<joint name="box_wrist_right_joint_2" type="revolute">
-		<origin xyz="0 0 0" rpy="0 0 0" />
-		<parent link="wrist_right_fake_1"/>
-		<child link="wrist_right_fake_2"/>
-				<axis xyz="0 1 0" />
-				<limit lower="${abd_lb *pi/180}" upper="${abd_ub *pi/180}" effort="${effort}" velocity="${velocity}"/>
-    	<dynamics damping="${damping}" friction="${friction}"/>
-	</joint>
-	<link name="wrist_right_fake_2">
-	</link>
-	<joint name="box_wrist_right_joint_3" type="revolute">
-		<origin xyz="0 0 0" rpy="0 0 0" />
-		<parent link="wrist_right_fake_2"/>
-		<child link="wrist_right"/>
-				<axis xyz="0 0 1" />
-				<limit lower="${abd_lb *pi/180}" upper="${abd_ub *pi/180}" effort="${effort}" velocity="${velocity}"/>
-    	<dynamics damping="${damping}" friction="${friction}"/>
-	</joint>
-	<link name="wrist_right">
-	</link>
-	<xacro:human_hand parent="wrist_right" name="human_hand_right" left="false" useMimicTag="$(arg use_mimic_tag)" >
+	<link name="world"/>
+	<xacro:human_hand parent="world" name="human_hand_right" left="false" useMimicTag="$(arg use_mimic_tag)" >
 		<origin xyz="0.002 0.009 0.038" rpy="0 0 0"/>
 	</xacro:human_hand>
