Commit message: integrated glove_markers into hand model

File: model/human_hand.urdf.xacro (robot description, xacro)
@@ -3,5 +3,5 @@
 	<!--
 		HUMAN HAND MODEL v 0.1
-		urdf derived from human soft_hand
+		urdf derived from human Pisa SoftHand
 		author Guillaume Walck
 		meshes from GrabCAD, author Joerg Schmit
@@ -9,4 +9,5 @@
 	-->
 	<xacro:include filename="$(find human_hand_description)/model/materials.urdf.xacro"/>
+	<xacro:include filename="$(find human_hand_description)/model/glove_markers.urdf.xacro"/>
 	<xacro:property name="pi" value="3.1415926535897931" />
 	<!-- joint properties -->
@@ -65,5 +66,5 @@
 	<!-- SOFT FINGER model -->
 	<!-- 4 fingers are equal (index, middle, ring, little) -->
-	<xacro:macro name="soft_finger" params="parent parent_name prefix name swap position orientation proximal_len middle_len useMimicTag abd_R inner_R middle_R outer_R index:=1 middle:=0 ring:=0 little:=0 ">
+	<xacro:macro name="finger" params="parent parent_name prefix name reflect position orientation proximal_len middle_len useMimicTag abd_R inner_R middle_R outer_R index:=1 middle:=0 ring:=0 little:=0 ">
 		<!-- KNUCKLE -->
 		<joint name="${prefix}${name}_abd_joint" type="revolute">
@@ -71,5 +72,5 @@
 			<parent link="${parent}"/>
 			<child link="${prefix}${name}_knuckle_link"/>
-			<axis xyz="0 ${-1*swap} 0" />
+			<axis xyz="0 ${-1*reflect} 0" />
 			<limit lower="${abd_lb *pi/180}" upper="${abd_ub *pi/180}" effort="${effort}" velocity="${velocity}"/>
 			<dynamics damping="${damping}" friction="${friction}"/>
@@ -98,5 +99,5 @@
 				<geometry>
 						<mesh filename="package://human_hand_description/meshes/${name}_proximal.stl"
-						      scale="${0.001*swap} 0.001 .001" />
+						      scale="${0.001*reflect} 0.001 .001" />
 				</geometry>
 				<material name="HumanHand/Skin" />
@@ -119,5 +120,5 @@
 				<geometry>
 					<mesh filename="package://human_hand_description/meshes/${name}_middle.stl"
-					      scale="${0.001*swap} 0.001 .001" />
+					      scale="${0.001*reflect} 0.001 .001" />
 				</geometry>
 				<material name="HumanHand/Skin" />
@@ -140,5 +141,5 @@
 				<geometry>
 					<mesh filename="package://human_hand_description/meshes/${name}_distal.stl"
-					      scale="${0.001*swap} 0.001 .001" />
+					      scale="${0.001*reflect} 0.001 .001" />
 				</geometry>
 				 <material name="HumanHand/Skin" />
@@ -148,5 +149,5 @@
 	<!-- THUMB MODEL -->
 	<!-- It has one joint less than rest of fingers -->
-	<xacro:macro name="soft_thumb" params="parent parent_name name swap position orientation base_len proximal_len  useMimicTag abd_R inner_R outer_R ">
+	<xacro:macro name="thumb" params="parent parent_name name reflect position orientation base_len proximal_len  useMimicTag abd_R inner_R outer_R ">
 		<!-- THUMB -->
 			<!-- KNUCKLE -->
@@ -167,5 +168,5 @@
 				<parent link="${name}_fake_link"/>
 				<child link="${name}_knuckle_link"/>
-				<axis xyz="0 ${-1*swap} 0" />
+				<axis xyz="0 ${-1*reflect} 0" />
 				<limit lower="${thumb_abd_lb *pi/180}" upper="${thumb_abd_ub *pi/180}" effort="${effort}" velocity="${velocity}"/>
 				<dynamics damping="${damping}" friction="${friction}"/>
@@ -176,5 +177,5 @@
 					<geometry>
 						<mesh filename="package://human_hand_description/meshes/thumb_base.stl"
-						      scale="${0.001*swap} 0.001 .001" />
+						      scale="${0.001*reflect} 0.001 .001" />
 					</geometry>
 					<material name="HumanHand/Skin" />
@@ -186,5 +187,5 @@
 				<parent link="${name}_knuckle_link"/>
 				<child link="${name}_proximal_link"/>
-				<axis xyz="0 ${-1*swap} 0" />
+				<axis xyz="0 ${-1*reflect} 0" />
 				<limit lower="${inner_lb *pi/180}" upper="${inner_ub *pi/180}" effort="${effort}" velocity="${velocity}"/>
 				<dynamics damping="${damping}" friction="${friction}"/>
@@ -197,5 +198,5 @@
 				<geometry>
 					<mesh filename="package://human_hand_description/meshes/thumb_proximal.stl"
-					      scale="${0.001*swap} 0.001 .001" />
+					      scale="${0.001*reflect} 0.001 .001" />
 				</geometry>
 				<material name="HumanHand/Skin" />
@@ -207,5 +208,5 @@
 			<parent link="${name}_proximal_link"/>
 			<child link="${name}_distal_link"/>
-			<axis xyz="0 ${-1*swap} 0" />
+			<axis xyz="0 ${-1*reflect} 0" />
 			<limit lower="${outer_lb *pi/180}" upper="${outer_ub *pi/180}" effort="${effort}" velocity="${velocity}"/>
 			<xacro:if value="${useMimicTag}">
@@ -217,5 +218,5 @@
 				<geometry>
 					<mesh filename="package://human_hand_description/meshes/thumb_distal.stl"
-					      scale="${0.001*swap} 0.001 .001" />
+					      scale="${0.001*reflect} 0.001 .001" />
 				</geometry>
 				<material name="HumanHand/Skin" />
@@ -226,7 +227,7 @@
 	<xacro:macro name="human_hand" params="parent name useMimicTag left *origin">
 		<!-- left/right hand model-->
-		<xacro:property name="swap" value="1" />
+		<xacro:property name="reflect" value="1" />
 		<xacro:if value="${left}">
-			<xacro:property name="swap" value="-1" />
+			<xacro:property name="reflect" value="-1" />
 		</xacro:if>
 		<!-- PALM -->
@@ -240,5 +241,5 @@
 				<geometry>
 					<mesh filename="package://human_hand_description/meshes/palm.stl"
-					      scale=" ${.001*swap} .001 .001" />
+					      scale=" ${.001*reflect} .001 .001" />
 				</geometry>
 				<material name="HumanHand/Skin" />
@@ -257,9 +258,10 @@
 		</xacro:if>
 		<!-- THUMB AND FINGERS -->
-			<xacro:soft_thumb parent="${name}_palm_link" parent_name="${name}" name="${name}_thumb" swap="${swap}" position="${0.02475*swap} -0.0125 0.0125" orientation="0.0 ${0.6240*swap} 0" base_len="${thumb_base_len}" proximal_len="${thumb_proximal_len}" useMimicTag="${useMimicTag}" abd_R="${thumb_abd_R *(thumb_abd_ub - thumb_abd_lb)*pi/180}"  inner_R="${thumb_inner_R *(inner_ub - inner_lb)*pi/180}" outer_R="${thumb_outer_R *(outer_ub - outer_lb)*pi/180}" />
-			<xacro:soft_finger parent="${name}_palm_link" parent_name="${name}" prefix="${name}_" name="index" swap="${swap}" position="${0.02175*swap} -0.002 0.099" orientation="0 0 0" proximal_len="${index_proximal_len}" middle_len="${index_middle_len}"   useMimicTag="${useMimicTag}" abd_R="${index_abd_R}" inner_R="${index_inner_R *(inner_ub - inner_lb)*pi/180}" middle_R="${index_middle_R *(middle_ub - middle_lb)*pi/180}" outer_R="${index_outer_R *(outer_ub - outer_lb)*pi/180}" />
-			<xacro:soft_finger parent="${name}_palm_link" parent_name="${name}" prefix="${name}_" name="middle" swap="${swap}" position="${-0.002*swap} 0.0015 0.0955" orientation="0 0 0.0" proximal_len="${middle_proximal_len}" middle_len="${middle_middle_len}" useMimicTag="${useMimicTag}" abd_R="${middle_abd_R}" inner_R="${middle_inner_R *(inner_ub - inner_lb)*pi/180}" middle_R="${middle_middle_R *(middle_ub - middle_lb)*pi/180}" outer_R="${middle_outer_R *(outer_ub - outer_lb)*pi/180}"  />
-			<xacro:soft_finger parent="${name}_palm_link" parent_name="${name}" prefix="${name}_" name="ring" swap="${swap}" position="${-0.02225*swap} 0.0010 0.090" orientation="0 0 0" proximal_len="${ring_proximal_len}" middle_len="${ring_middle_len}" useMimicTag="${useMimicTag}" abd_R="${ring_abd_R}" inner_R="${ring_inner_R *(inner_ub - inner_lb)*pi/180}" middle_R="${ring_middle_R *(middle_ub - middle_lb)*pi/180}" outer_R="${ring_outer_R *(outer_ub - outer_lb)*pi/180}" />
-			<xacro:soft_finger parent="${name}_palm_link" parent_name="${name}" prefix="${name}_" name="little" swap="${swap}" position="${-0.04175*swap} -0.003 0.079" orientation="0 0 0" proximal_len="${little_proximal_len}" middle_len="${little_middle_len}" useMimicTag="${useMimicTag}" abd_R="${little_abd_R}" inner_R="${little_inner_R *(inner_ub - inner_lb)*pi/180}" middle_R="${little_middle_R *(middle_ub - middle_lb)*pi/180}" outer_R="${little_outer_R *(outer_ub - outer_lb)*pi/180}" />
+			<xacro:thumb parent="${name}_palm_link" parent_name="${name}" name="${name}_thumb" reflect="${reflect}" position="${0.02475*reflect} -0.0125 0.0125" orientation="0.0 ${0.6240*reflect} 0" base_len="${thumb_base_len}" proximal_len="${thumb_proximal_len}" useMimicTag="${useMimicTag}" abd_R="${thumb_abd_R *(thumb_abd_ub - thumb_abd_lb)*pi/180}"  inner_R="${thumb_inner_R *(inner_ub - inner_lb)*pi/180}" outer_R="${thumb_outer_R *(outer_ub - outer_lb)*pi/180}" />
+			<xacro:finger parent="${name}_palm_link" parent_name="${name}" prefix="${name}_" name="index" reflect="${reflect}" position="${0.02175*reflect} -0.002 0.099" orientation="0 0 0" proximal_len="${index_proximal_len}" middle_len="${index_middle_len}"   useMimicTag="${useMimicTag}" abd_R="${index_abd_R}" inner_R="${index_inner_R *(inner_ub - inner_lb)*pi/180}" middle_R="${index_middle_R *(middle_ub - middle_lb)*pi/180}" outer_R="${index_outer_R *(outer_ub - outer_lb)*pi/180}" />
+			<xacro:finger parent="${name}_palm_link" parent_name="${name}" prefix="${name}_" name="middle" reflect="${reflect}" position="${-0.002*reflect} 0.0015 0.0955" orientation="0 0 0.0" proximal_len="${middle_proximal_len}" middle_len="${middle_middle_len}" useMimicTag="${useMimicTag}" abd_R="${middle_abd_R}" inner_R="${middle_inner_R *(inner_ub - inner_lb)*pi/180}" middle_R="${middle_middle_R *(middle_ub - middle_lb)*pi/180}" outer_R="${middle_outer_R *(outer_ub - outer_lb)*pi/180}"  />
+			<xacro:finger parent="${name}_palm_link" parent_name="${name}" prefix="${name}_" name="ring" reflect="${reflect}" position="${-0.02225*reflect} 0.0010 0.090" orientation="0 0 0" proximal_len="${ring_proximal_len}" middle_len="${ring_middle_len}" useMimicTag="${useMimicTag}" abd_R="${ring_abd_R}" inner_R="${ring_inner_R *(inner_ub - inner_lb)*pi/180}" middle_R="${ring_middle_R *(middle_ub - middle_lb)*pi/180}" outer_R="${ring_outer_R *(outer_ub - outer_lb)*pi/180}" />
+			<xacro:finger parent="${name}_palm_link" parent_name="${name}" prefix="${name}_" name="little" reflect="${reflect}" position="${-0.04175*reflect} -0.003 0.079" orientation="0 0 0" proximal_len="${little_proximal_len}" middle_len="${little_middle_len}" useMimicTag="${useMimicTag}" abd_R="${little_abd_R}" inner_R="${little_inner_R *(inner_ub - inner_lb)*pi/180}" middle_R="${little_middle_R *(middle_ub - middle_lb)*pi/180}" outer_R="${little_outer_R *(outer_ub - outer_lb)*pi/180}" />
+			<xacro:tactile_glove name="${name}" reflect="${reflect}"/>
 	</xacro:macro>
 </robot>
