Commit message: separated taxel mapping from layout using a python dict for the mapping in xacro added mappings for P2 and P3r

File: model/P2.urdf.xacro (robot description, xacro)
@@ -2,4 +2,5 @@
 <robot name="tactile_glove_markers" xmlns:xacro="http://ros.org/wiki/xacro">
 	<xacro:macro name="taxel" params="channel link mesh offset ns">
+		<xacro:if value="${channel >= 0}">
 		<tactile topic="/TactileGlove" data="data[${channel}]" link="${_name}${link}" ns="${ns}" xs="0 4095">
 			<geometry>
@@ -9,71 +10,72 @@
 			<origin xyz="${offset}"/>
 		</tactile>
+		</xacro:if>
 	</xacro:macro>
 	<xacro:macro name="tactile_glove" params="name reflect:=1">
 		<xacro:property name="_name" value="${name}_"/>
 		<xacro:property name="_reflect" value="${reflect}"/>
-		<xacro:taxel channel="17"  ns="index" link="index_distal_link" mesh="idd" offset="0 0 1e-3"/>
-		<xacro:taxel channel="16" ns="index" link="index_distal_link" mesh="ido" offset="${-1e-3*_reflect} 0 0"/>
-		<xacro:taxel channel="29" ns="index" link="index_distal_link" mesh="idm" offset="0 -1e-3 0"/>
-		<xacro:taxel channel="18" ns="index" link="index_distal_link" mesh="idi" offset="${1e-3*_reflect} 0 0"/>
-		<xacro:taxel channel="20" ns="index" link="index_middle_link" mesh="imo" offset="${-1e-3*_reflect} 0 0"/>
-		<xacro:taxel channel="28" ns="index" link="index_middle_link" mesh="imm" offset="0 -1e-3 0"/>
-		<xacro:taxel channel="19" ns="index" link="index_middle_link" mesh="imi" offset="${1e-3*_reflect} 0 0"/>
-		<xacro:taxel channel="24" ns="index" link="index_proximal_link" mesh="ip" offset="0 -1e-3 0"/>
-		<xacro:taxel channel="30" ns="index" link="index_proximal_link" mesh="ipi" offset="${1e-3*_reflect} 0 0"/>
-		<xacro:taxel channel="39" ns="middle" link="middle_distal_link" mesh="mdd" offset="0 0 1e-3"/>
-		<xacro:taxel channel="40" ns="middle" link="middle_distal_link" mesh="mdo" offset="${-1e-3*_reflect} 0 0"/>
-		<xacro:taxel channel="44" ns="middle" link="middle_distal_link" mesh="mdm" offset="0 -1e-3 0"/>
-		<xacro:taxel channel="42" ns="middle" link="middle_distal_link" mesh="mdi" offset="${1e-3*_reflect} 0 0"/>
-		<xacro:taxel channel="38" ns="middle" link="middle_middle_link" mesh="mmo" offset="${-1e-3*_reflect} 0 0"/>
-		<xacro:taxel channel="43" ns="middle" link="middle_middle_link" mesh="mmm" offset="0 -1e-3 0"/>
-		<xacro:taxel channel="37" ns="middle" link="middle_middle_link" mesh="mmi" offset="${1e-3*_reflect} 0 0"/>
-		<xacro:taxel channel="41" ns="middle" link="middle_proximal_link" mesh="mp" offset="0 -1e-3 0"/>
-		<xacro:taxel channel="34" ns="ring" link="ring_distal_link" mesh="rdd" offset="0 0 1e-3"/>
-		<xacro:taxel channel="33" ns="ring" link="ring_distal_link" mesh="rdo" offset="${-1e-3*_reflect} 0 0"/>
-		<xacro:taxel channel="32" ns="ring" link="ring_distal_link" mesh="rdm" offset="0 -1e-3 0"/>
-		<xacro:taxel channel="46" ns="ring" link="ring_distal_link" mesh="rdi" offset="${1e-3*_reflect} 0 0"/>
-		<xacro:taxel channel="36" ns="ring" link="ring_middle_link" mesh="rmo" offset="${-1e-3*_reflect} 0 0"/>
-		<xacro:taxel channel="35" ns="ring" link="ring_middle_link" mesh="rmm" offset="0 -1e-3 0"/>
-		<xacro:taxel channel="31" ns="ring" link="ring_middle_link" mesh="rmi" offset="${1e-3*_reflect} 0 0"/>
-		<xacro:taxel channel="47" ns="ring" link="ring_proximal_link" mesh="rp" offset="0 -1e-3 0"/>
-		<xacro:taxel channel="6" ns="little" link="little_distal_link" mesh="ldd" offset="0 0 1e-3"/>
-		<xacro:taxel channel="5" ns="little" link="little_distal_link" mesh="ldo" offset="${-1e-3*_reflect} 0 0"/>
-		<xacro:taxel channel="7" ns="little" link="little_distal_link" mesh="ldm" offset="0 -1e-3 0"/>
-		<xacro:taxel channel="9" ns="little" link="little_distal_link" mesh="ldi" offset="${1e-3*_reflect} 0 0"/>
-		<xacro:taxel channel="10" ns="little" link="little_middle_link" mesh="lmo" offset="${-1e-3*_reflect} 0 0"/>
-		<xacro:taxel channel="11" ns="little" link="little_middle_link" mesh="lmm" offset="0 -1e-3 0"/>
-		<xacro:taxel channel="8" ns="little" link="little_middle_link" mesh="lmi" offset="${1e-3*_reflect} 0 0"/>
-		<xacro:taxel channel="13" ns="little" link="little_proximal_link" mesh="lpo" offset="${-1e-3*_reflect} 0 0"/>
-		<xacro:taxel channel="12" ns="little" link="little_proximal_link" mesh="lp" offset="0 -1e-3 0"/>
-		<xacro:taxel channel="51" ns="palm" link="palm_link" mesh="pdlo" offset="0 -1e-3 0"/>
-		<xacro:taxel channel="54" ns="palm" link="palm_link" mesh="pdl" offset="0 -1e-3 0"/>
-		<xacro:taxel channel="59" ns="palm" link="palm_link" mesh="pdr" offset="0 -1e-3 0"/>
-		<xacro:taxel channel="55" ns="palm" link="palm_link" mesh="pdm" offset="0 -1e-3 0"/>
-		<xacro:taxel channel="53" ns="palm" link="palm_link" mesh="pdi" offset="0 -1e-3 0"/>
-		<xacro:taxel channel="53" ns="palm" link="palm_link" mesh="pdii" offset="0 -1e-3 0"/>
-		<xacro:taxel channel="51" ns="palm" link="palm_link" mesh="pco" offset="0 -1e-3 0"/>
-		<xacro:taxel channel="50" ns="palm" link="palm_link" mesh="pcmp" offset="0 -1e-3 0"/>
-		<xacro:taxel channel="49" ns="palm" link="palm_link" mesh="pcmd" offset="0 -1e-3 0"/>
-		<xacro:taxel channel="62" ns="palm" link="palm_link" mesh="pcip" offset="0 -1e-3 0"/>
-		<xacro:taxel channel="48" ns="palm" link="palm_link" mesh="pcim" offset="0 -1e-3 0"/>n
-		<xacro:taxel channel="61" ns="palm" link="palm_link" mesh="pcid" offset="0 -1e-3 0"/>
-		<xacro:taxel channel="60" ns="palm" link="palm_link" mesh="ptop" offset="0 -1e-3 0"/>
-		<xacro:taxel channel="58" ns="palm" link="palm_link" mesh="ptod" offset="0 -1e-3 0"/>
-		<xacro:taxel channel="60" ns="palm" link="palm_link" mesh="ptmp" offset="0 -1e-3 0"/>
-		<xacro:taxel channel="58" ns="palm" link="palm_link" mesh="ptmd" offset="0 -1e-3 0"/>
-		<xacro:taxel channel="57" ns="palm" link="palm_link" mesh="ptip" offset="0 -1e-3 0"/>
-		<xacro:taxel channel="56" ns="palm" link="palm_link" mesh="ptid" offset="0 -1e-3 0"/>
-		<xacro:taxel channel="60" ns="thumb" link="thumb_knuckle_link" mesh="ptmp2" offset="0 -1e-3 0"/>
-		<xacro:taxel channel="58" ns="thumb" link="thumb_knuckle_link" mesh="ptmd2" offset="0 -1e-3 0"/>
-		<xacro:taxel channel="57" ns="thumb" link="thumb_knuckle_link" mesh="ptip2" offset="0 -1e-3 0"/>
-		<xacro:taxel channel="56" ns="thumb" link="thumb_knuckle_link" mesh="ptid2" offset="0 -1e-3 0"/>
-		<xacro:taxel channel="22" ns="thumb" link="thumb_distal_link" mesh="tdd" offset="0 0 1e-3"/>
-		<xacro:taxel channel="23" ns="thumb" link="thumb_distal_link" mesh="tdo" offset="0 1e-3 0"/>
-		<xacro:taxel channel="21" ns="thumb" link="thumb_distal_link" mesh="tdm" offset="${-1e-3*_reflect} 0 0"/>
-		<xacro:taxel channel="25" ns="thumb" link="thumb_distal_link" mesh="tdi" offset="0 -1e-3 0"/>
-		<xacro:taxel channel="27" ns="thumb" link="thumb_proximal_link" mesh="tpo" offset="0 1e-3 0"/>
-		<xacro:taxel channel="27" ns="thumb" link="thumb_proximal_link" mesh="tpm" offset="${-1e-3*_reflect} 0 0"/>
-		<xacro:taxel channel="26" ns="thumb" link="thumb_proximal_link" mesh="tpi" offset="0 -1e-3 0"/>
+		<xacro:taxel ns="index" link="index_distal_link" mesh="idd" channel="${tactMap.get('idd', -1)}" offset="0 0 1e-3"/>
+		<xacro:taxel ns="index" link="index_distal_link" mesh="ido" channel="${tactMap.get('ido', -1)}" offset="${-1e-3*_reflect} 0 0"/>
+		<xacro:taxel ns="index" link="index_distal_link" mesh="idm" channel="${tactMap.get('idm', -1)}" offset="0 -1e-3 0"/>
+		<xacro:taxel ns="index" link="index_distal_link" mesh="idi" channel="${tactMap.get('idi', -1)}" offset="${1e-3*_reflect} 0 0"/>
+		<xacro:taxel ns="index" link="index_middle_link" mesh="imo" channel="${tactMap.get('imo', -1)}" offset="${-1e-3*_reflect} 0 0"/>
+		<xacro:taxel ns="index" link="index_middle_link" mesh="imm" channel="${tactMap.get('imm', -1)}" offset="0 -1e-3 0"/>
+		<xacro:taxel ns="index" link="index_middle_link" mesh="imi" channel="${tactMap.get('imi', -1)}" offset="${1e-3*_reflect} 0 0"/>
+		<xacro:taxel ns="index" link="index_proximal_link" mesh="ip" channel="${tactMap.get('ip', -1)}" offset="0 -1e-3 0"/>
+		<xacro:taxel ns="index" link="index_proximal_link" mesh="ipi" channel="${tactMap.get('ipi', -1)}" offset="${1e-3*_reflect} 0 0"/>
+		<xacro:taxel ns="middle" link="middle_distal_link" mesh="mdd" channel="${tactMap.get('mdd', -1)}" offset="0 0 1e-3"/>
+		<xacro:taxel ns="middle" link="middle_distal_link" mesh="mdo" channel="${tactMap.get('mdo', -1)}" offset="${-1e-3*_reflect} 0 0"/>
+		<xacro:taxel ns="middle" link="middle_distal_link" mesh="mdm" channel="${tactMap.get('mdm', -1)}" offset="0 -1e-3 0"/>
+		<xacro:taxel ns="middle" link="middle_distal_link" mesh="mdi" channel="${tactMap.get('mdi', -1)}" offset="${1e-3*_reflect} 0 0"/>
+		<xacro:taxel ns="middle" link="middle_middle_link" mesh="mmo" channel="${tactMap.get('mmo', -1)}" offset="${-1e-3*_reflect} 0 0"/>
+		<xacro:taxel ns="middle" link="middle_middle_link" mesh="mmm" channel="${tactMap.get('mmm', -1)}" offset="0 -1e-3 0"/>
+		<xacro:taxel ns="middle" link="middle_middle_link" mesh="mmi" channel="${tactMap.get('mmi', -1)}" offset="${1e-3*_reflect} 0 0"/>
+		<xacro:taxel ns="middle" link="middle_proximal_link" mesh="mp" channel="${tactMap.get('mp', -1)}" offset="0 -1e-3 0"/>
+		<xacro:taxel ns="ring" link="ring_distal_link" mesh="rdd" channel="${tactMap.get('rdd', -1)}" offset="0 0 1e-3"/>
+		<xacro:taxel ns="ring" link="ring_distal_link" mesh="rdo" channel="${tactMap.get('rdo', -1)}" offset="${-1e-3*_reflect} 0 0"/>
+		<xacro:taxel ns="ring" link="ring_distal_link" mesh="rdm" channel="${tactMap.get('rdm', -1)}" offset="0 -1e-3 0"/>
+		<xacro:taxel ns="ring" link="ring_distal_link" mesh="rdi" channel="${tactMap.get('rdi', -1)}" offset="${1e-3*_reflect} 0 0"/>
+		<xacro:taxel ns="ring" link="ring_middle_link" mesh="rmo" channel="${tactMap.get('rmo', -1)}" offset="${-1e-3*_reflect} 0 0"/>
+		<xacro:taxel ns="ring" link="ring_middle_link" mesh="rmm" channel="${tactMap.get('rmm', -1)}" offset="0 -1e-3 0"/>
+		<xacro:taxel ns="ring" link="ring_middle_link" mesh="rmi" channel="${tactMap.get('rmi', -1)}" offset="${1e-3*_reflect} 0 0"/>
+		<xacro:taxel ns="ring" link="ring_proximal_link" mesh="rp" channel="${tactMap.get('rp', -1)}" offset="0 -1e-3 0"/>
+		<xacro:taxel ns="little" link="little_distal_link" mesh="ldd" channel="${tactMap.get('ldd', -1)}" offset="0 0 1e-3"/>
+		<xacro:taxel ns="little" link="little_distal_link" mesh="ldo" channel="${tactMap.get('ldo', -1)}" offset="${-1e-3*_reflect} 0 0"/>
+		<xacro:taxel ns="little" link="little_distal_link" mesh="ldm" channel="${tactMap.get('ldm', -1)}" offset="0 -1e-3 0"/>
+		<xacro:taxel ns="little" link="little_distal_link" mesh="ldi" channel="${tactMap.get('ldi', -1)}" offset="${1e-3*_reflect} 0 0"/>
+		<xacro:taxel ns="little" link="little_middle_link" mesh="lmo" channel="${tactMap.get('lmo', -1)}" offset="${-1e-3*_reflect} 0 0"/>
+		<xacro:taxel ns="little" link="little_middle_link" mesh="lmm" channel="${tactMap.get('lmm', -1)}" offset="0 -1e-3 0"/>
+		<xacro:taxel ns="little" link="little_middle_link" mesh="lmi" channel="${tactMap.get('lmi', -1)}" offset="${1e-3*_reflect} 0 0"/>
+		<xacro:taxel ns="little" link="little_proximal_link" mesh="lpo" channel="${tactMap.get('lpo', -1)}" offset="${-1e-3*_reflect} 0 0"/>
+		<xacro:taxel ns="little" link="little_proximal_link" mesh="lp" channel="${tactMap.get('lp', -1)}" offset="0 -1e-3 0"/>
+		<xacro:taxel ns="palm" link="palm_link" mesh="pdlo" channel="${tactMap.get('po', -1)}" offset="0 -1e-3 0"/>
+		<xacro:taxel ns="palm" link="palm_link" mesh="pdl" channel="${tactMap.get('pdl', -1)}" offset="0 -1e-3 0"/>
+		<xacro:taxel ns="palm" link="palm_link" mesh="pdr" channel="${tactMap.get('pdr', -1)}" offset="0 -1e-3 0"/>
+		<xacro:taxel ns="palm" link="palm_link" mesh="pdm" channel="${tactMap.get('pdm', -1)}" offset="0 -1e-3 0"/>
+		<xacro:taxel ns="palm" link="palm_link" mesh="pdi" channel="${tactMap.get('pdi', -1)}" offset="0 -1e-3 0"/>
+		<xacro:taxel ns="palm" link="palm_link" mesh="pdii" channel="${tactMap.get('pdii', -1)}" offset="0 -1e-3 0"/>
+		<xacro:taxel ns="palm" link="palm_link" mesh="pco" channel="${tactMap.get('po', -1)}" offset="0 -1e-3 0"/>
+		<xacro:taxel ns="palm" link="palm_link" mesh="pcmp" channel="${tactMap.get('pcmp', -1)}" offset="0 -1e-3 0"/>
+		<xacro:taxel ns="palm" link="palm_link" mesh="pcmd" channel="${tactMap.get('pcmd', -1)}" offset="0 -1e-3 0"/>
+		<xacro:taxel ns="palm" link="palm_link" mesh="pcip" channel="${tactMap.get('pcip', -1)}" offset="0 -1e-3 0"/>
+		<xacro:taxel ns="palm" link="palm_link" mesh="pcim" channel="${tactMap.get('pcim', -1)}" offset="0 -1e-3 0"/>n
+		<xacro:taxel ns="palm" link="palm_link" mesh="pcid" channel="${tactMap.get('pcid', -1)}" offset="0 -1e-3 0"/>
+		<xacro:taxel ns="palm" link="palm_link" mesh="ptop" channel="${tactMap.get('ptop', -1)}" offset="0 -1e-3 0"/>
+		<xacro:taxel ns="palm" link="palm_link" mesh="ptod" channel="${tactMap.get('ptod', -1)}" offset="0 -1e-3 0"/>
+		<xacro:taxel ns="palm" link="palm_link" mesh="ptmp" channel="${tactMap.get('ptop', -1)}" offset="0 -1e-3 0"/>
+		<xacro:taxel ns="palm" link="palm_link" mesh="ptmd" channel="${tactMap.get('ptod', -1)}" offset="0 -1e-3 0"/>
+		<xacro:taxel ns="palm" link="palm_link" mesh="ptip" channel="${tactMap.get('ptip', -1)}" offset="0 -1e-3 0"/>
+		<xacro:taxel ns="palm" link="palm_link" mesh="ptid" channel="${tactMap.get('ptid', -1)}" offset="0 -1e-3 0"/>
+		<xacro:taxel ns="thumb" link="thumb_knuckle_link" mesh="ptmp2" channel="${tactMap.get('ptop', -1)}" offset="0 -1e-3 0"/>
+		<xacro:taxel ns="thumb" link="thumb_knuckle_link" mesh="ptmd2" channel="${tactMap.get('ptod', -1)}" offset="0 -1e-3 0"/>
+		<xacro:taxel ns="thumb" link="thumb_knuckle_link" mesh="ptip2" channel="${tactMap.get('ptip', -1)}" offset="0 -1e-3 0"/>
+		<xacro:taxel ns="thumb" link="thumb_knuckle_link" mesh="ptid2" channel="${tactMap.get('ptid', -1)}" offset="0 -1e-3 0"/>
+		<xacro:taxel ns="thumb" link="thumb_distal_link" mesh="tdd" channel="${tactMap.get('tdd', -1)}" offset="0 0 1e-3"/>
+		<xacro:taxel ns="thumb" link="thumb_distal_link" mesh="tdo" channel="${tactMap.get('tdo', -1)}" offset="0 1e-3 0"/>
+		<xacro:taxel ns="thumb" link="thumb_distal_link" mesh="tdm" channel="${tactMap.get('tdm', -1)}" offset="${-1e-3*_reflect} 0 0"/>
+		<xacro:taxel ns="thumb" link="thumb_distal_link" mesh="tdi" channel="${tactMap.get('tdi', -1)}" offset="0 -1e-3 0"/>
+		<xacro:taxel ns="thumb" link="thumb_proximal_link" mesh="tpo" channel="${tactMap.get('tpo', -1)}" offset="0 1e-3 0"/>
+		<xacro:taxel ns="thumb" link="thumb_proximal_link" mesh="tpm" channel="${tactMap.get('tpm', -1)}" offset="${-1e-3*_reflect} 0 0"/>
+		<xacro:taxel ns="thumb" link="thumb_proximal_link" mesh="tpi" channel="${tactMap.get('tpi', -1)}" offset="0 -1e-3 0"/>
 	</xacro:macro>
 </robot>
