Commit message: separated taxel mapping from layout using a python dict for the mapping in xacro added mappings for P2 and P3r

File: model/P3.urdf.xacro (robot description, xacro)
@@ -2,79 +2,81 @@
 <robot name="tactile_glove_markers" xmlns:xacro="http://ros.org/wiki/xacro">
 	<xacro:macro name="taxel" params="channel link mesh offset ns">
-		<tactile topic="/TactileGlove" data="data[${channel}]" link="${_name}${link}" ns="${ns}" xs="0 4095">
-			<geometry>
-				<mesh filename="package://human_hand_description/meshes/taxels/${mesh}.stl"
-				      scale="${0.00101*_reflect} 0.00101 0.00101"/>
-			</geometry>
-			<origin xyz="${offset}"/>
-		</tactile>
+		<xacro:if value="${channel >= 0}">
+			<tactile topic="/TactileGlove" data="data[${channel}]" link="${_name}${link}" ns="${ns}" xs="0 4095">
+				<geometry>
+					<mesh filename="package://human_hand_description/meshes/taxels/${mesh}.stl"
+					      scale="${0.00101*_reflect} 0.00101 0.00101"/>
+				</geometry>
+				<origin xyz="${offset}"/>
+			</tactile>
+		</xacro:if>
 	</xacro:macro>
 	<xacro:macro name="tactile_glove" params="name reflect:=1">
 		<xacro:property name="_name" value="${name}_"/>
 		<xacro:property name="_reflect" value="${reflect}"/>
-		<xacro:taxel channel="45"  ns="index" link="index_distal_link" mesh="idd" offset="0 0 1e-3"/>
-		<xacro:taxel channel="42" ns="index" link="index_distal_link" mesh="ido" offset="${-1e-3*_reflect} 0 0"/>
-		<xacro:taxel channel="44" ns="index" link="index_distal_link" mesh="idm" offset="0 -1e-3 0"/>
-		<xacro:taxel channel="19" ns="index" link="index_distal_link" mesh="idi" offset="${1e-3*_reflect} 0 0"/>
-		<xacro:taxel channel="33" ns="index" link="index_middle_link" mesh="imo" offset="${-1e-3*_reflect} 0 0"/>
-		<xacro:taxel channel="40" ns="index" link="index_middle_link" mesh="imm" offset="0 -1e-3 0"/>
-		<xacro:taxel channel="28" ns="index" link="index_middle_link" mesh="imi" offset="${1e-3*_reflect} 0 0"/>
-		<xacro:taxel channel="43" ns="index" link="index_proximal_link" mesh="ip" offset="0 -1e-3 0"/>
-		<xacro:taxel channel="17" ns="index" link="index_proximal_link" mesh="ipi" offset="${1e-3*_reflect} 0 0"/>
-		<xacro:taxel channel="34" ns="middle" link="middle_distal_link" mesh="mdd" offset="0 0 1e-3"/>
-		<xacro:taxel channel="48" ns="middle" link="middle_distal_link" mesh="mdo" offset="${-1e-3*_reflect} 0 0"/>
-<!--		<xacro:taxel channel="-1" ns="middle" link="middle_distal_link" mesh="mdm" offset="0 -1e-3 0"/> -->
-		<xacro:taxel channel="38" ns="middle" link="middle_distal_link" mesh="mdi" offset="${1e-3*_reflect} 0 0"/>
-		<xacro:taxel channel="49" ns="middle" link="middle_middle_link" mesh="mmo" offset="${-1e-3*_reflect} 0 0"/>
-		<xacro:taxel channel="37" ns="middle" link="middle_middle_link" mesh="mmm" offset="0 -1e-3 0"/>
-		<xacro:taxel channel="39" ns="middle" link="middle_middle_link" mesh="mmi" offset="${1e-3*_reflect} 0 0"/>
-		<xacro:taxel channel="41" ns="middle" link="middle_proximal_link" mesh="mp" offset="0 -1e-3 0"/>
-		<xacro:taxel channel="61" ns="ring" link="ring_distal_link" mesh="rdd" offset="0 0 1e-3"/>
-		<xacro:taxel channel="55" ns="ring" link="ring_distal_link" mesh="rdo" offset="${-1e-3*_reflect} 0 0"/>
-		<xacro:taxel channel="52" ns="ring" link="ring_distal_link" mesh="rdm" offset="0 -1e-3 0"/>
-		<xacro:taxel channel="50" ns="ring" link="ring_distal_link" mesh="rdi" offset="${1e-3*_reflect} 0 0"/>
-		<xacro:taxel channel="54" ns="ring" link="ring_middle_link" mesh="rmo" offset="${-1e-3*_reflect} 0 0"/>
-		<xacro:taxel channel="63" ns="ring" link="ring_middle_link" mesh="rmm" offset="0 -1e-3 0"/>
-		<xacro:taxel channel="51" ns="ring" link="ring_middle_link" mesh="rmi" offset="${1e-3*_reflect} 0 0"/>
-		<xacro:taxel channel="62" ns="ring" link="ring_proximal_link" mesh="rp" offset="0 -1e-3 0"/>
-		<xacro:taxel channel="58" ns="little" link="little_distal_link" mesh="ldd" offset="0 0 1e-3"/>
-		<xacro:taxel channel="26" ns="little" link="little_distal_link" mesh="ldo" offset="${-1e-3*_reflect} 0 0"/>
-		<xacro:taxel channel="56" ns="little" link="little_distal_link" mesh="ldm" offset="0 -1e-3 0"/>
-		<xacro:taxel channel="53" ns="little" link="little_distal_link" mesh="ldi" offset="${1e-3*_reflect} 0 0"/>
-		<xacro:taxel channel="23" ns="little" link="little_middle_link" mesh="lmo" offset="${-1e-3*_reflect} 0 0"/>
-		<xacro:taxel channel="60" ns="little" link="little_middle_link" mesh="lmm" offset="0 -1e-3 0"/>
-		<xacro:taxel channel="57" ns="little" link="little_middle_link" mesh="lmi" offset="${1e-3*_reflect} 0 0"/>
-		<xacro:taxel channel="27" ns="little" link="little_proximal_link" mesh="lpo" offset="${-1e-3*_reflect} 0 0"/>
-		<xacro:taxel channel="59" ns="little" link="little_proximal_link" mesh="lp" offset="0 -1e-3 0"/>
-		<xacro:taxel channel="21" ns="palm" link="palm_link" mesh="pdlo" offset="0 -1e-3 0"/>
-		<xacro:taxel channel="23" ns="palm" link="palm_link" mesh="pdl" offset="0 -1e-3 0"/>
-		<xacro:taxel channel="25" ns="palm" link="palm_link" mesh="pdr" offset="0 -1e-3 0"/>
-		<xacro:taxel channel="29" ns="palm" link="palm_link" mesh="pdm" offset="0 -1e-3 0"/>
-		<xacro:taxel channel="30" ns="palm" link="palm_link" mesh="pdi" offset="0 -1e-3 0"/>
-		<xacro:taxel channel="18" ns="palm" link="palm_link" mesh="pdii" offset="0 -1e-3 0"/>
-		<xacro:taxel channel="7" ns="palm" link="palm_link" mesh="pco" offset="0 -1e-3 0"/>
-		<xacro:taxel channel="5" ns="palm" link="palm_link" mesh="pcmp" offset="0 -1e-3 0"/>
-		<xacro:taxel channel="24" ns="palm" link="palm_link" mesh="pcmd" offset="0 -1e-3 0"/>
-		<xacro:taxel channel="13" ns="palm" link="palm_link" mesh="pcip" offset="0 -1e-3 0"/>
-		<xacro:taxel channel="2" ns="palm" link="palm_link" mesh="pcim" offset="0 -1e-3 0"/>n
-		<xacro:taxel channel="10" ns="palm" link="palm_link" mesh="pcid" offset="0 -1e-3 0"/>
-		<xacro:taxel channel="16" ns="palm" link="palm_link" mesh="pi" offset="0 -1e-3 0"/>
-		<xacro:taxel channel="4" ns="palm" link="palm_link" mesh="ptop" offset="0 -1e-3 0"/>
-		<xacro:taxel channel="20" ns="palm" link="palm_link" mesh="ptod" offset="0 -1e-3 0"/>
-		<xacro:taxel channel="11" ns="palm" link="palm_link" mesh="ptmp" offset="0 -1e-3 0"/>
-		<xacro:taxel channel="6" ns="palm" link="palm_link" mesh="ptmd" offset="0 -1e-3 0"/>
-		<xacro:taxel channel="8" ns="palm" link="palm_link" mesh="ptip" offset="0 -1e-3 0"/>
-		<xacro:taxel channel="1" ns="palm" link="palm_link" mesh="ptid" offset="0 -1e-3 0"/>
-		<xacro:taxel channel="11" ns="thumb" link="thumb_knuckle_link" mesh="ptmp2" offset="0 -1e-3 0"/>
-		<xacro:taxel channel="6" ns="thumb" link="thumb_knuckle_link" mesh="ptmd2" offset="0 -1e-3 0"/>
-		<xacro:taxel channel="8" ns="thumb" link="thumb_knuckle_link" mesh="ptip2" offset="0 -1e-3 0"/>
-		<xacro:taxel channel="1" ns="thumb" link="thumb_knuckle_link" mesh="ptid2" offset="0 -1e-3 0"/>
-		<xacro:taxel channel="15" ns="thumb" link="thumb_distal_link" mesh="tdd" offset="0 0 1e-3"/>
-		<xacro:taxel channel="12" ns="thumb" link="thumb_distal_link" mesh="tdo" offset="0 1e-3 0"/>
-		<xacro:taxel channel="9" ns="thumb" link="thumb_distal_link" mesh="tdm" offset="${-1e-3*_reflect} 0 0"/>
-		<xacro:taxel channel="0" ns="thumb" link="thumb_distal_link" mesh="tdi" offset="0 -1e-3 0"/>
-		<xacro:taxel channel="14" ns="thumb" link="thumb_proximal_link" mesh="tpo" offset="0 1e-3 0"/>
-		<xacro:taxel channel="31" ns="thumb" link="thumb_proximal_link" mesh="tpm" offset="${-1e-3*_reflect} 0 0"/>
-		<xacro:taxel channel="2" ns="thumb" link="thumb_proximal_link" mesh="tpi" offset="0 -1e-3 0"/>
+		<xacro:taxel ns="index" link="index_distal_link" mesh="idd" channel="${tactMap.get('idd', -1)}" offset="0 0 1e-3"/>
+		<xacro:taxel ns="index" link="index_distal_link" mesh="ido" channel="${tactMap.get('ido', -1)}" offset="${-1e-3*_reflect} 0 0"/>
+		<xacro:taxel ns="index" link="index_distal_link" mesh="idm" channel="${tactMap.get('idm', -1)}" offset="0 -1e-3 0"/>
+		<xacro:taxel ns="index" link="index_distal_link" mesh="idi" channel="${tactMap.get('idi', -1)}" offset="${1e-3*_reflect} 0 0"/>
+		<xacro:taxel ns="index" link="index_middle_link" mesh="imo" channel="${tactMap.get('imo', -1)}" offset="${-1e-3*_reflect} 0 0"/>
+		<xacro:taxel ns="index" link="index_middle_link" mesh="imm" channel="${tactMap.get('imm', -1)}" offset="0 -1e-3 0"/>
+		<xacro:taxel ns="index" link="index_middle_link" mesh="imi" channel="${tactMap.get('imi', -1)}" offset="${1e-3*_reflect} 0 0"/>
+		<xacro:taxel ns="index" link="index_proximal_link" mesh="ip" channel="${tactMap.get('ip', -1)}" offset="0 -1e-3 0"/>
+		<xacro:taxel ns="index" link="index_proximal_link" mesh="ipi" channel="${tactMap.get('ipi', -1)}" offset="${1e-3*_reflect} 0 0"/>
+		<xacro:taxel ns="middle" link="middle_distal_link" mesh="mdd" channel="${tactMap.get('mdd', -1)}" offset="0 0 1e-3"/>
+		<xacro:taxel ns="middle" link="middle_distal_link" mesh="mdo" channel="${tactMap.get('mdo', -1)}" offset="${-1e-3*_reflect} 0 0"/>
+		<xacro:taxel ns="middle" link="middle_distal_link" mesh="mdm" channel="${tactMap.get('mdm', -1)}" offset="0 -1e-3 0"/>
+		<xacro:taxel ns="middle" link="middle_distal_link" mesh="mdi" channel="${tactMap.get('mdi', -1)}" offset="${1e-3*_reflect} 0 0"/>
+		<xacro:taxel ns="middle" link="middle_middle_link" mesh="mmo" channel="${tactMap.get('mmo', -1)}" offset="${-1e-3*_reflect} 0 0"/>
+		<xacro:taxel ns="middle" link="middle_middle_link" mesh="mmm" channel="${tactMap.get('mmm', -1)}" offset="0 -1e-3 0"/>
+		<xacro:taxel ns="middle" link="middle_middle_link" mesh="mmi" channel="${tactMap.get('mmi', -1)}" offset="${1e-3*_reflect} 0 0"/>
+		<xacro:taxel ns="middle" link="middle_proximal_link" mesh="mp" channel="${tactMap.get('mp', -1)}" offset="0 -1e-3 0"/>
+		<xacro:taxel ns="ring" link="ring_distal_link" mesh="rdd" channel="${tactMap.get('rdd', -1)}" offset="0 0 1e-3"/>
+		<xacro:taxel ns="ring" link="ring_distal_link" mesh="rdo" channel="${tactMap.get('rdo', -1)}" offset="${-1e-3*_reflect} 0 0"/>
+		<xacro:taxel ns="ring" link="ring_distal_link" mesh="rdm" channel="${tactMap.get('rdm', -1)}" offset="0 -1e-3 0"/>
+		<xacro:taxel ns="ring" link="ring_distal_link" mesh="rdi" channel="${tactMap.get('rdi', -1)}" offset="${1e-3*_reflect} 0 0"/>
+		<xacro:taxel ns="ring" link="ring_middle_link" mesh="rmo" channel="${tactMap.get('rmo', -1)}" offset="${-1e-3*_reflect} 0 0"/>
+		<xacro:taxel ns="ring" link="ring_middle_link" mesh="rmm" channel="${tactMap.get('rmm', -1)}" offset="0 -1e-3 0"/>
+		<xacro:taxel ns="ring" link="ring_middle_link" mesh="rmi" channel="${tactMap.get('rmi', -1)}" offset="${1e-3*_reflect} 0 0"/>
+		<xacro:taxel ns="ring" link="ring_proximal_link" mesh="rp" channel="${tactMap.get('rp', -1)}" offset="0 -1e-3 0"/>
+		<xacro:taxel ns="little" link="little_distal_link" mesh="ldd" channel="${tactMap.get('ldd', -1)}" offset="0 0 1e-3"/>
+		<xacro:taxel ns="little" link="little_distal_link" mesh="ldo" channel="${tactMap.get('ldo', -1)}" offset="${-1e-3*_reflect} 0 0"/>
+		<xacro:taxel ns="little" link="little_distal_link" mesh="ldm" channel="${tactMap.get('ldm', -1)}" offset="0 -1e-3 0"/>
+		<xacro:taxel ns="little" link="little_distal_link" mesh="ldi" channel="${tactMap.get('ldi', -1)}" offset="${1e-3*_reflect} 0 0"/>
+		<xacro:taxel ns="little" link="little_middle_link" mesh="lmo" channel="${tactMap.get('lmo', -1)}" offset="${-1e-3*_reflect} 0 0"/>
+		<xacro:taxel ns="little" link="little_middle_link" mesh="lmm" channel="${tactMap.get('lmm', -1)}" offset="0 -1e-3 0"/>
+		<xacro:taxel ns="little" link="little_middle_link" mesh="lmi" channel="${tactMap.get('lmi', -1)}" offset="${1e-3*_reflect} 0 0"/>
+		<xacro:taxel ns="little" link="little_proximal_link" mesh="lpo" channel="${tactMap.get('lpo', -1)}" offset="${-1e-3*_reflect} 0 0"/>
+		<xacro:taxel ns="little" link="little_proximal_link" mesh="lp" channel="${tactMap.get('lp', -1)}" offset="0 -1e-3 0"/>
+		<xacro:taxel ns="palm" link="palm_link" mesh="pdlo" channel="${tactMap.get('pdlo', -1)}" offset="0 -1e-3 0"/>
+		<xacro:taxel ns="palm" link="palm_link" mesh="pdl" channel="${tactMap.get('pdl', -1)}" offset="0 -1e-3 0"/>
+		<xacro:taxel ns="palm" link="palm_link" mesh="pdr" channel="${tactMap.get('pdr', -1)}" offset="0 -1e-3 0"/>
+		<xacro:taxel ns="palm" link="palm_link" mesh="pdm" channel="${tactMap.get('pdm', -1)}" offset="0 -1e-3 0"/>
+		<xacro:taxel ns="palm" link="palm_link" mesh="pdi" channel="${tactMap.get('pdi', -1)}" offset="0 -1e-3 0"/>
+		<xacro:taxel ns="palm" link="palm_link" mesh="pdii" channel="${tactMap.get('pdii', -1)}" offset="0 -1e-3 0"/>
+		<xacro:taxel ns="palm" link="palm_link" mesh="pco" channel="${tactMap.get('pco', -1)}" offset="0 -1e-3 0"/>
+		<xacro:taxel ns="palm" link="palm_link" mesh="pcmp" channel="${tactMap.get('pcmp', -1)}" offset="0 -1e-3 0"/>
+		<xacro:taxel ns="palm" link="palm_link" mesh="pcmd" channel="${tactMap.get('pcmd', -1)}" offset="0 -1e-3 0"/>
+		<xacro:taxel ns="palm" link="palm_link" mesh="pcip" channel="${tactMap.get('pcip', -1)}" offset="0 -1e-3 0"/>
+		<xacro:taxel ns="palm" link="palm_link" mesh="pcim" channel="${tactMap.get('pcim', -1)}" offset="0 -1e-3 0"/>n
+		<xacro:taxel ns="palm" link="palm_link" mesh="pcid" channel="${tactMap.get('pcid', -1)}" offset="0 -1e-3 0"/>
+		<xacro:taxel ns="palm" link="palm_link" mesh="pi" channel="${tactMap.get('pi', -1)}" offset="0 -1e-3 0"/>
+		<xacro:taxel ns="palm" link="palm_link" mesh="ptop" channel="${tactMap.get('ptop', -1)}" offset="0 -1e-3 0"/>
+		<xacro:taxel ns="palm" link="palm_link" mesh="ptod" channel="${tactMap.get('ptod', -1)}" offset="0 -1e-3 0"/>
+		<xacro:taxel ns="palm" link="palm_link" mesh="ptmp" channel="${tactMap.get('ptmp', -1)}" offset="0 -1e-3 0"/>
+		<xacro:taxel ns="palm" link="palm_link" mesh="ptmd" channel="${tactMap.get('ptmd', -1)}" offset="0 -1e-3 0"/>
+		<xacro:taxel ns="palm" link="palm_link" mesh="ptip" channel="${tactMap.get('ptip', -1)}" offset="0 -1e-3 0"/>
+		<xacro:taxel ns="palm" link="palm_link" mesh="ptid" channel="${tactMap.get('ptid', -1)}" offset="0 -1e-3 0"/>
+		<xacro:taxel ns="thumb" link="thumb_knuckle_link" mesh="ptmp2" channel="${tactMap.get('ptmp', -1)}" offset="0 -1e-3 0"/>
+		<xacro:taxel ns="thumb" link="thumb_knuckle_link" mesh="ptmd2" channel="${tactMap.get('ptmd', -1)}" offset="0 -1e-3 0"/>
+		<xacro:taxel ns="thumb" link="thumb_knuckle_link" mesh="ptip2" channel="${tactMap.get('ptip', -1)}" offset="0 -1e-3 0"/>
+		<xacro:taxel ns="thumb" link="thumb_knuckle_link" mesh="ptid2" channel="${tactMap.get('ptid', -1)}" offset="0 -1e-3 0"/>
+		<xacro:taxel ns="thumb" link="thumb_distal_link" mesh="tdd" channel="${tactMap.get('tdd', -1)}" offset="0 0 1e-3"/>
+		<xacro:taxel ns="thumb" link="thumb_distal_link" mesh="tdo" channel="${tactMap.get('tdo', -1)}" offset="0 1e-3 0"/>
+		<xacro:taxel ns="thumb" link="thumb_distal_link" mesh="tdm" channel="${tactMap.get('tdm', -1)}" offset="${-1e-3*_reflect} 0 0"/>
+		<xacro:taxel ns="thumb" link="thumb_distal_link" mesh="tdi" channel="${tactMap.get('tdi', -1)}" offset="0 -1e-3 0"/>
+		<xacro:taxel ns="thumb" link="thumb_proximal_link" mesh="tpo" channel="${tactMap.get('tpo', -1)}" offset="0 1e-3 0"/>
+		<xacro:taxel ns="thumb" link="thumb_proximal_link" mesh="tpm" channel="${tactMap.get('tpm', -1)}" offset="${-1e-3*_reflect} 0 0"/>
+		<xacro:taxel ns="thumb" link="thumb_proximal_link" mesh="tpi" channel="${tactMap.get('tpi', -1)}" offset="0 -1e-3 0"/>
 	</xacro:macro>
 </robot>

File: model/human_hand.urdf.xacro (robot description, xacro)
@@ -9,6 +9,5 @@
 	-->
 	<xacro:include filename="$(find human_hand_description)/model/materials.urdf.xacro"/>
-	<xacro:include filename="$(find human_hand_description)/model/${tactile_mapping}.urdf.xacro"/>
-	<xacro:property name="pi" value="3.1415926535897931" />
+	<xacro:property name="_tactileMappingToLayout" value="{'P2':'P2', 'P3l':'P3', 'P3r':'P3'}"/>
 	<!-- joint properties -->
 	<xacro:property name="abd_lb" value="-30" />
@@ -263,4 +262,6 @@
 			<xacro:finger parent="${name}_palm_link" parent_name="${name}" prefix="${name}_" name="ring" reflect="${reflect}" position="${-0.02225*reflect} 0.0010 0.090" orientation="0 0 0" proximal_len="${ring_proximal_len}" middle_len="${ring_middle_len}" useMimicTag="${useMimicTag}" abd_R="${ring_abd_R}" inner_R="${ring_inner_R *(inner_ub - inner_lb)*pi/180}" middle_R="${ring_middle_R *(middle_ub - middle_lb)*pi/180}" outer_R="${ring_outer_R *(outer_ub - outer_lb)*pi/180}" />
 			<xacro:finger parent="${name}_palm_link" parent_name="${name}" prefix="${name}_" name="little" reflect="${reflect}" position="${-0.04175*reflect} -0.003 0.079" orientation="0 0 0" proximal_len="${little_proximal_len}" middle_len="${little_middle_len}" useMimicTag="${useMimicTag}" abd_R="${little_abd_R}" inner_R="${little_inner_R *(inner_ub - inner_lb)*pi/180}" middle_R="${little_middle_R *(middle_ub - middle_lb)*pi/180}" outer_R="${little_outer_R *(outer_ub - outer_lb)*pi/180}" />
+			<xacro:include filename="$(find human_hand_description)/model/${tactile_mapping}.mapping.xacro"/>
+			<xacro:include filename="$(find human_hand_description)/model/${_tactileMappingToLayout[tactile_mapping]}.urdf.xacro"/>
 			<xacro:tactile_glove name="${name}" reflect="${reflect}"/>
 	</xacro:macro>

File: robot/human_hand.urdf.xacro (robot description, xacro)
@@ -3,5 +3,5 @@
 	<xacro:arg name="left_hand" default="false"/>
 	<xacro:arg name="use_mimic_tag" default="false"/>
-	<xacro:arg name="tactile_mapping" default="P3"/>
+	<xacro:arg name="tactile_mapping" default="P3r"/>
 	<xacro:property name="tactile_mapping" value="$(arg tactile_mapping)"/>
 	<xacro:include filename="$(find human_hand_description)/model/human_hand.urdf.xacro"/>
