Commit message: renamed: robot->robots, meshes->model/meshes

File: model/P2.urdf.xacro (robot description, xacro)
@@ -5,5 +5,5 @@
 		<tactile topic="/TactileGlove" data="data[${channel}]" link="${_name}${link}" ns="${ns}" xs="0 4095">
 			<geometry>
-				<mesh filename="package://human_hand_description/meshes/taxels/${mesh}.stl"
+				<mesh filename="package://human_hand_description/model/meshes/taxels/${mesh}.stl"
 				      scale="${0.00101*_reflect} 0.00101 0.00101"/>
 			</geometry>

File: model/P3.urdf.xacro (robot description, xacro)
@@ -5,5 +5,5 @@
 			<tactile topic="/TactileGlove" data="data[${channel}]" link="${_name}${link}" ns="${ns}" xs="0 4095">
 				<geometry>
-					<mesh filename="package://human_hand_description/meshes/taxels/${mesh}.stl"
+					<mesh filename="package://human_hand_description/model/meshes/taxels/${mesh}.stl"
 					      scale="${0.00101*_reflect} 0.00101 0.00101"/>
 				</geometry>

File: model/human_hand.urdf.xacro (robot description, xacro)
@@ -2,9 +2,9 @@
 <robot xmlns:xacro="http://ros.org/wiki/xacro">
 	<!--
-		HUMAN HAND MODEL v 0.1
-		urdf derived from human Pisa SoftHand
-		author Guillaume Walck
-		meshes from GrabCAD, author Joerg Schmit
-		original CAD model available at: https://grabcad.com/library/human-left-hand/
+	    HUMAN HAND MODEL v 0.1
+	    urdf derived from human Pisa SoftHand
+	    author Guillaume Walck
+	    meshes from GrabCAD, author Joerg Schmit
+	    original CAD model available at: https://grabcad.com/library/human-left-hand/
 	-->
 	<xacro:include filename="$(find human_hand_description)/model/materials.urdf.xacro"/>
@@ -93,10 +93,10 @@
 		<link name="${prefix}${name}_proximal_link">
 			<!-- <inertial>
-				<insert_block name="phalanx_inertia"/>
-			</inertial> -->
-			<visual>
-				<geometry>
-						<mesh filename="package://human_hand_description/meshes/${name}_proximal.stl"
-						      scale="${0.001*reflect} 0.001 .001" />
+			     <insert_block name="phalanx_inertia"/>
+			     </inertial> -->
+			<visual>
+				<geometry>
+					<mesh filename="package://human_hand_description/model/meshes/${name}_proximal.stl"
+					      scale="${0.001*reflect} 0.001 .001" />
 				</geometry>
 				<material name="HumanHand/Skin" />
@@ -118,5 +118,5 @@
 			<visual>
 				<geometry>
-					<mesh filename="package://human_hand_description/meshes/${name}_middle.stl"
+					<mesh filename="package://human_hand_description/model/meshes/${name}_middle.stl"
 					      scale="${0.001*reflect} 0.001 .001" />
 				</geometry>
@@ -139,8 +139,8 @@
 			<visual>
 				<geometry>
-					<mesh filename="package://human_hand_description/meshes/${name}_distal.stl"
-					      scale="${0.001*reflect} 0.001 .001" />
-				</geometry>
-				 <material name="HumanHand/Skin" />
+					<mesh filename="package://human_hand_description/model/meshes/${name}_distal.stl"
+					      scale="${0.001*reflect} 0.001 .001" />
+				</geometry>
+				<material name="HumanHand/Skin" />
 			</visual>
 		</link>
@@ -150,51 +150,51 @@
 	<xacro:macro name="thumb" params="parent parent_name name reflect position orientation base_len proximal_len  useMimicTag abd_R inner_R outer_R ">
 		<!-- THUMB -->
-			<!-- KNUCKLE -->
-			<joint name="${name}_abd_joint" type="revolute">
-				<origin xyz="${position}" rpy="${orientation}" />
-				<parent link="${parent}"/>
-				<child link="${name}_fake_link"/>
-				<axis xyz="1 0 0" />
-				<limit lower="${thumb_abd_lb *pi/180}" upper="${thumb_abd_ub *pi/180}" effort="${effort}" velocity="${velocity}"/>
-				<dynamics damping="${damping}" friction="${friction}"/>
-				<xacro:if value="${useMimicTag}">
-					<mimic joint="${parent_name}_synergy_joint" multiplier="${abd_R}"/>
-				</xacro:if>
-			</joint>
-			<link name="${name}_fake_link"/>
-			<joint name="${name}_rot_joint" type="revolute">
+		<!-- KNUCKLE -->
+		<joint name="${name}_abd_joint" type="revolute">
+			<origin xyz="${position}" rpy="${orientation}" />
+			<parent link="${parent}"/>
+			<child link="${name}_fake_link"/>
+			<axis xyz="1 0 0" />
+			<limit lower="${thumb_abd_lb *pi/180}" upper="${thumb_abd_ub *pi/180}" effort="${effort}" velocity="${velocity}"/>
+			<dynamics damping="${damping}" friction="${friction}"/>
+			<xacro:if value="${useMimicTag}">
+				<mimic joint="${parent_name}_synergy_joint" multiplier="${abd_R}"/>
+			</xacro:if>
+		</joint>
+		<link name="${name}_fake_link"/>
+		<joint name="${name}_rot_joint" type="revolute">
+			<origin xyz="0 0 0" rpy="0 0 0" />
+			<parent link="${name}_fake_link"/>
+			<child link="${name}_knuckle_link"/>
+			<axis xyz="0 ${-1*reflect} 0" />
+			<limit lower="${thumb_abd_lb *pi/180}" upper="${thumb_abd_ub *pi/180}" effort="${effort}" velocity="${velocity}"/>
+			<dynamics damping="${damping}" friction="${friction}"/>
+		</joint>
+		<link name="${name}_knuckle_link">
+			<visual>
 				<origin xyz="0 0 0" rpy="0 0 0" />
-				<parent link="${name}_fake_link"/>
-				<child link="${name}_knuckle_link"/>
-				<axis xyz="0 ${-1*reflect} 0" />
-				<limit lower="${thumb_abd_lb *pi/180}" upper="${thumb_abd_ub *pi/180}" effort="${effort}" velocity="${velocity}"/>
-				<dynamics damping="${damping}" friction="${friction}"/>
-			</joint>
-			<link name="${name}_knuckle_link">
-				<visual>
-					<origin xyz="0 0 0" rpy="0 0 0" />
-					<geometry>
-						<mesh filename="package://human_hand_description/meshes/thumb_base.stl"
-						      scale="${0.001*reflect} 0.001 .001" />
-					</geometry>
-					<material name="HumanHand/Skin" />
-				</visual>
-			</link>
-			<!-- PROXIMAL PHALANGE -->
-			<joint name="${name}_inner_joint" type="revolute">
-				<origin xyz="0.0 0.0 ${base_len}" rpy="0.0 0.0 0.0" />
-				<parent link="${name}_knuckle_link"/>
-				<child link="${name}_proximal_link"/>
-				<axis xyz="0 ${-1*reflect} 0" />
-				<limit lower="${inner_lb *pi/180}" upper="${inner_ub *pi/180}" effort="${effort}" velocity="${velocity}"/>
-				<dynamics damping="${damping}" friction="${friction}"/>
-				<xacro:if value="${useMimicTag}">
-					<mimic joint="${parent_name}_synergy_joint" multiplier="${inner_R}"/>
-				</xacro:if>
-			</joint>
+				<geometry>
+					<mesh filename="package://human_hand_description/model/meshes/thumb_base.stl"
+					      scale="${0.001*reflect} 0.001 .001" />
+				</geometry>
+				<material name="HumanHand/Skin" />
+			</visual>
+		</link>
+		<!-- PROXIMAL PHALANGE -->
+		<joint name="${name}_inner_joint" type="revolute">
+			<origin xyz="0.0 0.0 ${base_len}" rpy="0.0 0.0 0.0" />
+			<parent link="${name}_knuckle_link"/>
+			<child link="${name}_proximal_link"/>
+			<axis xyz="0 ${-1*reflect} 0" />
+			<limit lower="${inner_lb *pi/180}" upper="${inner_ub *pi/180}" effort="${effort}" velocity="${velocity}"/>
+			<dynamics damping="${damping}" friction="${friction}"/>
+			<xacro:if value="${useMimicTag}">
+				<mimic joint="${parent_name}_synergy_joint" multiplier="${inner_R}"/>
+			</xacro:if>
+		</joint>
 		<link name="${name}_proximal_link">
 			<visual>
 				<geometry>
-					<mesh filename="package://human_hand_description/meshes/thumb_proximal.stl"
+					<mesh filename="package://human_hand_description/model/meshes/thumb_proximal.stl"
 					      scale="${0.001*reflect} 0.001 .001" />
 				</geometry>
@@ -216,5 +216,5 @@
 			<visual>
 				<geometry>
-					<mesh filename="package://human_hand_description/meshes/thumb_distal.stl"
+					<mesh filename="package://human_hand_description/model/meshes/thumb_distal.stl"
 					      scale="${0.001*reflect} 0.001 .001" />
 				</geometry>
@@ -239,5 +239,5 @@
 			<visual>
 				<geometry>
-					<mesh filename="package://human_hand_description/meshes/palm.stl"
+					<mesh filename="package://human_hand_description/model/meshes/palm.stl"
 					      scale=" ${.001*reflect} .001 .001" />
 				</geometry>
@@ -257,12 +257,12 @@
 		</xacro:if>
 		<!-- THUMB AND FINGERS -->
-			<xacro:thumb parent="${name}_palm_link" parent_name="${name}" name="${name}_thumb" reflect="${reflect}" position="${0.02475*reflect} -0.0125 0.0125" orientation="0.0 ${0.6240*reflect} 0" base_len="${thumb_base_len}" proximal_len="${thumb_proximal_len}" useMimicTag="${useMimicTag}" abd_R="${thumb_abd_R *(thumb_abd_ub - thumb_abd_lb)*pi/180}"  inner_R="${thumb_inner_R *(inner_ub - inner_lb)*pi/180}" outer_R="${thumb_outer_R *(outer_ub - outer_lb)*pi/180}" />
-			<xacro:finger parent="${name}_palm_link" parent_name="${name}" prefix="${name}_" name="index" reflect="${reflect}" position="${0.02175*reflect} -0.002 0.099" orientation="0 0 0" proximal_len="${index_proximal_len}" middle_len="${index_middle_len}"   useMimicTag="${useMimicTag}" abd_R="${index_abd_R}" inner_R="${index_inner_R *(inner_ub - inner_lb)*pi/180}" middle_R="${index_middle_R *(middle_ub - middle_lb)*pi/180}" outer_R="${index_outer_R *(outer_ub - outer_lb)*pi/180}" />
-			<xacro:finger parent="${name}_palm_link" parent_name="${name}" prefix="${name}_" name="middle" reflect="${reflect}" position="${-0.002*reflect} 0.0015 0.0955" orientation="0 0 0.0" proximal_len="${middle_proximal_len}" middle_len="${middle_middle_len}" useMimicTag="${useMimicTag}" abd_R="${middle_abd_R}" inner_R="${middle_inner_R *(inner_ub - inner_lb)*pi/180}" middle_R="${middle_middle_R *(middle_ub - middle_lb)*pi/180}" outer_R="${middle_outer_R *(outer_ub - outer_lb)*pi/180}"  />
-			<xacro:finger parent="${name}_palm_link" parent_name="${name}" prefix="${name}_" name="ring" reflect="${reflect}" position="${-0.02225*reflect} 0.0010 0.090" orientation="0 0 0" proximal_len="${ring_proximal_len}" middle_len="${ring_middle_len}" useMimicTag="${useMimicTag}" abd_R="${ring_abd_R}" inner_R="${ring_inner_R *(inner_ub - inner_lb)*pi/180}" middle_R="${ring_middle_R *(middle_ub - middle_lb)*pi/180}" outer_R="${ring_outer_R *(outer_ub - outer_lb)*pi/180}" />
-			<xacro:finger parent="${name}_palm_link" parent_name="${name}" prefix="${name}_" name="little" reflect="${reflect}" position="${-0.04175*reflect} -0.003 0.079" orientation="0 0 0" proximal_len="${little_proximal_len}" middle_len="${little_middle_len}" useMimicTag="${useMimicTag}" abd_R="${little_abd_R}" inner_R="${little_inner_R *(inner_ub - inner_lb)*pi/180}" middle_R="${little_middle_R *(middle_ub - middle_lb)*pi/180}" outer_R="${little_outer_R *(outer_ub - outer_lb)*pi/180}" />
-			<xacro:include filename="$(find human_hand_description)/model/${tactile_mapping}.mapping.xacro"/>
-			<xacro:include filename="$(find human_hand_description)/model/${_tactileMappingToLayout[tactile_mapping]}.urdf.xacro"/>
-			<xacro:tactile_glove name="${name}" reflect="${reflect}"/>
+		<xacro:thumb parent="${name}_palm_link" parent_name="${name}" name="${name}_thumb" reflect="${reflect}" position="${0.02475*reflect} -0.0125 0.0125" orientation="0.0 ${0.6240*reflect} 0" base_len="${thumb_base_len}" proximal_len="${thumb_proximal_len}" useMimicTag="${useMimicTag}" abd_R="${thumb_abd_R *(thumb_abd_ub - thumb_abd_lb)*pi/180}"  inner_R="${thumb_inner_R *(inner_ub - inner_lb)*pi/180}" outer_R="${thumb_outer_R *(outer_ub - outer_lb)*pi/180}" />
+		<xacro:finger parent="${name}_palm_link" parent_name="${name}" prefix="${name}_" name="index" reflect="${reflect}" position="${0.02175*reflect} -0.002 0.099" orientation="0 0 0" proximal_len="${index_proximal_len}" middle_len="${index_middle_len}"   useMimicTag="${useMimicTag}" abd_R="${index_abd_R}" inner_R="${index_inner_R *(inner_ub - inner_lb)*pi/180}" middle_R="${index_middle_R *(middle_ub - middle_lb)*pi/180}" outer_R="${index_outer_R *(outer_ub - outer_lb)*pi/180}" />
+		<xacro:finger parent="${name}_palm_link" parent_name="${name}" prefix="${name}_" name="middle" reflect="${reflect}" position="${-0.002*reflect} 0.0015 0.0955" orientation="0 0 0.0" proximal_len="${middle_proximal_len}" middle_len="${middle_middle_len}" useMimicTag="${useMimicTag}" abd_R="${middle_abd_R}" inner_R="${middle_inner_R *(inner_ub - inner_lb)*pi/180}" middle_R="${middle_middle_R *(middle_ub - middle_lb)*pi/180}" outer_R="${middle_outer_R *(outer_ub - outer_lb)*pi/180}"  />
+		<xacro:finger parent="${name}_palm_link" parent_name="${name}" prefix="${name}_" name="ring" reflect="${reflect}" position="${-0.02225*reflect} 0.0010 0.090" orientation="0 0 0" proximal_len="${ring_proximal_len}" middle_len="${ring_middle_len}" useMimicTag="${useMimicTag}" abd_R="${ring_abd_R}" inner_R="${ring_inner_R *(inner_ub - inner_lb)*pi/180}" middle_R="${ring_middle_R *(middle_ub - middle_lb)*pi/180}" outer_R="${ring_outer_R *(outer_ub - outer_lb)*pi/180}" />
+		<xacro:finger parent="${name}_palm_link" parent_name="${name}" prefix="${name}_" name="little" reflect="${reflect}" position="${-0.04175*reflect} -0.003 0.079" orientation="0 0 0" proximal_len="${little_proximal_len}" middle_len="${little_middle_len}" useMimicTag="${useMimicTag}" abd_R="${little_abd_R}" inner_R="${little_inner_R *(inner_ub - inner_lb)*pi/180}" middle_R="${little_middle_R *(middle_ub - middle_lb)*pi/180}" outer_R="${little_outer_R *(outer_ub - outer_lb)*pi/180}" />
+		<xacro:include filename="$(find human_hand_description)/model/${tactile_mapping}.mapping.xacro"/>
+		<xacro:include filename="$(find human_hand_description)/model/${_tactileMappingToLayout[tactile_mapping]}.urdf.xacro"/>
+		<xacro:tactile_glove name="${name}" reflect="${reflect}"/>
 	</xacro:macro>
 </robot>

Commit message: use yaml for tactile mapping (with new xacro)

File: model/P2.urdf.xacro (robot description, xacro)
@@ -12,5 +12,5 @@
 		</xacro:if>
 	</xacro:macro>
-	<xacro:macro name="tactile_glove" params="name reflect:=1">
+	<xacro:macro name="tactile_glove" params="name reflect:=1 tactMap">
 		<xacro:property name="_name" value="${name}_"/>
 		<xacro:property name="_reflect" value="${reflect}"/>

File: model/P3.urdf.xacro (robot description, xacro)
@@ -12,5 +12,5 @@
 		</xacro:if>
 	</xacro:macro>
-	<xacro:macro name="tactile_glove" params="name reflect:=1">
+	<xacro:macro name="tactile_glove" params="name reflect:=1 tactMap">
 		<xacro:property name="_name" value="${name}_"/>
 		<xacro:property name="_reflect" value="${reflect}"/>

File: model/human_hand.urdf.xacro (robot description, xacro)
@@ -9,5 +9,5 @@
 	-->
 	<xacro:include filename="$(find human_hand_description)/model/materials.urdf.xacro"/>
-	<xacro:property name="_tactileMappingToLayout" value="{'P2':'P2', 'P3l':'P3', 'P3r':'P3'}"/>
+	<xacro:property name="_tactileMappingToLayout" value="${dict(P2='P2', P3l='P3', P3r='P3')}"/>
 	<!-- joint properties -->
 	<xacro:property name="abd_lb" value="-30" />
@@ -262,7 +262,7 @@
 		<xacro:finger parent="${name}_palm_link" parent_name="${name}" prefix="${name}_" name="ring" reflect="${reflect}" position="${-0.02225*reflect} 0.0010 0.090" orientation="0 0 0" proximal_len="${ring_proximal_len}" middle_len="${ring_middle_len}" useMimicTag="${useMimicTag}" abd_R="${ring_abd_R}" inner_R="${ring_inner_R *(inner_ub - inner_lb)*pi/180}" middle_R="${ring_middle_R *(middle_ub - middle_lb)*pi/180}" outer_R="${ring_outer_R *(outer_ub - outer_lb)*pi/180}" />
 		<xacro:finger parent="${name}_palm_link" parent_name="${name}" prefix="${name}_" name="little" reflect="${reflect}" position="${-0.04175*reflect} -0.003 0.079" orientation="0 0 0" proximal_len="${little_proximal_len}" middle_len="${little_middle_len}" useMimicTag="${useMimicTag}" abd_R="${little_abd_R}" inner_R="${little_inner_R *(inner_ub - inner_lb)*pi/180}" middle_R="${little_middle_R *(middle_ub - middle_lb)*pi/180}" outer_R="${little_outer_R *(outer_ub - outer_lb)*pi/180}" />
-		<xacro:include filename="$(find human_hand_description)/model/${tactile_mapping}.mapping.xacro"/>
+		<xacro:property name="tactile_mapping_file" value="../model/${tactile_mapping}.mapping.yaml"/>
 		<xacro:include filename="$(find human_hand_description)/model/${_tactileMappingToLayout[tactile_mapping]}.urdf.xacro"/>
-		<xacro:tactile_glove name="${name}" reflect="${reflect}"/>
+		<xacro:tactile_glove name="${name}" reflect="${reflect}" tactMap="${load_yaml(tactile_mapping_file)}"/>
 	</xacro:macro>
 </robot>
