Commit message: moved joint properties into yaml

File: robots/twohands.urdf.xacro (robot description, xacro)
@@ -2,12 +2,14 @@
 <robot xmlns:xacro="http://www.ros.org/wiki/xacro" name="human_hand">
 	<xacro:arg name="use_mimic_tag" default="false"/>
-	<xacro:arg name="tactile_mapping" default="P3"/>
-	<xacro:property name="tactile_mapping" value="$(arg tactile_mapping)"/>
-	<xacro:include filename="$(find human_hand_description)/model/human_hand.urdf.xacro"/>
+	<xacro:include filename="../model/human_hand.urdf.xacro"/>
 	<link name="world"/>
-	<xacro:human_hand parent="world" name="right_hand" left="false" useMimicTag="$(arg use_mimic_tag)" >
+	<xacro:human_hand parent="world" prefix="right_" side="right"
+	                  useMimicTag="$(arg use_mimic_tag)"
+	                  tactile_mapping="">
 		<origin xyz="+0.06 0.0 0" rpy="0 0 0"/>
 	</xacro:human_hand>
-	<xacro:human_hand parent="world" name="left_hand" left="true" useMimicTag="$(arg use_mimic_tag)" >
+	<xacro:human_hand parent="world" prefix="left_" side="left"
+	                  useMimicTag="$(arg use_mimic_tag)"
+	                  tactile_mapping="">
 		<origin xyz="-0.06 0 0" rpy="0 0 0"/>
 	</xacro:human_hand>

Commit message: adapted thumb definition to be more similar to finger's definition

File: model/P1.urdf.xacro (robot description, xacro)
@@ -65,15 +65,15 @@
 		<xacro:taxel ns="palm" link="palm_link" mesh="ptip" channel="${tactMap.get('ptip', -1)}" offset="0 -1e-3 0"/>
 		<xacro:taxel ns="palm" link="palm_link" mesh="ptid" channel="${tactMap.get('ptid', -1)}" offset="0 -1e-3 0"/>
-		<xacro:taxel ns="thumb" link="thumb_knuckle_link" mesh="ptmp2" channel="${tactMap.get('ptop', -1)}" offset="0 -1e-3 0"/>
-		<xacro:taxel ns="thumb" link="thumb_knuckle_link" mesh="ptmd2" channel="${tactMap.get('ptod', -1)}" offset="0 -1e-3 0"/>
-		<xacro:taxel ns="thumb" link="thumb_knuckle_link" mesh="ptip2" channel="${tactMap.get('ptip', -1)}" offset="0 -1e-3 0"/>
-		<xacro:taxel ns="thumb" link="thumb_knuckle_link" mesh="ptid2" channel="${tactMap.get('ptid', -1)}" offset="0 -1e-3 0"/>
+		<xacro:taxel ns="thumb" link="thumb_proximal_link" mesh="ptmp2" channel="${tactMap.get('ptop', -1)}" offset="0 -1e-3 0"/>
+		<xacro:taxel ns="thumb" link="thumb_proximal_link" mesh="ptmd2" channel="${tactMap.get('ptod', -1)}" offset="0 -1e-3 0"/>
+		<xacro:taxel ns="thumb" link="thumb_proximal_link" mesh="ptip2" channel="${tactMap.get('ptip', -1)}" offset="0 -1e-3 0"/>
+		<xacro:taxel ns="thumb" link="thumb_proximal_link" mesh="ptid2" channel="${tactMap.get('ptid', -1)}" offset="0 -1e-3 0"/>
 		<xacro:taxel ns="thumb" link="thumb_distal_link" mesh="tdd" channel="${tactMap.get('tdd', -1)}" offset="0 0 1e-3"/>
 		<xacro:taxel ns="thumb" link="thumb_distal_link" mesh="tdo" channel="${tactMap.get('tdo', -1)}" offset="0 1e-3 0"/>
 		<xacro:taxel ns="thumb" link="thumb_distal_link" mesh="tdm" channel="${tactMap.get('tdm', -1)}" offset="${-1e-3*reflect} 0 0"/>
 		<xacro:taxel ns="thumb" link="thumb_distal_link" mesh="tdi" channel="${tactMap.get('tdi', -1)}" offset="0 -1e-3 0"/>
-		<xacro:taxel ns="thumb" link="thumb_proximal_link" mesh="tpo" channel="${tactMap.get('tpo', -1)}" offset="0 1e-3 0"/>
-		<xacro:taxel ns="thumb" link="thumb_proximal_link" mesh="tpm" channel="${tactMap.get('tpm', -1)}" offset="${-1e-3*reflect} 0 0"/>
-		<xacro:taxel ns="thumb" link="thumb_proximal_link" mesh="tpi" channel="${tactMap.get('tpi', -1)}" offset="0 -1e-3 0"/>
+		<xacro:taxel ns="thumb" link="thumb_middle_link" mesh="tpo" channel="${tactMap.get('tpo', -1)}" offset="0 1e-3 0"/>
+		<xacro:taxel ns="thumb" link="thumb_middle_link" mesh="tpm" channel="${tactMap.get('tpm', -1)}" offset="${-1e-3*reflect} 0 0"/>
+		<xacro:taxel ns="thumb" link="thumb_middle_link" mesh="tpi" channel="${tactMap.get('tpi', -1)}" offset="0 -1e-3 0"/>
 	</xacro:macro>
 </robot>

File: model/P3.urdf.xacro (robot description, xacro)
@@ -66,15 +66,15 @@
 		<xacro:taxel ns="palm" link="palm_link" mesh="ptip" channel="${tactMap.get('ptip', -1)}" offset="0 -1e-3 0"/>
 		<xacro:taxel ns="palm" link="palm_link" mesh="ptid" channel="${tactMap.get('ptid', -1)}" offset="0 -1e-3 0"/>
-		<xacro:taxel ns="thumb" link="thumb_knuckle_link" mesh="ptmp2" channel="${tactMap.get('ptmp', -1)}" offset="0 -1e-3 0"/>
-		<xacro:taxel ns="thumb" link="thumb_knuckle_link" mesh="ptmd2" channel="${tactMap.get('ptmd', -1)}" offset="0 -1e-3 0"/>
-		<xacro:taxel ns="thumb" link="thumb_knuckle_link" mesh="ptip2" channel="${tactMap.get('ptip', -1)}" offset="0 -1e-3 0"/>
-		<xacro:taxel ns="thumb" link="thumb_knuckle_link" mesh="ptid2" channel="${tactMap.get('ptid', -1)}" offset="0 -1e-3 0"/>
+		<xacro:taxel ns="thumb" link="thumb_proximal_link" mesh="ptmp2" channel="${tactMap.get('ptmp', -1)}" offset="0 -1e-3 0"/>
+		<xacro:taxel ns="thumb" link="thumb_proximal_link" mesh="ptmd2" channel="${tactMap.get('ptmd', -1)}" offset="0 -1e-3 0"/>
+		<xacro:taxel ns="thumb" link="thumb_proximal_link" mesh="ptip2" channel="${tactMap.get('ptip', -1)}" offset="0 -1e-3 0"/>
+		<xacro:taxel ns="thumb" link="thumb_proximal_link" mesh="ptid2" channel="${tactMap.get('ptid', -1)}" offset="0 -1e-3 0"/>
 		<xacro:taxel ns="thumb" link="thumb_distal_link" mesh="tdd" channel="${tactMap.get('tdd', -1)}" offset="0 0 1e-3"/>
 		<xacro:taxel ns="thumb" link="thumb_distal_link" mesh="tdo" channel="${tactMap.get('tdo', -1)}" offset="0 1e-3 0"/>
 		<xacro:taxel ns="thumb" link="thumb_distal_link" mesh="tdm" channel="${tactMap.get('tdm', -1)}" offset="${-1e-3*reflect} 0 0"/>
 		<xacro:taxel ns="thumb" link="thumb_distal_link" mesh="tdi" channel="${tactMap.get('tdi', -1)}" offset="0 -1e-3 0"/>
-		<xacro:taxel ns="thumb" link="thumb_proximal_link" mesh="tpo" channel="${tactMap.get('tpo', -1)}" offset="0 1e-3 0"/>
-		<xacro:taxel ns="thumb" link="thumb_proximal_link" mesh="tpm" channel="${tactMap.get('tpm', -1)}" offset="${-1e-3*reflect} 0 0"/>
-		<xacro:taxel ns="thumb" link="thumb_proximal_link" mesh="tpi" channel="${tactMap.get('tpi', -1)}" offset="0 -1e-3 0"/>
+		<xacro:taxel ns="thumb" link="thumb_middle_link" mesh="tpo" channel="${tactMap.get('tpo', -1)}" offset="0 1e-3 0"/>
+		<xacro:taxel ns="thumb" link="thumb_middle_link" mesh="tpm" channel="${tactMap.get('tpm', -1)}" offset="${-1e-3*reflect} 0 0"/>
+		<xacro:taxel ns="thumb" link="thumb_middle_link" mesh="tpi" channel="${tactMap.get('tpi', -1)}" offset="0 -1e-3 0"/>
 	</xacro:macro>
 </robot>

File: model/human_hand.urdf.xacro (robot description, xacro)
@@ -24,5 +24,5 @@
 			<xacro:if value="${use_synergy}">
 				<xacro:if value="${synergy_weight is None}">
-					<xacro:property name="synergy_weight" value="${synergies[finger+'_'+joint]}"/>
+					<xacro:property name="synergy_weight" value="${synergies[finger][joint]}"/>
 				</xacro:if>
 				<mimic joint="${synergy_joint}"
@@ -49,6 +49,6 @@
 	             params="parent prefix:=$ finger reflect:=$ *origin
 	                     joint_props:=${properties['joints']}">
-		<xacro:property name="proximal_len" value="${properties['link_lengths'][finger+'_proximal']}"/>
-		<xacro:property name="middle_len" value="${properties['link_lengths'][finger+'_middle']}"/>
+		<xacro:property name="proximal_len" value="${properties['link_lengths'][finger]['proximal']}"/>
+		<xacro:property name="middle_len" value="${properties['link_lengths'][finger]['middle']}"/>
 		<!-- KNUCKLE -->
 		<xacro:segment joint="abduction" link="knuckle" parent="${parent}" mesh="0">
@@ -72,28 +72,29 @@
 		</xacro:segment>
 	</xacro:macro>
-	<!-- THUMB MODEL (thumb has one link less than fingers -->
+	<!-- THUMB MODEL -->
 	<xacro:macro name="thumb"
 	             params="parent prefix:=$ finger:='thumb' reflect:=$ *origin
 	                     joint_props:=${properties['joints']}">
-		<xacro:property name="base_len" value="${properties['link_lengths'][finger+'_base']}"/>
-		<xacro:property name="proximal_len" value="${properties['link_lengths'][finger+'_proximal']}"/>
+		<xacro:property name="proximal_len" value="${properties['link_lengths'][finger]['proximal']}"/>
+		<xacro:property name="middle_len" value="${properties['link_lengths'][finger]['middle']}"/>
 		<!-- KNUCKLE -->
-		<xacro:segment joint="abduction" link="fake" parent="${parent}" mesh="False">
+		<xacro:segment joint="abduction" link="knuckle" parent="${parent}"
+		               mesh="False" use_synergy="0">
 			<xacro:insert_block name="origin"/>
 			<axis xyz="1 0 0" />
 		</xacro:segment>
-		<xacro:segment joint="rotate" link="knuckle" parent="${prefix}${finger}_fake_link"
-		             mesh="thumb_base" use_synergy="0">
+		<!-- PROXIMAL PHALANGE -->
+		<xacro:segment joint="proximal" link="proximal" parent="${prefix}${finger}_knuckle_link">
 			<origin xyz="0 0 0" rpy="0 0 0" />
 			<axis xyz="0 ${-1*reflect} 0" />
 		</xacro:segment>
-		<!-- PROXIMAL PHALANGE -->
-		<xacro:segment joint="proximal" link="proximal" parent="${prefix}${finger}_knuckle_link">
-			<origin xyz="0 0 ${base_len}" rpy="0 0 0"/>
+		<!-- MIDDLE PHALANGE -->
+		<xacro:segment joint="middle" link="middle" parent="${prefix}${finger}_proximal_link">
+			<origin xyz="0 0 ${proximal_len}" rpy="0 0 0"/>
 			<axis xyz="0 ${-1*reflect} 0" />
 		</xacro:segment>
 		<!-- DISTAL PHALANGE -->
-		<xacro:segment joint="distal" link="distal" parent="${prefix}${finger}_proximal_link">
-			<origin xyz="0 0 ${proximal_len}" rpy="0 0 0"/>
+		<xacro:segment joint="distal" link="distal" parent="${prefix}${finger}_middle_link">
+			<origin xyz="0 0 ${middle_len}" rpy="0 0 0"/>
 			<axis xyz="0 ${-1*reflect} 0" />
 		</xacro:segment>

Commit message: switched '$|' syntax to '^|' syntax for arg forwarding

File: model/P1.urdf.xacro (robot description, xacro)
@@ -1,5 +1,5 @@
 <?xml version="1.0"?>
 <robot name="tactile_glove_markers" xmlns:xacro="http://www.ros.org/wiki/xacro">
-	<xacro:macro name="taxel" params="prefix:=$ channel link mesh offset ns">
+	<xacro:macro name="taxel" params="prefix:=^ channel link mesh offset ns">
 		<xacro:if value="${channel >= 0}">
 		<tactile topic="TactileGlove" data="data[${channel}]" link="${prefix}${link}" ns="${ns}" xs="0 4095">

File: model/P3.urdf.xacro (robot description, xacro)
@@ -1,5 +1,5 @@
 <?xml version="1.0"?>
 <robot name="tactile_glove_markers" xmlns:xacro="http://www.ros.org/wiki/xacro">
-	<xacro:macro name="taxel" params="prefix:=$ channel link mesh offset ns">
+	<xacro:macro name="taxel" params="prefix:=^ channel link mesh offset ns">
 		<xacro:if value="${channel >= 0}">
 			<tactile topic="TactileGlove" data="data[${channel}]" link="${prefix}${link}" ns="${ns}" xs="0 4095">

File: model/human_hand.urdf.xacro (robot description, xacro)
@@ -11,6 +11,6 @@
 	<!-- a segment is composed of a joint and the attached link -->
 	<xacro:macro name="xacro:segment"
-	             params="prefix:=$|'' finger:=$ joint link parent reflect:=$ *origin *axis
-	                     synergy_weight:=None mesh:=1 use_synergy:=$">
+	             params="prefix:=^|'' finger:=^ joint link parent reflect:=^ *origin *axis
+	                     synergy_weight:=None mesh:=1 use_synergy:=^">
 		<xacro:property name="props" value="${joint_props[finger][joint]}"/>
 		<joint name="${prefix}${finger}_${joint}_joint" type="revolute">
@@ -47,5 +47,5 @@
 	<!-- FINGER MODEL -->
 	<xacro:macro name="finger"
-	             params="parent prefix:=$ finger reflect:=$ *origin
+	             params="parent prefix:=^ finger reflect:=^ *origin
 	                     joint_props:=${properties['joints']}">
 		<xacro:property name="proximal_len" value="${properties['link_lengths'][finger]['proximal']}"/>
@@ -74,5 +74,5 @@
 	<!-- THUMB MODEL -->
 	<xacro:macro name="thumb"
-	             params="parent prefix:=$ finger:='thumb' reflect:=$ *origin
+	             params="parent prefix:=^ finger:='thumb' reflect:=^ *origin
 	                     joint_props:=${properties['joints']}">
 		<xacro:property name="proximal_len" value="${properties['link_lengths'][finger]['proximal']}"/>
