Commit message: removed obsolete offsets

File: model/L1.urdf.xacro (robot description, xacro)
@@ -1,5 +1,5 @@
 <?xml version="1.0"?>
 <robot name="tactile_glove_markers" xmlns:xacro="http://www.ros.org/wiki/xacro">
-	<xacro:macro name="taxel" params="prefix:=^ mesh idx offset">
+	<xacro:macro name="taxel" params="prefix:=^ mesh idx">
 		<xacro:if value="${idx >= 0}">
 			<taxel idx="${idx}">
@@ -16,8 +16,8 @@
 			<parent link="${finger}_distal_link"/>
 			<tactile channel="tactile">
-				<xacro:taxel mesh="${F}dd" idx="${tactMap.get(F+'dd', -1)}" offset="0 0 1e-3"/>
-				<xacro:taxel mesh="${F}do" idx="${tactMap.get(F+'do', -1)}" offset="${-1e-3*reflect} 0 0"/>
-				<xacro:taxel mesh="${F}dm" idx="${tactMap.get(F+'dm', -1)}" offset="0 -1e-3 0"/>
-				<xacro:taxel mesh="${F}di" idx="${tactMap.get(F+'di', -1)}" offset="${1e-3*reflect} 0 0"/>
+				<xacro:taxel mesh="${F}dd" idx="${tactMap.get(F+'dd', -1)}"/>
+				<xacro:taxel mesh="${F}do" idx="${tactMap.get(F+'do', -1)}"/>
+				<xacro:taxel mesh="${F}dm" idx="${tactMap.get(F+'dm', -1)}"/>
+				<xacro:taxel mesh="${F}di" idx="${tactMap.get(F+'di', -1)}"/>
 			</tactile>
 		</sensor>
@@ -25,7 +25,7 @@
 			<parent link="${finger}_middle_link"/>
 			<tactile channel="tactile">
-				<xacro:taxel mesh="${F}mo" idx="${tactMap.get(F+'mo', -1)}" offset="${-1e-3*reflect} 0 0"/>
-				<xacro:taxel mesh="${F}mm" idx="${tactMap.get(F+'mm', -1)}" offset="0 -1e-3 0"/>
-				<xacro:taxel mesh="${F}mi" idx="${tactMap.get(F+'mi', -1)}" offset="${1e-3*reflect} 0 0"/>
+				<xacro:taxel mesh="${F}mo" idx="${tactMap.get(F+'mo', -1)}"/>
+				<xacro:taxel mesh="${F}mm" idx="${tactMap.get(F+'mm', -1)}"/>
+				<xacro:taxel mesh="${F}mi" idx="${tactMap.get(F+'mi', -1)}"/>
 			</tactile>
 		</sensor>
@@ -33,7 +33,7 @@
 			<parent link="${finger}_proximal_link"/>
 			<tactile channel="tactile">
-				<xacro:taxel mesh="${F}p" idx="${tactMap.get(F+'p', -1)}" offset="0 -1e-3 0"/>
-				<xacro:taxel mesh="${F}pi" idx="${tactMap.get(F+'pi', -1)}" offset="${1e-3*reflect} 0 0"/>
-				<xacro:taxel mesh="${F}po" idx="${tactMap.get(F+'po', -1)}" offset="${-1e-3*reflect} 0 0"/>
+				<xacro:taxel mesh="${F}p" idx="${tactMap.get(F+'p', -1)}"/>
+				<xacro:taxel mesh="${F}pi" idx="${tactMap.get(F+'pi', -1)}"/>
+				<xacro:taxel mesh="${F}po" idx="${tactMap.get(F+'po', -1)}"/>
 			</tactile>
 		</sensor>
@@ -48,8 +48,8 @@
 			<parent link="${prefix}thumb_proximal_link"/>
 			<tactile channel="tactile">
-				<xacro:taxel mesh="ptmp2" idx="${tactMap.get('ptop', -1)}" offset="0 -1e-3 0"/>
-				<xacro:taxel mesh="ptmd2" idx="${tactMap.get('ptod', -1)}" offset="0 -1e-3 0"/>
-				<xacro:taxel mesh="ptip2" idx="${tactMap.get('ptip', -1)}" offset="0 -1e-3 0"/>
-				<xacro:taxel mesh="ptid2" idx="${tactMap.get('ptid', -1)}" offset="0 -1e-3 0"/>
+				<xacro:taxel mesh="ptmp2" idx="${tactMap.get('ptop', -1)}"/>
+				<xacro:taxel mesh="ptmd2" idx="${tactMap.get('ptod', -1)}"/>
+				<xacro:taxel mesh="ptip2" idx="${tactMap.get('ptip', -1)}"/>
+				<xacro:taxel mesh="ptid2" idx="${tactMap.get('ptid', -1)}"/>
 			</tactile>
 		</sensor>
@@ -57,22 +57,22 @@
 			<parent link="${prefix}palm_link"/>
 			<tactile channel="tactile">
-				<xacro:taxel mesh="pdlo" idx="${tactMap.get('po', -1)}" offset="0 -1e-3 0"/>
-				<xacro:taxel mesh="pdl" idx="${tactMap.get('pdl', -1)}" offset="0 -1e-3 0"/>
-				<xacro:taxel mesh="pdr" idx="${tactMap.get('pdr', -1)}" offset="0 -1e-3 0"/>
-				<xacro:taxel mesh="pdm" idx="${tactMap.get('pdm', -1)}" offset="0 -1e-3 0"/>
-				<xacro:taxel mesh="pdi" idx="${tactMap.get('pdi', -1)}" offset="0 -1e-3 0"/>
-				<xacro:taxel mesh="pdii" idx="${tactMap.get('pdii', -1)}" offset="0 -1e-3 0"/>
-				<xacro:taxel mesh="pco" idx="${tactMap.get('po', -1)}" offset="0 -1e-3 0"/>
-				<xacro:taxel mesh="pcmp" idx="${tactMap.get('pcmp', -1)}" offset="0 -1e-3 0"/>
-				<xacro:taxel mesh="pcmd" idx="${tactMap.get('pcmd', -1)}" offset="0 -1e-3 0"/>
-				<xacro:taxel mesh="pcip" idx="${tactMap.get('pcip', -1)}" offset="0 -1e-3 0"/>
-				<xacro:taxel mesh="pcim" idx="${tactMap.get('pcim', -1)}" offset="0 -1e-3 0"/>
-				<xacro:taxel mesh="pcid" idx="${tactMap.get('pcid', -1)}" offset="0 -1e-3 0"/>
-				<xacro:taxel mesh="ptop" idx="${tactMap.get('ptop', -1)}" offset="0 -1e-3 0"/>
-				<xacro:taxel mesh="ptod" idx="${tactMap.get('ptod', -1)}" offset="0 -1e-3 0"/>
-				<xacro:taxel mesh="ptmp" idx="${tactMap.get('ptop', -1)}" offset="0 -1e-3 0"/>
-				<xacro:taxel mesh="ptmd" idx="${tactMap.get('ptod', -1)}" offset="0 -1e-3 0"/>
-				<xacro:taxel mesh="ptip" idx="${tactMap.get('ptip', -1)}" offset="0 -1e-3 0"/>
-				<xacro:taxel mesh="ptid" idx="${tactMap.get('ptid', -1)}" offset="0 -1e-3 0"/>
+				<xacro:taxel mesh="pdlo" idx="${tactMap.get('po', -1)}"/>
+				<xacro:taxel mesh="pdl" idx="${tactMap.get('pdl', -1)}"/>
+				<xacro:taxel mesh="pdr" idx="${tactMap.get('pdr', -1)}"/>
+				<xacro:taxel mesh="pdm" idx="${tactMap.get('pdm', -1)}"/>
+				<xacro:taxel mesh="pdi" idx="${tactMap.get('pdi', -1)}"/>
+				<xacro:taxel mesh="pdii" idx="${tactMap.get('pdii', -1)}"/>
+				<xacro:taxel mesh="pco" idx="${tactMap.get('po', -1)}"/>
+				<xacro:taxel mesh="pcmp" idx="${tactMap.get('pcmp', -1)}"/>
+				<xacro:taxel mesh="pcmd" idx="${tactMap.get('pcmd', -1)}"/>
+				<xacro:taxel mesh="pcip" idx="${tactMap.get('pcip', -1)}"/>
+				<xacro:taxel mesh="pcim" idx="${tactMap.get('pcim', -1)}"/>
+				<xacro:taxel mesh="pcid" idx="${tactMap.get('pcid', -1)}"/>
+				<xacro:taxel mesh="ptop" idx="${tactMap.get('ptop', -1)}"/>
+				<xacro:taxel mesh="ptod" idx="${tactMap.get('ptod', -1)}"/>
+				<xacro:taxel mesh="ptmp" idx="${tactMap.get('ptop', -1)}"/>
+				<xacro:taxel mesh="ptmd" idx="${tactMap.get('ptod', -1)}"/>
+				<xacro:taxel mesh="ptip" idx="${tactMap.get('ptip', -1)}"/>
+				<xacro:taxel mesh="ptid" idx="${tactMap.get('ptid', -1)}"/>
 			</tactile>
 		</sensor>

File: model/L2.urdf.xacro (robot description, xacro)
@@ -1,5 +1,5 @@
 <?xml version="1.0"?>
 <robot name="tactile_glove_markers" xmlns:xacro="http://www.ros.org/wiki/xacro">
-	<xacro:macro name="taxel" params="prefix:=^ mesh idx offset">
+	<xacro:macro name="taxel" params="prefix:=^ mesh idx">
 		<xacro:if value="${idx >= 0}">
 			<taxel idx="${idx}">
@@ -16,8 +16,8 @@
 			<parent link="${finger}_distal_link"/>
 			<tactile channel="tactile">
-				<xacro:taxel mesh="${F}dd" idx="${tactMap.get(F+'dd', -1)}" offset="0 0 1e-3"/>
-				<xacro:taxel mesh="${F}do" idx="${tactMap.get(F+'do', -1)}" offset="${-1e-3*reflect} 0 0"/>
-				<xacro:taxel mesh="${F}dm" idx="${tactMap.get(F+'dm', -1)}" offset="0 -1e-3 0"/>
-				<xacro:taxel mesh="${F}di" idx="${tactMap.get(F+'di', -1)}" offset="${1e-3*reflect} 0 0"/>
+				<xacro:taxel mesh="${F}dd" idx="${tactMap.get(F+'dd', -1)}"/>
+				<xacro:taxel mesh="${F}do" idx="${tactMap.get(F+'do', -1)}"/>
+				<xacro:taxel mesh="${F}dm" idx="${tactMap.get(F+'dm', -1)}"/>
+				<xacro:taxel mesh="${F}di" idx="${tactMap.get(F+'di', -1)}"/>
 			</tactile>
 		</sensor>
@@ -25,7 +25,7 @@
 			<parent link="${finger}_middle_link"/>
 			<tactile channel="tactile">
-				<xacro:taxel mesh="${F}mo" idx="${tactMap.get(F+'mo', -1)}" offset="${-1e-3*reflect} 0 0"/>
-				<xacro:taxel mesh="${F}mm" idx="${tactMap.get(F+'mm', -1)}" offset="0 -1e-3 0"/>
-				<xacro:taxel mesh="${F}mi" idx="${tactMap.get(F+'mi', -1)}" offset="${1e-3*reflect} 0 0"/>
+				<xacro:taxel mesh="${F}mo" idx="${tactMap.get(F+'mo', -1)}"/>
+				<xacro:taxel mesh="${F}mm" idx="${tactMap.get(F+'mm', -1)}"/>
+				<xacro:taxel mesh="${F}mi" idx="${tactMap.get(F+'mi', -1)}"/>
 			</tactile>
 		</sensor>
@@ -33,7 +33,7 @@
 			<parent link="${finger}_proximal_link"/>
 			<tactile channel="tactile">
-				<xacro:taxel mesh="${F}p" idx="${tactMap.get(F+'p', -1)}" offset="0 -1e-3 0"/>
-				<xacro:taxel mesh="${F}pi" idx="${tactMap.get(F+'pi', -1)}" offset="${1e-3*reflect} 0 0"/>
-				<xacro:taxel mesh="${F}po" idx="${tactMap.get(F+'po', -1)}" offset="${-1e-3*reflect} 0 0"/>
+				<xacro:taxel mesh="${F}p" idx="${tactMap.get(F+'p', -1)}"/>
+				<xacro:taxel mesh="${F}pi" idx="${tactMap.get(F+'pi', -1)}"/>
+				<xacro:taxel mesh="${F}po" idx="${tactMap.get(F+'po', -1)}"/>
 			</tactile>
 		</sensor>
@@ -48,8 +48,8 @@
 			<parent link="${prefix}thumb_proximal_link"/>
 			<tactile channel="tactile">
-				<xacro:taxel mesh="ptmp2" idx="${tactMap.get('ptmp', -1)}" offset="0 -1e-3 0"/>
-				<xacro:taxel mesh="ptmd2" idx="${tactMap.get('ptmd', -1)}" offset="0 -1e-3 0"/>
-				<xacro:taxel mesh="ptip2" idx="${tactMap.get('ptip', -1)}" offset="0 -1e-3 0"/>
-				<xacro:taxel mesh="ptid2" idx="${tactMap.get('ptid', -1)}" offset="0 -1e-3 0"/>
+				<xacro:taxel mesh="ptmp2" idx="${tactMap.get('ptmp', -1)}"/>
+				<xacro:taxel mesh="ptmd2" idx="${tactMap.get('ptmd', -1)}"/>
+				<xacro:taxel mesh="ptip2" idx="${tactMap.get('ptip', -1)}"/>
+				<xacro:taxel mesh="ptid2" idx="${tactMap.get('ptid', -1)}"/>
 			</tactile>
 		</sensor>
@@ -57,23 +57,23 @@
 			<parent link="${prefix}palm_link"/>
 			<tactile channel="tactile">
-				<xacro:taxel mesh="pdlo" idx="${tactMap.get('pdlo', -1)}" offset="0 -1e-3 0"/>
-				<xacro:taxel mesh="pdl" idx="${tactMap.get('pdl', -1)}" offset="0 -1e-3 0"/>
-				<xacro:taxel mesh="pdr" idx="${tactMap.get('pdr', -1)}" offset="0 -1e-3 0"/>
-				<xacro:taxel mesh="pdm" idx="${tactMap.get('pdm', -1)}" offset="0 -1e-3 0"/>
-				<xacro:taxel mesh="pdi" idx="${tactMap.get('pdi', -1)}" offset="0 -1e-3 0"/>
-				<xacro:taxel mesh="pdii" idx="${tactMap.get('pdii', -1)}" offset="0 -1e-3 0"/>
-				<xacro:taxel mesh="pco" idx="${tactMap.get('pco', -1)}" offset="0 -1e-3 0"/>
-				<xacro:taxel mesh="pcmp" idx="${tactMap.get('pcmp', -1)}" offset="0 -1e-3 0"/>
-				<xacro:taxel mesh="pcmd" idx="${tactMap.get('pcmd', -1)}" offset="0 -1e-3 0"/>
-				<xacro:taxel mesh="pcip" idx="${tactMap.get('pcip', -1)}" offset="0 -1e-3 0"/>
-				<xacro:taxel mesh="pcim" idx="${tactMap.get('pcim', -1)}" offset="0 -1e-3 0"/>
-				<xacro:taxel mesh="pcid" idx="${tactMap.get('pcid', -1)}" offset="0 -1e-3 0"/>
-				<xacro:taxel mesh="pi" idx="${tactMap.get('pi', -1)}" offset="0 -1e-3 0"/>
-				<xacro:taxel mesh="ptop" idx="${tactMap.get('ptop', -1)}" offset="0 -1e-3 0"/>
-				<xacro:taxel mesh="ptod" idx="${tactMap.get('ptod', -1)}" offset="0 -1e-3 0"/>
-				<xacro:taxel mesh="ptmp" idx="${tactMap.get('ptmp', -1)}" offset="0 -1e-3 0"/>
-				<xacro:taxel mesh="ptmd" idx="${tactMap.get('ptmd', -1)}" offset="0 -1e-3 0"/>
-				<xacro:taxel mesh="ptip" idx="${tactMap.get('ptip', -1)}" offset="0 -1e-3 0"/>
-				<xacro:taxel mesh="ptid" idx="${tactMap.get('ptid', -1)}" offset="0 -1e-3 0"/>
+				<xacro:taxel mesh="pdlo" idx="${tactMap.get('pdlo', -1)}"/>
+				<xacro:taxel mesh="pdl" idx="${tactMap.get('pdl', -1)}"/>
+				<xacro:taxel mesh="pdr" idx="${tactMap.get('pdr', -1)}"/>
+				<xacro:taxel mesh="pdm" idx="${tactMap.get('pdm', -1)}"/>
+				<xacro:taxel mesh="pdi" idx="${tactMap.get('pdi', -1)}"/>
+				<xacro:taxel mesh="pdii" idx="${tactMap.get('pdii', -1)}"/>
+				<xacro:taxel mesh="pco" idx="${tactMap.get('pco', -1)}"/>
+				<xacro:taxel mesh="pcmp" idx="${tactMap.get('pcmp', -1)}"/>
+				<xacro:taxel mesh="pcmd" idx="${tactMap.get('pcmd', -1)}"/>
+				<xacro:taxel mesh="pcip" idx="${tactMap.get('pcip', -1)}"/>
+				<xacro:taxel mesh="pcim" idx="${tactMap.get('pcim', -1)}"/>
+				<xacro:taxel mesh="pcid" idx="${tactMap.get('pcid', -1)}"/>
+				<xacro:taxel mesh="pi" idx="${tactMap.get('pi', -1)}"/>
+				<xacro:taxel mesh="ptop" idx="${tactMap.get('ptop', -1)}"/>
+				<xacro:taxel mesh="ptod" idx="${tactMap.get('ptod', -1)}"/>
+				<xacro:taxel mesh="ptmp" idx="${tactMap.get('ptmp', -1)}"/>
+				<xacro:taxel mesh="ptmd" idx="${tactMap.get('ptmd', -1)}"/>
+				<xacro:taxel mesh="ptip" idx="${tactMap.get('ptip', -1)}"/>
+				<xacro:taxel mesh="ptid" idx="${tactMap.get('ptid', -1)}"/>
 			</tactile>
 		</sensor>

File: model/L3.urdf.xacro (robot description, xacro)
@@ -1,5 +1,5 @@
 <?xml version="1.0"?>
 <robot name="tactile_glove_markers" xmlns:xacro="http://www.ros.org/wiki/xacro">
-	<xacro:macro name="taxel" params="prefix:=^ mesh idx offset">
+	<xacro:macro name="taxel" params="prefix:=^ mesh idx">
 		<xacro:if value="${idx >= 0}">
 			<taxel idx="${idx}">
@@ -16,8 +16,8 @@
 			<parent link="${finger}_distal_link"/>
 			<tactile channel="tactile">
-				<xacro:taxel mesh="${F}dd" idx="${tactMap.get(F+'dd', -1)}" offset="0 0 1e-3"/>
-				<xacro:taxel mesh="${F}do" idx="${tactMap.get(F+'do', -1)}" offset="${-1e-3*reflect} 0 0"/>
-				<xacro:taxel mesh="${F}dm" idx="${tactMap.get(F+'dm', -1)}" offset="0 -1e-3 0"/>
-				<xacro:taxel mesh="${F}di" idx="${tactMap.get(F+'di', -1)}" offset="${1e-3*reflect} 0 0"/>
+				<xacro:taxel mesh="${F}dd" idx="${tactMap.get(F+'dd', -1)}"/>
+				<xacro:taxel mesh="${F}do" idx="${tactMap.get(F+'do', -1)}"/>
+				<xacro:taxel mesh="${F}dm" idx="${tactMap.get(F+'dm', -1)}"/>
+				<xacro:taxel mesh="${F}di" idx="${tactMap.get(F+'di', -1)}"/>
 			</tactile>
 		</sensor>
@@ -25,7 +25,7 @@
 			<parent link="${finger}_middle_link"/>
 			<tactile channel="tactile">
-				<xacro:taxel mesh="${F}mo" idx="${tactMap.get(F+'mo', -1)}" offset="${-1e-3*reflect} 0 0"/>
-				<xacro:taxel mesh="${F}mm" idx="${tactMap.get(F+'mm', -1)}" offset="0 -1e-3 0"/>
-				<xacro:taxel mesh="${F}mi" idx="${tactMap.get(F+'mi', -1)}" offset="${1e-3*reflect} 0 0"/>
+				<xacro:taxel mesh="${F}mo" idx="${tactMap.get(F+'mo', -1)}"/>
+				<xacro:taxel mesh="${F}mm" idx="${tactMap.get(F+'mm', -1)}"/>
+				<xacro:taxel mesh="${F}mi" idx="${tactMap.get(F+'mi', -1)}"/>
 			</tactile>
 		</sensor>
@@ -33,7 +33,7 @@
 			<parent link="${finger}_proximal_link"/>
 			<tactile channel="tactile">
-				<xacro:taxel mesh="${F}p" idx="${tactMap.get(F+'p', -1)}" offset="0 -1e-3 0"/>
-				<xacro:taxel mesh="${F}pi" idx="${tactMap.get(F+'pi', -1)}" offset="${1e-3*reflect} 0 0"/>
-				<xacro:taxel mesh="${F}po" idx="${tactMap.get(F+'po', -1)}" offset="${-1e-3*reflect} 0 0"/>
+				<xacro:taxel mesh="${F}p" idx="${tactMap.get(F+'p', -1)}"/>
+				<xacro:taxel mesh="${F}pi" idx="${tactMap.get(F+'pi', -1)}"/>
+				<xacro:taxel mesh="${F}po" idx="${tactMap.get(F+'po', -1)}"/>
 			</tactile>
 		</sensor>
@@ -48,8 +48,8 @@
 			<parent link="${prefix}thumb_proximal_link"/>
 			<tactile channel="tactile">
-				<xacro:taxel mesh="ptmp2" idx="${tactMap.get('ptmp', -1)}" offset="0 -1e-3 0"/>
-				<xacro:taxel mesh="ptmd2" idx="${tactMap.get('ptmd', -1)}" offset="0 -1e-3 0"/>
-				<xacro:taxel mesh="ptip2" idx="${tactMap.get('ptip', -1)}" offset="0 -1e-3 0"/>
-				<xacro:taxel mesh="ptid2" idx="${tactMap.get('ptid', -1)}" offset="0 -1e-3 0"/>
+				<xacro:taxel mesh="ptmp2" idx="${tactMap.get('ptmp', -1)}"/>
+				<xacro:taxel mesh="ptmd2" idx="${tactMap.get('ptmd', -1)}"/>
+				<xacro:taxel mesh="ptip2" idx="${tactMap.get('ptip', -1)}"/>
+				<xacro:taxel mesh="ptid2" idx="${tactMap.get('ptid', -1)}"/>
 			</tactile>
 		</sensor>
@@ -57,21 +57,21 @@
 			<parent link="${prefix}palm_link"/>
 			<tactile channel="tactile">
-				<xacro:taxel mesh="pdlo" idx="${tactMap.get('pdlo', -1)}" offset="0 -1e-3 0"/>
-				<xacro:taxel mesh="pdl" idx="${tactMap.get('pdl', -1)}" offset="0 -1e-3 0"/>
-				<xacro:taxel mesh="pdr" idx="${tactMap.get('pdr', -1)}" offset="0 -1e-3 0"/>
-				<xacro:taxel mesh="pdm" idx="${tactMap.get('pdm', -1)}" offset="0 -1e-3 0"/>
-				<xacro:taxel mesh="pdi" idx="${tactMap.get('pdi', -1)}" offset="0 -1e-3 0"/>
-				<xacro:taxel mesh="pdii" idx="${tactMap.get('pdii', -1)}" offset="0 -1e-3 0"/>
-				<xacro:taxel mesh="pcmp" idx="${tactMap.get('pcmp', -1)}" offset="0 -1e-3 0"/>
-				<xacro:taxel mesh="pcmd" idx="${tactMap.get('pcmd', -1)}" offset="0 -1e-3 0"/>
-				<xacro:taxel mesh="pcip" idx="${tactMap.get('pcip', -1)}" offset="0 -1e-3 0"/>
-				<xacro:taxel mesh="pcim" idx="${tactMap.get('pcim', -1)}" offset="0 -1e-3 0"/>
-				<xacro:taxel mesh="pcid" idx="${tactMap.get('pcid', -1)}" offset="0 -1e-3 0"/>
-				<xacro:taxel mesh="ptop" idx="${tactMap.get('ptop', -1)}" offset="0 -1e-3 0"/>
-				<xacro:taxel mesh="ptod" idx="${tactMap.get('ptod', -1)}" offset="0 -1e-3 0"/>
-				<xacro:taxel mesh="ptmp" idx="${tactMap.get('ptmp', -1)}" offset="0 -1e-3 0"/>
-				<xacro:taxel mesh="ptmd" idx="${tactMap.get('ptmd', -1)}" offset="0 -1e-3 0"/>
-				<xacro:taxel mesh="ptip" idx="${tactMap.get('ptip', -1)}" offset="0 -1e-3 0"/>
-				<xacro:taxel mesh="ptid" idx="${tactMap.get('ptid', -1)}" offset="0 -1e-3 0"/>
+				<xacro:taxel mesh="pdlo" idx="${tactMap.get('pdlo', -1)}"/>
+				<xacro:taxel mesh="pdl" idx="${tactMap.get('pdl', -1)}"/>
+				<xacro:taxel mesh="pdr" idx="${tactMap.get('pdr', -1)}"/>
+				<xacro:taxel mesh="pdm" idx="${tactMap.get('pdm', -1)}"/>
+				<xacro:taxel mesh="pdi" idx="${tactMap.get('pdi', -1)}"/>
+				<xacro:taxel mesh="pdii" idx="${tactMap.get('pdii', -1)}"/>
+				<xacro:taxel mesh="pcmp" idx="${tactMap.get('pcmp', -1)}"/>
+				<xacro:taxel mesh="pcmd" idx="${tactMap.get('pcmd', -1)}"/>
+				<xacro:taxel mesh="pcip" idx="${tactMap.get('pcip', -1)}"/>
+				<xacro:taxel mesh="pcim" idx="${tactMap.get('pcim', -1)}"/>
+				<xacro:taxel mesh="pcid" idx="${tactMap.get('pcid', -1)}"/>
+				<xacro:taxel mesh="ptop" idx="${tactMap.get('ptop', -1)}"/>
+				<xacro:taxel mesh="ptod" idx="${tactMap.get('ptod', -1)}"/>
+				<xacro:taxel mesh="ptmp" idx="${tactMap.get('ptmp', -1)}"/>
+				<xacro:taxel mesh="ptmd" idx="${tactMap.get('ptmd', -1)}"/>
+				<xacro:taxel mesh="ptip" idx="${tactMap.get('ptip', -1)}"/>
+				<xacro:taxel mesh="ptid" idx="${tactMap.get('ptid', -1)}"/>
 			</tactile>
 		</sensor>
