Commit message: Added support for taxel normals and position (only L3 currently)

File: model/L3.urdf.xacro (robot description, xacro)
@@ -1,7 +1,9 @@
 <?xml version="1.0"?>
 <robot name="tactile_glove_markers" xmlns:xacro="http://www.ros.org/wiki/xacro">
-	<xacro:macro name="taxel" params="prefix:=^ mesh idx">
+	<xacro:macro name="taxel" params="prefix:=^ tactData:=^ reflect:=^ mesh idx">
 		<xacro:if value="${idx >= 0}">
-			<taxel idx="${idx}">
+			<taxel idx="${idx}"
+			       xyz="${' '.join([str(v) for v in tactData['positions'][mesh]])}"
+			       rpy="${' '.join([str(v) for v in tactData['orientations'][mesh]])}">
 				<geometry>
 					<mesh filename="package://human_hand_description/model/meshes/taxels/L3/${mesh}.stl"
@@ -11,5 +13,5 @@
 		</xacro:if>
 	</xacro:macro>
-	<xacro:macro name="tactile_glove_finger" params="prefix:=^ finger tactMap:=^">
+	<xacro:macro name="tactile_glove_finger" params="prefix:=^ finger tactMap:=^ tactData:=^">
 		<xacro:property name="F" value="${finger[0]}"/>
 		<sensor name="${prefix}${finger}_distal" update_rate="100" group="distal">
@@ -39,5 +41,5 @@
 		</sensor>
 	</xacro:macro>
-	<xacro:macro name="tactile_glove" params="prefix reflect:=1 tactMap">
+	<xacro:macro name="tactile_glove" params="prefix reflect:=1 tactMap tactData">
 		<xacro:tactile_glove_finger finger="index"/>
 		<xacro:tactile_glove_finger finger="middle"/>

File: model/human_hand.urdf.xacro (robot description, xacro)
@@ -113,4 +113,6 @@
 				<xacro:property name="side" value="${mapping.get('handedness','right')}"/>
 			</xacro:if>
+			<xacro:property name="layout" value="${mapping.get('layout','L3')}"/>
+			<xacro:property name="taxel_data" value="${load_yaml('../model/'+layout+side+'.yaml')}"/>
 		</xacro:if>
 		<!-- left/right hand model-->
@@ -164,5 +166,5 @@
 		<xacro:if value="${tactile_mapping not in ['', '-']}">
 			<xacro:include filename="$(find human_hand_description)/model/${mapping['layout']}.urdf.xacro"/>
-			<xacro:tactile_glove prefix="${prefix}" reflect="${reflect}" tactMap="${mapping}"/>
+			<xacro:tactile_glove prefix="${prefix}" reflect="${reflect}" tactMap="${mapping}" tactData="${taxel_data}"/>
 		</xacro:if>
 	</xacro:macro>
