Commit message: Handle missing tactData in L2.urdf.xacro

File: model/L2.urdf.xacro (robot description, xacro)
@@ -1,15 +1,27 @@
 <?xml version="1.0"?>
 <robot name="tactile_glove_markers" xmlns:xacro="http://www.ros.org/wiki/xacro">
-	<xacro:macro name="taxel" params="prefix:=^ mesh idx">
+	<xacro:macro name="taxel" params="prefix:=^ tactData:=^|'-' reflect:=^ mesh idx">
 		<xacro:if value="${idx >= 0}">
-			<taxel idx="${idx}">
+			<xacro:if value="${tactData not in ['-']}" >
+				<taxel idx="${idx}"
+			       xyz="${' '.join([str(v) for v in tactData['positions'][mesh]])}"
+			       rpy="${' '.join([str(v) for v in tactData['orientations'][mesh]])}">
 				<geometry>
 					<mesh filename="package://human_hand_description/model/meshes/taxels/L2/${mesh}.stl"
 					      scale="${0.00101*reflect} 0.00101 0.00101"/>
 				</geometry>
-			</taxel>
+				</taxel>
+			</xacro:if>
+			<xacro:unless value="${tactData not in ['-']}" >
+				<taxel idx="${idx}">
+					<geometry>
+						<mesh filename="package://human_hand_description/model/meshes/taxels/L2/${mesh}.stl"
+									scale="${0.00101*reflect} 0.00101 0.00101"/>
+					</geometry>
+				</taxel>
+			</xacro:unless>
 		</xacro:if>
 	</xacro:macro>
-	<xacro:macro name="tactile_glove_finger" params="prefix:=^ finger tactMap:=^">
+	<xacro:macro name="tactile_glove_finger" params="prefix:=^ finger tactMap:=^ tactData:=^|'-'">
 		<xacro:property name="F" value="${finger[0]}"/>
 		<sensor name="${prefix}${finger}_distal" update_rate="100" group="distal">
@@ -39,5 +51,5 @@
 		</sensor>
 	</xacro:macro>
-	<xacro:macro name="tactile_glove" params="prefix reflect:=1 tactMap">
+	<xacro:macro name="tactile_glove" params="prefix reflect:=1 tactMap tactData:='-'">
 		<xacro:tactile_glove_finger finger="index"/>
 		<xacro:tactile_glove_finger finger="middle"/>
