Commit message: add missing ${prefix} to finger tactile sensors

File: model/tactile_markers.urdf.xacro (robot description, xacro)
@@ -28,5 +28,5 @@
 		<xacro:property name="F" value="${finger[0]}"/>
 		<sensor name="${prefix}${finger}_distal" update_rate="100" group="distal">
-			<parent link="${finger}_distal_link"/>
+			<parent link="${prefix}${finger}_distal_link"/>
 			<tactile channel="tactile glove">
 				<xacro:taxel mesh="${F}dd" idx="${tactMap.get(F+'dd', -1)}"/>
@@ -37,5 +37,5 @@
 		</sensor>
 		<sensor name="${prefix}${finger}_middle" update_rate="100" group="middle">
-			<parent link="${finger}_middle_link"/>
+			<parent link="${prefix}${finger}_middle_link"/>
 			<tactile channel="tactile glove">
 				<xacro:taxel mesh="${F}mo" idx="${tactMap.get(F+'mo', -1)}"/>
@@ -45,5 +45,5 @@
 		</sensor>
 		<sensor name="${prefix}${finger}_proximal" update_rate="100" group="proximal">
-			<parent link="${finger}_proximal_link"/>
+			<parent link="${prefix}${finger}_proximal_link"/>
 			<tactile channel="tactile glove">
 				<xacro:taxel mesh="${F}p" idx="${tactMap.get(F+'p', -1)}"/>
@@ -59,5 +59,5 @@
 		<xacro:tactile_glove_finger finger="little"/>
 		<xacro:tactile_glove_finger finger="thumb"/>
-		<sensor name="thumb_base" update_rate="100" group="proximal">
+		<sensor name="${prefix}thumb_base" update_rate="100" group="proximal">
 			<parent link="${prefix}thumb_proximal_link"/>
 			<tactile channel="tactile glove">
@@ -70,5 +70,5 @@
 			</tactile>
 		</sensor>
-		<sensor name="palm" update_rate="100" group="palm">
+		<sensor name="${prefix}palm" update_rate="100" group="palm">
 			<parent link="${prefix}palm_link"/>
 			<tactile channel="tactile glove">
