Commit message: Added taxel markers for the TactileGlove display Re-oriented the thumb base

File: model/human_hand.urdf.xacro (robot description, xacro)
@@ -157,5 +157,5 @@
 			<link name="${name}_knuckle_link">
 				<visual>
-          <origin xyz="0 0 0" rpy="0 -0.6240 0" />
+          <origin xyz="0 0 0" rpy="0 0 0" />
 					<geometry>
 						<mesh filename="package://pisa_hand_description/meshes/thumb_base.stl" scale=" 0.001 0.001 .001" />

Commit message: Renamed the package to human_hand_description

File: model/human_hand.urdf.xacro (robot description, xacro)
@@ -3,10 +3,10 @@
 	<!--
 		HUMAN HAND MODEL v 0.1
-    urdf derived from pisa soft_hand
+    urdf derived from human soft_hand
     author Guillaume Walck
     meshes from GrabCAD, author Joerg Schmit
 		original CAD model available at: https://grabcad.com/library/human-left-hand/
 	-->
-	<xacro:include filename="$(find pisa_hand_description)/model/materials.urdf.xacro"/>
+	<xacro:include filename="$(find human_hand_description)/model/materials.urdf.xacro"/>
 	<xacro:property name="pi" value="3.1415926535897931" />
 	<!-- joint properties -->
@@ -92,5 +92,5 @@
 			<visual>
 				<geometry>
-            <mesh filename="package://pisa_hand_description/meshes/${name}_proximal.stl" scale="0.001 0.001 .001" />
+            <mesh filename="package://human_hand_description/meshes/${name}_proximal.stl" scale="0.001 0.001 .001" />
 				</geometry>
 				<material name="HumanHand/Skin" />
@@ -109,5 +109,5 @@
 			<visual>
 				<geometry>
-					<mesh filename="package://pisa_hand_description/meshes/${name}_middle.stl" scale="0.001 0.001 .001" />
+					<mesh filename="package://human_hand_description/meshes/${name}_middle.stl" scale="0.001 0.001 .001" />
 				</geometry>
 				<material name="HumanHand/Skin" />
@@ -126,5 +126,5 @@
 			<visual>
 				<geometry>
-					<mesh filename="package://pisa_hand_description/meshes/${name}_distal.stl" scale=" 0.001 0.001 .001" />
+					<mesh filename="package://human_hand_description/meshes/${name}_distal.stl" scale=" 0.001 0.001 .001" />
 				</geometry>
 				 <material name="HumanHand/Skin" />
@@ -159,5 +159,5 @@
           <origin xyz="0 0 0" rpy="0 0 0" />
 					<geometry>
-						<mesh filename="package://pisa_hand_description/meshes/thumb_base.stl" scale=" 0.001 0.001 .001" />
+						<mesh filename="package://human_hand_description/meshes/thumb_base.stl" scale=" 0.001 0.001 .001" />
 					</geometry>
 					<material name="HumanHand/Skin" />
@@ -176,5 +176,5 @@
 			<visual>
 				<geometry>
-					<mesh filename="package://pisa_hand_description/meshes/thumb_proximal.stl" scale="0.001 0.001 .001" />
+					<mesh filename="package://human_hand_description/meshes/thumb_proximal.stl" scale="0.001 0.001 .001" />
 				</geometry>
 				<material name="HumanHand/Skin" />
@@ -192,5 +192,5 @@
 			<visual>
 				<geometry>
-					<mesh filename="package://pisa_hand_description/meshes/thumb_distal.stl" scale=" 0.001 0.001 .001" />
+					<mesh filename="package://human_hand_description/meshes/thumb_distal.stl" scale=" 0.001 0.001 .001" />
 				</geometry>
 				<material name="HumanHand/Skin" />
@@ -211,5 +211,5 @@
 				<visual>
 					<geometry>
-						<mesh filename="package://pisa_hand_description/meshes/palm.stl" scale="-0.001 -0.001 -0.001" />
+						<mesh filename="package://human_hand_description/meshes/palm.stl" scale="-0.001 -0.001 -0.001" />
 					</geometry>
 					<material name="HumanHand/Skin" />
@@ -219,5 +219,5 @@
 				<visual>
 					<geometry>
-						<mesh filename="package://pisa_hand_description/meshes/palm.stl" scale=" .001 .001 .001" />
+						<mesh filename="package://human_hand_description/meshes/palm.stl" scale=" .001 .001 .001" />
 					</geometry>
 					<material name="HumanHand/Skin" />

File: model/materials.urdf.xacro (robot description, xacro)
@@ -1,28 +1,4 @@
 <?xml version="1.0"?>
 <robot>
-	<material name="SoftHand/Red">
-		<color rgba="1.0 0.0 0.0 1.0"/>
-	</material>
-	<material name="SoftHand/Green">
-		<color rgba="0.0 1 0.0 1.0"/>
-	</material>
-	<material name="SoftHand/DarkGolden">
-		<color rgba="0.4 0.4 0.3 1.0"/>
-	</material>
-	<material name="SoftHand/Blue">
-		<color rgba="0.0 0.0 0.8 0.9"/>
-	</material>
-	<material name="SoftHand/LightBlue">
-		<color rgba="0.0 0.4 1.0 0.5"/>
-	</material>
-	<material name="SoftHand/LightGrey">
-		<color rgba="0.7 0.7 0.7 1.0"/>
-	</material>
-	<material name="SoftHand/DarkGrey">
-		<color rgba="0.4 0.4 0.4 1.0"/>
-	</material>
-	<material name="SoftHand/Black">
-		<color rgba="0.0 0.0 0.0 1.0"/>
-	</material>
   <material name="HumanHand/Skin">
 		<color rgba="0.802 0.732 0.673 1.0"/>

File: robot/human_hand_simple.urdf.xacro (robot description, xacro)
@@ -1,5 +1,5 @@
 <?xml version="1.0"?>
-<robot xmlns:xacro="http://www.ros.org/wiki/xacro" name="pisa_hand">
-	<xacro:include filename="$(find pisa_hand_description)/model/human_hand.urdf.xacro"/>
+<robot xmlns:xacro="http://www.ros.org/wiki/xacro" name="human_hand">
+	<xacro:include filename="$(find human_hand_description)/model/human_hand.urdf.xacro"/>
 	<link name="box">
 		<visual>
@@ -40,5 +40,5 @@
 	<link name="wrist_right">
 	</link>
-	<xacro:human_hand parent="wrist_right" name="pisa_hand_right" left="false">
+	<xacro:human_hand parent="wrist_right" name="human_hand_right" left="false">
 		<origin xyz="0.002 0.009 0.038" rpy="0 0 0"/>
 	</xacro:human_hand>

Commit message: Re-added mimic joint to the joints to close the hand in synergy fashion (copied from Pisa soft hand)

File: model/human_hand.urdf.xacro (robot description, xacro)
@@ -3,7 +3,7 @@
 	<!--
 		HUMAN HAND MODEL v 0.1
-    urdf derived from human soft_hand
-    author Guillaume Walck
-    meshes from GrabCAD, author Joerg Schmit
+		urdf derived from human soft_hand
+		author Guillaume Walck
+		meshes from GrabCAD, author Joerg Schmit
 		original CAD model available at: https://grabcad.com/library/human-left-hand/
 	-->
@@ -25,15 +25,15 @@
 	<xacro:property name="damping" value="0.0" />
 	<xacro:property name="friction" value="0.0" />
-  <!-- link properties -->
-  <xacro:property name="thumb_base_len" value="0.05415" />
-  <xacro:property name="thumb_proximal_len" value="0.03803" />
-  <xacro:property name="index_middle_len" value="0.027" />
-  <xacro:property name="index_proximal_len" value="0.046" />
-  <xacro:property name="middle_middle_len" value="0.033" />
-  <xacro:property name="middle_proximal_len" value="0.0495" />
-  <xacro:property name="ring_middle_len" value="0.033" />
-  <xacro:property name="ring_proximal_len" value="0.048" />
-  <xacro:property name="little_middle_len" value="0.0215" />
-  <xacro:property name="little_proximal_len" value="0.037" />
+	<!-- link properties -->
+	<xacro:property name="thumb_base_len" value="0.05415" />
+	<xacro:property name="thumb_proximal_len" value="0.03803" />
+	<xacro:property name="index_middle_len" value="0.027" />
+	<xacro:property name="index_proximal_len" value="0.046" />
+	<xacro:property name="middle_middle_len" value="0.033" />
+	<xacro:property name="middle_proximal_len" value="0.0495" />
+	<xacro:property name="ring_middle_len" value="0.033" />
+	<xacro:property name="ring_proximal_len" value="0.048" />
+	<xacro:property name="little_middle_len" value="0.0215" />
+	<xacro:property name="little_proximal_len" value="0.037" />
 	<!-- synergy vector -->
 	<xacro:property name="thumb_abd_R" value="1.3" />
@@ -65,5 +65,5 @@
 	<!-- SOFT FINGER model -->
 	<!-- 4 fingers are equal (index, middle, ring, little) -->
-	<xacro:macro name="soft_finger" params="parent parent_name prefix name position orientation proximal_len middle_len abd_R index:=1 middle:=0 ring:=0 little:=0 ">
+	<xacro:macro name="soft_finger" params="parent parent_name prefix name position orientation proximal_len middle_len useMimicTag abd_R inner_R middle_R outer_R index:=1 middle:=0 ring:=0 little:=0 ">
 		<!-- KNUCKLE -->
 		<joint name="${prefix}${name}_abd_joint" type="revolute">
@@ -74,4 +74,7 @@
 			<limit lower="${abd_lb *pi/180}" upper="${abd_ub *pi/180}" effort="${effort}" velocity="${velocity}"/>
 			<dynamics damping="${damping}" friction="${friction}"/>
+			<xacro:if value="${useMimicTag}">
+				<mimic joint="${parent_name}_synergy_joint" multiplier="${abd_R}"/>
+			</xacro:if>
 		</joint>
 		<link name="${prefix}${name}_knuckle_link">
@@ -85,4 +88,7 @@
 			<limit lower="${inner_lb *pi/180}" upper="${inner_ub *pi/180}" effort="${effort}" velocity="${velocity}"/>
 			<dynamics damping="${damping}" friction="${friction}"/>
+			<xacro:if value="${useMimicTag}">
+				<mimic joint="${parent_name}_synergy_joint" multiplier="${inner_R}"/>
+			</xacro:if>
 		</joint>
 		<link name="${prefix}${name}_proximal_link">
@@ -92,5 +98,5 @@
 			<visual>
 				<geometry>
-            <mesh filename="package://human_hand_description/meshes/${name}_proximal.stl" scale="0.001 0.001 .001" />
+						<mesh filename="package://human_hand_description/meshes/${name}_proximal.stl" scale="0.001 0.001 .001" />
 				</geometry>
 				<material name="HumanHand/Skin" />
@@ -105,4 +111,7 @@
 			<limit lower="${middle_lb *pi/180}" upper="${middle_ub *pi/180}" effort="${effort}" velocity="${velocity}"/>
 			<dynamics damping="${damping}" friction="${friction}"/>
+			<xacro:if value="${useMimicTag}">
+				<mimic joint="${parent_name}_synergy_joint" multiplier="${middle_R}"/>
+			</xacro:if>
 		</joint>
 		<link name="${prefix}${name}_middle_link">
@@ -122,4 +131,7 @@
 			<limit lower="${outer_lb *pi/180}" upper="${outer_ub *pi/180}" effort="${effort}" velocity="${velocity}"/>
 			<dynamics damping="${damping}" friction="${friction}"/>
+			<xacro:if value="${useMimicTag}">
+				<mimic joint="${parent_name}_synergy_joint" multiplier="${outer_R}"/>
+			</xacro:if>
 		</joint>
 		<link name="${prefix}${name}_distal_link">
@@ -134,5 +146,5 @@
 	<!-- THUMB MODEL -->
 	<!-- It has one joint less than rest of fingers -->
-	<xacro:macro name="soft_thumb" params="parent parent_name name position orientation base_len proximal_len abd_R ">
+	<xacro:macro name="soft_thumb" params="parent parent_name name position orientation base_len proximal_len  useMimicTag abd_R inner_R outer_R ">
 		<!-- THUMB RIGHT HAND -->
 			<!-- KNUCKLE -->
@@ -144,4 +156,7 @@
 				<limit lower="${thumb_abd_lb *pi/180}" upper="${thumb_abd_ub *pi/180}" effort="${effort}" velocity="${velocity}"/>
 				<dynamics damping="${damping}" friction="${friction}"/>
+				<xacro:if value="${useMimicTag}">
+					<mimic joint="${parent_name}_synergy_joint" multiplier="${abd_R}"/>
+				</xacro:if>
 			</joint>
 			<link name="${name}_fake_link">
@@ -157,5 +172,5 @@
 			<link name="${name}_knuckle_link">
 				<visual>
-          <origin xyz="0 0 0" rpy="0 0 0" />
+					<origin xyz="0 0 0" rpy="0 0 0" />
 					<geometry>
 						<mesh filename="package://human_hand_description/meshes/thumb_base.stl" scale=" 0.001 0.001 .001" />
@@ -165,6 +180,6 @@
 			</link>
 			<!-- PROXIMAL PHALANGE -->
-			    <joint name="${name}_inner_joint" type="revolute">
-	           	<origin xyz="0.0 0.0 ${base_len}" rpy="0.0 0.0 0.0" />
+			<joint name="${name}_inner_joint" type="revolute">
+				<origin xyz="0.0 0.0 ${base_len}" rpy="0.0 0.0 0.0" />
 				<parent link="${name}_knuckle_link"/>
 				<child link="${name}_proximal_link"/>
@@ -172,4 +187,7 @@
 				<limit lower="${inner_lb *pi/180}" upper="${inner_ub *pi/180}" effort="${effort}" velocity="${velocity}"/>
 				<dynamics damping="${damping}" friction="${friction}"/>
+				<xacro:if value="${useMimicTag}">
+					<mimic joint="${parent_name}_synergy_joint" multiplier="${inner_R}"/>
+				</xacro:if>
 			</joint>
 		<link name="${name}_proximal_link">
@@ -188,4 +206,7 @@
 			<axis xyz="0 -1 0" />
 			<limit lower="${outer_lb *pi/180}" upper="${outer_ub *pi/180}" effort="${effort}" velocity="${velocity}"/>
+			<xacro:if value="${useMimicTag}">
+				<mimic joint="${parent_name}_synergy_joint" multiplier="${outer_R}"/>
+			</xacro:if>
 		</joint>
 		<link name="${name}_distal_link">
@@ -199,5 +220,5 @@
 	</xacro:macro>
 	<!-- HUMAN HAND MODEL -->
-	<xacro:macro name="human_hand" params="parent name left *origin">
+	<xacro:macro name="human_hand" params="parent name useMimicTag left *origin">
 		<!-- PALM -->
 		<joint name="${name}_palm_joint" type="fixed" >
@@ -225,10 +246,27 @@
 			</xacro:unless>
 		</link>
+		<!-- MOTOR JOINT -->
+		<xacro:if value="${useMimicTag}">
+			<joint name="${name}_synergy_joint" type="revolute" >
+				<parent link="${name}_palm_link" />
+				<child link="${name}_invisible_wire_link"/>
+				<axis xyz="0 0 1" />
+				<limit lower="${synergy_lb}" upper="${synergy_ub}" effort="${max_synergy_effort}" velocity="${max_synergy_velocity}"/>
+				<dynamics damping="${synergy_damping}" friction="${synergy_friction}"/>
+			</joint>
+			<link name="${name}_invisible_wire_link">
+				<inertial>
+					 <origin xyz="0 0 0"/>
+					<mass value="0.001"/>
+					<inertia ixx="0.000001" ixy="0.0" ixz="0.0" iyy="0.000001" iyz="0.0" izz="0.000001"/>
+				</inertial>
+			</link>
+		</xacro:if>
 		<!-- THUMB AND FINGERS -->
-			<xacro:soft_thumb parent="${name}_palm_link" parent_name="${name}" name="${name}_thumb" position="0.02475 -0.0125 0.0125" orientation="0.0 0.6240 0" base_len="${thumb_base_len}" proximal_len="${thumb_proximal_len}" abd_R="${thumb_abd_R *(thumb_abd_ub - thumb_abd_lb)*pi/180}"  />
-			<xacro:soft_finger parent="${name}_palm_link" parent_name="${name}" prefix="${name}_" name="index" position="0.02175 -0.002 0.099" orientation="0 0 0" proximal_len="${index_proximal_len}" middle_len="${index_middle_len}"  abd_R="${index_abd_R}"  />
-			<xacro:soft_finger parent="${name}_palm_link" parent_name="${name}" prefix="${name}_" name="middle" position="-0.002 0.0015 0.0955" orientation="0 0 0.0" proximal_len="${middle_proximal_len}" middle_len="${middle_middle_len}" abd_R="${middle_abd_R}"  />
-			<xacro:soft_finger parent="${name}_palm_link" parent_name="${name}" prefix="${name}_" name="ring" position="-0.02225 0.0010 0.090" orientation="0 0 0" proximal_len="${ring_proximal_len}" middle_len="${ring_middle_len}" abd_R="${ring_abd_R}" />
-			<xacro:soft_finger parent="${name}_palm_link" parent_name="${name}" prefix="${name}_" name="little" position=" -0.04175 -0.003 0.079" orientation="0 0 0" proximal_len="${little_proximal_len}" middle_len="${little_middle_len}" abd_R="${little_abd_R}" />
+			<xacro:soft_thumb parent="${name}_palm_link" parent_name="${name}" name="${name}_thumb" position="0.02475 -0.0125 0.0125" orientation="0.0 0.6240 0" base_len="${thumb_base_len}" proximal_len="${thumb_proximal_len}" useMimicTag="${useMimicTag}" abd_R="${thumb_abd_R *(thumb_abd_ub - thumb_abd_lb)*pi/180}"  inner_R="${thumb_inner_R *(inner_ub - inner_lb)*pi/180}" outer_R="${thumb_outer_R *(outer_ub - outer_lb)*pi/180}" />
+			<xacro:soft_finger parent="${name}_palm_link" parent_name="${name}" prefix="${name}_" name="index" position="0.02175 -0.002 0.099" orientation="0 0 0" proximal_len="${index_proximal_len}" middle_len="${index_middle_len}"   useMimicTag="${useMimicTag}" abd_R="${index_abd_R}" inner_R="${index_inner_R *(inner_ub - inner_lb)*pi/180}" middle_R="${index_middle_R *(middle_ub - middle_lb)*pi/180}" outer_R="${index_outer_R *(outer_ub - outer_lb)*pi/180}" />
+			<xacro:soft_finger parent="${name}_palm_link" parent_name="${name}" prefix="${name}_" name="middle" position="-0.002 0.0015 0.0955" orientation="0 0 0.0" proximal_len="${middle_proximal_len}" middle_len="${middle_middle_len}" useMimicTag="${useMimicTag}" abd_R="${middle_abd_R}" inner_R="${middle_inner_R *(inner_ub - inner_lb)*pi/180}" middle_R="${middle_middle_R *(middle_ub - middle_lb)*pi/180}" outer_R="${middle_outer_R *(outer_ub - outer_lb)*pi/180}"  />
+			<xacro:soft_finger parent="${name}_palm_link" parent_name="${name}" prefix="${name}_" name="ring" position="-0.02225 0.0010 0.090" orientation="0 0 0" proximal_len="${ring_proximal_len}" middle_len="${ring_middle_len}" useMimicTag="${useMimicTag}" abd_R="${ring_abd_R}" inner_R="${ring_inner_R *(inner_ub - inner_lb)*pi/180}" middle_R="${ring_middle_R *(middle_ub - middle_lb)*pi/180}" outer_R="${ring_outer_R *(outer_ub - outer_lb)*pi/180}" />
+			<xacro:soft_finger parent="${name}_palm_link" parent_name="${name}" prefix="${name}_" name="little" position=" -0.04175 -0.003 0.079" orientation="0 0 0" proximal_len="${little_proximal_len}" middle_len="${little_middle_len}" useMimicTag="${useMimicTag}" abd_R="${little_abd_R}" inner_R="${little_inner_R *(inner_ub - inner_lb)*pi/180}" middle_R="${little_middle_R *(middle_ub - middle_lb)*pi/180}" outer_R="${little_outer_R *(outer_ub - outer_lb)*pi/180}" />
 	</xacro:macro>
 </robot>

File: robot/human_hand_simple.urdf.xacro (robot description, xacro)
@@ -40,5 +40,5 @@
 	<link name="wrist_right">
 	</link>
-	<xacro:human_hand parent="wrist_right" name="human_hand_right" left="false">
+	<xacro:human_hand parent="wrist_right" name="human_hand_right" left="false" useMimicTag="$(arg use_mimic_tag)" >
 		<origin xyz="0.002 0.009 0.038" rpy="0 0 0"/>
 	</xacro:human_hand>
