Commit message: allow left and right hand version
switching is done by substitution arg left_hand:=false/true

File: model/human_hand.urdf.xacro (robot description, xacro)
@@ -65,5 +65,5 @@
 	<!-- SOFT FINGER model -->
 	<!-- 4 fingers are equal (index, middle, ring, little) -->
-	<xacro:macro name="soft_finger" params="parent parent_name prefix name position orientation proximal_len middle_len useMimicTag abd_R inner_R middle_R outer_R index:=1 middle:=0 ring:=0 little:=0 ">
+	<xacro:macro name="soft_finger" params="parent parent_name prefix name swap position orientation proximal_len middle_len useMimicTag abd_R inner_R middle_R outer_R index:=1 middle:=0 ring:=0 little:=0 ">
 		<!-- KNUCKLE -->
 		<joint name="${prefix}${name}_abd_joint" type="revolute">
@@ -71,5 +71,5 @@
 			<parent link="${parent}"/>
 			<child link="${prefix}${name}_knuckle_link"/>
-			<axis xyz="0 -1 0" />
+			<axis xyz="0 ${-1*swap} 0" />
 			<limit lower="${abd_lb *pi/180}" upper="${abd_ub *pi/180}" effort="${effort}" velocity="${velocity}"/>
 			<dynamics damping="${damping}" friction="${friction}"/>
@@ -78,6 +78,5 @@
 			</xacro:if>
 		</joint>
-		<link name="${prefix}${name}_knuckle_link">
-		</link>
+		<link name="${prefix}${name}_knuckle_link"/>
 		<!-- PROXIMAL PHALANGE -->
 		<joint name="${prefix}${name}_inner_joint" type="revolute">
@@ -98,5 +97,6 @@
 			<visual>
 				<geometry>
-						<mesh filename="package://human_hand_description/meshes/${name}_proximal.stl" scale="0.001 0.001 .001" />
+						<mesh filename="package://human_hand_description/meshes/${name}_proximal.stl"
+						      scale="${0.001*swap} 0.001 .001" />
 				</geometry>
 				<material name="HumanHand/Skin" />
@@ -118,5 +118,6 @@
 			<visual>
 				<geometry>
-					<mesh filename="package://human_hand_description/meshes/${name}_middle.stl" scale="0.001 0.001 .001" />
+					<mesh filename="package://human_hand_description/meshes/${name}_middle.stl"
+					      scale="${0.001*swap} 0.001 .001" />
 				</geometry>
 				<material name="HumanHand/Skin" />
@@ -138,5 +139,6 @@
 			<visual>
 				<geometry>
-					<mesh filename="package://human_hand_description/meshes/${name}_distal.stl" scale=" 0.001 0.001 .001" />
+					<mesh filename="package://human_hand_description/meshes/${name}_distal.stl"
+					      scale="${0.001*swap} 0.001 .001" />
 				</geometry>
 				 <material name="HumanHand/Skin" />
@@ -146,6 +148,6 @@
 	<!-- THUMB MODEL -->
 	<!-- It has one joint less than rest of fingers -->
-	<xacro:macro name="soft_thumb" params="parent parent_name name position orientation base_len proximal_len  useMimicTag abd_R inner_R outer_R ">
-		<!-- THUMB RIGHT HAND -->
+	<xacro:macro name="soft_thumb" params="parent parent_name name swap position orientation base_len proximal_len  useMimicTag abd_R inner_R outer_R ">
+		<!-- THUMB -->
 			<!-- KNUCKLE -->
 			<joint name="${name}_abd_joint" type="revolute">
@@ -160,11 +162,10 @@
 				</xacro:if>
 			</joint>
-			<link name="${name}_fake_link">
-			</link>
+			<link name="${name}_fake_link"/>
 			<joint name="${name}_rot_joint" type="revolute">
 				<origin xyz="0 0 0" rpy="0 0 0" />
 				<parent link="${name}_fake_link"/>
 				<child link="${name}_knuckle_link"/>
-				<axis xyz="0 -1 0" />
+				<axis xyz="0 ${-1*swap} 0" />
 				<limit lower="${thumb_abd_lb *pi/180}" upper="${thumb_abd_ub *pi/180}" effort="${effort}" velocity="${velocity}"/>
 				<dynamics damping="${damping}" friction="${friction}"/>
@@ -174,5 +175,6 @@
 					<origin xyz="0 0 0" rpy="0 0 0" />
 					<geometry>
-						<mesh filename="package://human_hand_description/meshes/thumb_base.stl" scale=" 0.001 0.001 .001" />
+						<mesh filename="package://human_hand_description/meshes/thumb_base.stl"
+						      scale="${0.001*swap} 0.001 .001" />
 					</geometry>
 					<material name="HumanHand/Skin" />
@@ -184,5 +186,5 @@
 				<parent link="${name}_knuckle_link"/>
 				<child link="${name}_proximal_link"/>
-				<axis xyz="0 -1 0" />
+				<axis xyz="0 ${-1*swap} 0" />
 				<limit lower="${inner_lb *pi/180}" upper="${inner_ub *pi/180}" effort="${effort}" velocity="${velocity}"/>
 				<dynamics damping="${damping}" friction="${friction}"/>
@@ -194,5 +196,6 @@
 			<visual>
 				<geometry>
-					<mesh filename="package://human_hand_description/meshes/thumb_proximal.stl" scale="0.001 0.001 .001" />
+					<mesh filename="package://human_hand_description/meshes/thumb_proximal.stl"
+					      scale="${0.001*swap} 0.001 .001" />
 				</geometry>
 				<material name="HumanHand/Skin" />
@@ -204,5 +207,5 @@
 			<parent link="${name}_proximal_link"/>
 			<child link="${name}_distal_link"/>
-			<axis xyz="0 -1 0" />
+			<axis xyz="0 ${-1*swap} 0" />
 			<limit lower="${outer_lb *pi/180}" upper="${outer_ub *pi/180}" effort="${effort}" velocity="${velocity}"/>
 			<xacro:if value="${useMimicTag}">
@@ -213,5 +216,6 @@
 			<visual>
 				<geometry>
-					<mesh filename="package://human_hand_description/meshes/thumb_distal.stl" scale=" 0.001 0.001 .001" />
+					<mesh filename="package://human_hand_description/meshes/thumb_distal.stl"
+					      scale="${0.001*swap} 0.001 .001" />
 				</geometry>
 				<material name="HumanHand/Skin" />
@@ -221,7 +225,11 @@
 	<!-- HUMAN HAND MODEL -->
 	<xacro:macro name="human_hand" params="parent name useMimicTag left *origin">
+		<!-- left/right hand model-->
+		<xacro:property name="swap" value="1" />
+		<xacro:if value="${left}">
+			<xacro:property name="swap" value="-1" />
+		</xacro:if>
 		<!-- PALM -->
 		<joint name="${name}_palm_joint" type="fixed" >
-			<origin xyz="-0.01 0 0.06" rpy="0 0 0" />
 			<insert_block name="origin"/>
 			<parent link="${parent}" />
@@ -229,20 +237,11 @@
 		</joint>
 		<link name="${name}_palm_link">
-			<xacro:if value="${left}">
-				<visual>
-					<geometry>
-						<mesh filename="package://human_hand_description/meshes/palm.stl" scale="-0.001 -0.001 -0.001" />
-					</geometry>
-					<material name="HumanHand/Skin" />
-				</visual>
-			</xacro:if>
-			<xacro:unless value="${left}">
-				<visual>
-					<geometry>
-						<mesh filename="package://human_hand_description/meshes/palm.stl" scale=" .001 .001 .001" />
-					</geometry>
-					<material name="HumanHand/Skin" />
-				</visual>
-			</xacro:unless>
+			<visual>
+				<geometry>
+					<mesh filename="package://human_hand_description/meshes/palm.stl"
+					      scale=" ${.001*swap} .001 .001" />
+				</geometry>
+				<material name="HumanHand/Skin" />
+			</visual>
 		</link>
 		<!-- MOTOR JOINT -->
@@ -255,18 +254,12 @@
 				<dynamics damping="${synergy_damping}" friction="${synergy_friction}"/>
 			</joint>
-			<link name="${name}_invisible_wire_link">
-				<inertial>
-					 <origin xyz="0 0 0"/>
-					<mass value="0.001"/>
-					<inertia ixx="0.000001" ixy="0.0" ixz="0.0" iyy="0.000001" iyz="0.0" izz="0.000001"/>
-				</inertial>
-			</link>
+			<link name="${name}_invisible_wire_link"/>
 		</xacro:if>
 		<!-- THUMB AND FINGERS -->
-			<xacro:soft_thumb parent="${name}_palm_link" parent_name="${name}" name="${name}_thumb" position="0.02475 -0.0125 0.0125" orientation="0.0 0.6240 0" base_len="${thumb_base_len}" proximal_len="${thumb_proximal_len}" useMimicTag="${useMimicTag}" abd_R="${thumb_abd_R *(thumb_abd_ub - thumb_abd_lb)*pi/180}"  inner_R="${thumb_inner_R *(inner_ub - inner_lb)*pi/180}" outer_R="${thumb_outer_R *(outer_ub - outer_lb)*pi/180}" />
-			<xacro:soft_finger parent="${name}_palm_link" parent_name="${name}" prefix="${name}_" name="index" position="0.02175 -0.002 0.099" orientation="0 0 0" proximal_len="${index_proximal_len}" middle_len="${index_middle_len}"   useMimicTag="${useMimicTag}" abd_R="${index_abd_R}" inner_R="${index_inner_R *(inner_ub - inner_lb)*pi/180}" middle_R="${index_middle_R *(middle_ub - middle_lb)*pi/180}" outer_R="${index_outer_R *(outer_ub - outer_lb)*pi/180}" />
-			<xacro:soft_finger parent="${name}_palm_link" parent_name="${name}" prefix="${name}_" name="middle" position="-0.002 0.0015 0.0955" orientation="0 0 0.0" proximal_len="${middle_proximal_len}" middle_len="${middle_middle_len}" useMimicTag="${useMimicTag}" abd_R="${middle_abd_R}" inner_R="${middle_inner_R *(inner_ub - inner_lb)*pi/180}" middle_R="${middle_middle_R *(middle_ub - middle_lb)*pi/180}" outer_R="${middle_outer_R *(outer_ub - outer_lb)*pi/180}"  />
-			<xacro:soft_finger parent="${name}_palm_link" parent_name="${name}" prefix="${name}_" name="ring" position="-0.02225 0.0010 0.090" orientation="0 0 0" proximal_len="${ring_proximal_len}" middle_len="${ring_middle_len}" useMimicTag="${useMimicTag}" abd_R="${ring_abd_R}" inner_R="${ring_inner_R *(inner_ub - inner_lb)*pi/180}" middle_R="${ring_middle_R *(middle_ub - middle_lb)*pi/180}" outer_R="${ring_outer_R *(outer_ub - outer_lb)*pi/180}" />
-			<xacro:soft_finger parent="${name}_palm_link" parent_name="${name}" prefix="${name}_" name="little" position=" -0.04175 -0.003 0.079" orientation="0 0 0" proximal_len="${little_proximal_len}" middle_len="${little_middle_len}" useMimicTag="${useMimicTag}" abd_R="${little_abd_R}" inner_R="${little_inner_R *(inner_ub - inner_lb)*pi/180}" middle_R="${little_middle_R *(middle_ub - middle_lb)*pi/180}" outer_R="${little_outer_R *(outer_ub - outer_lb)*pi/180}" />
+			<xacro:soft_thumb parent="${name}_palm_link" parent_name="${name}" name="${name}_thumb" swap="${swap}" position="${0.02475*swap} -0.0125 0.0125" orientation="0.0 ${0.6240*swap} 0" base_len="${thumb_base_len}" proximal_len="${thumb_proximal_len}" useMimicTag="${useMimicTag}" abd_R="${thumb_abd_R *(thumb_abd_ub - thumb_abd_lb)*pi/180}"  inner_R="${thumb_inner_R *(inner_ub - inner_lb)*pi/180}" outer_R="${thumb_outer_R *(outer_ub - outer_lb)*pi/180}" />
+			<xacro:soft_finger parent="${name}_palm_link" parent_name="${name}" prefix="${name}_" name="index" swap="${swap}" position="${0.02175*swap} -0.002 0.099" orientation="0 0 0" proximal_len="${index_proximal_len}" middle_len="${index_middle_len}"   useMimicTag="${useMimicTag}" abd_R="${index_abd_R}" inner_R="${index_inner_R *(inner_ub - inner_lb)*pi/180}" middle_R="${index_middle_R *(middle_ub - middle_lb)*pi/180}" outer_R="${index_outer_R *(outer_ub - outer_lb)*pi/180}" />
+			<xacro:soft_finger parent="${name}_palm_link" parent_name="${name}" prefix="${name}_" name="middle" swap="${swap}" position="${-0.002*swap} 0.0015 0.0955" orientation="0 0 0.0" proximal_len="${middle_proximal_len}" middle_len="${middle_middle_len}" useMimicTag="${useMimicTag}" abd_R="${middle_abd_R}" inner_R="${middle_inner_R *(inner_ub - inner_lb)*pi/180}" middle_R="${middle_middle_R *(middle_ub - middle_lb)*pi/180}" outer_R="${middle_outer_R *(outer_ub - outer_lb)*pi/180}"  />
+			<xacro:soft_finger parent="${name}_palm_link" parent_name="${name}" prefix="${name}_" name="ring" swap="${swap}" position="${-0.02225*swap} 0.0010 0.090" orientation="0 0 0" proximal_len="${ring_proximal_len}" middle_len="${ring_middle_len}" useMimicTag="${useMimicTag}" abd_R="${ring_abd_R}" inner_R="${ring_inner_R *(inner_ub - inner_lb)*pi/180}" middle_R="${ring_middle_R *(middle_ub - middle_lb)*pi/180}" outer_R="${ring_outer_R *(outer_ub - outer_lb)*pi/180}" />
+			<xacro:soft_finger parent="${name}_palm_link" parent_name="${name}" prefix="${name}_" name="little" swap="${swap}" position="${-0.04175*swap} -0.003 0.079" orientation="0 0 0" proximal_len="${little_proximal_len}" middle_len="${little_middle_len}" useMimicTag="${useMimicTag}" abd_R="${little_abd_R}" inner_R="${little_inner_R *(inner_ub - inner_lb)*pi/180}" middle_R="${little_middle_R *(middle_ub - middle_lb)*pi/180}" outer_R="${little_outer_R *(outer_ub - outer_lb)*pi/180}" />
 	</xacro:macro>
 </robot>

File: robot/human_hand.urdf.xacro (robot description, xacro)
@@ -3,6 +3,6 @@
 	<xacro:include filename="$(find human_hand_description)/model/human_hand.urdf.xacro"/>
 	<link name="world"/>
-	<xacro:human_hand parent="world" name="human_hand_right" left="false" useMimicTag="$(arg use_mimic_tag)" >
-		<origin xyz="0.002 0.009 0.038" rpy="0 0 0"/>
+	<xacro:human_hand parent="world" name="human_hand_right" left="$(arg left_hand)" useMimicTag="$(arg use_mimic_tag)" >
+		<origin xyz="0 0 0" rpy="0 0 0"/>
 	</xacro:human_hand>
 </robot>

Commit message: distinguish P2 and P3 tactile mapping
arg "tactile_mapping" defines mapping name
defining xacro:property "tactile_mapping" before loading model/human_hand.urdf.xacro
ensures, that correct mapping file is loaded therein (requires inorder xacro processing!)

File: model/human_hand.urdf.xacro (robot description, xacro)
@@ -9,5 +9,5 @@
 	-->
 	<xacro:include filename="$(find human_hand_description)/model/materials.urdf.xacro"/>
-	<xacro:include filename="$(find human_hand_description)/model/glove_markers.urdf.xacro"/>
+	<xacro:include filename="$(find human_hand_description)/model/${tactile_mapping}.urdf.xacro"/>
 	<xacro:property name="pi" value="3.1415926535897931" />
 	<!-- joint properties -->

File: robot/human_hand.urdf.xacro (robot description, xacro)
@@ -1,4 +1,8 @@
 <?xml version="1.0"?>
 <robot xmlns:xacro="http://www.ros.org/wiki/xacro" name="human_hand">
+	<xacro:arg name="left_hand" default="false"/>
+	<xacro:arg name="use_mimic_tag" default="false"/>
+	<xacro:arg name="tactile_mapping" default="P3"/>
+	<xacro:property name="tactile_mapping" value="$(arg tactile_mapping)"/>
 	<xacro:include filename="$(find human_hand_description)/model/human_hand.urdf.xacro"/>
 	<link name="world"/>

File: robot/twohands.urdf.xacro (robot description, xacro)
@@ -1,4 +1,7 @@
 <?xml version="1.0"?>
 <robot xmlns:xacro="http://www.ros.org/wiki/xacro" name="human_hand">
+	<xacro:arg name="use_mimic_tag" default="false"/>
+	<xacro:arg name="tactile_mapping" default="P3"/>
+	<xacro:property name="tactile_mapping" value="$(arg tactile_mapping)"/>
 	<xacro:include filename="$(find human_hand_description)/model/human_hand.urdf.xacro"/>
 	<link name="world"/>

Commit message: moved all taxel mappings into the single file model/taxel.yaml

File: model/human_hand.urdf.xacro (robot description, xacro)
@@ -9,5 +9,4 @@
 	-->
 	<xacro:include filename="$(find human_hand_description)/model/materials.urdf.xacro"/>
-	<xacro:property name="_tactileMappingToLayout" value="${dict(P2='P2', P3l='P3', P3r='P3')}"/>
 	<!-- joint properties -->
 	<xacro:property name="abd_lb" value="-30" />
@@ -65,5 +64,5 @@
 	<!-- SOFT FINGER model -->
 	<!-- 4 fingers are equal (index, middle, ring, little) -->
-	<xacro:macro name="finger" params="parent parent_name prefix name reflect position orientation proximal_len middle_len useMimicTag abd_R inner_R middle_R outer_R index:=1 middle:=0 ring:=0 little:=0 ">
+	<xacro:macro name="finger" params="tactile_mapping:=$ parent parent_name prefix name reflect position orientation proximal_len middle_len useMimicTag abd_R inner_R middle_R outer_R index:=1 middle:=0 ring:=0 little:=0 ">
 		<!-- KNUCKLE -->
 		<joint name="${prefix}${name}_abd_joint" type="revolute">
@@ -262,7 +261,8 @@
 		<xacro:finger parent="${name}_palm_link" parent_name="${name}" prefix="${name}_" name="ring" reflect="${reflect}" position="${-0.02225*reflect} 0.0010 0.090" orientation="0 0 0" proximal_len="${ring_proximal_len}" middle_len="${ring_middle_len}" useMimicTag="${useMimicTag}" abd_R="${ring_abd_R}" inner_R="${ring_inner_R *(inner_ub - inner_lb)*pi/180}" middle_R="${ring_middle_R *(middle_ub - middle_lb)*pi/180}" outer_R="${ring_outer_R *(outer_ub - outer_lb)*pi/180}" />
 		<xacro:finger parent="${name}_palm_link" parent_name="${name}" prefix="${name}_" name="little" reflect="${reflect}" position="${-0.04175*reflect} -0.003 0.079" orientation="0 0 0" proximal_len="${little_proximal_len}" middle_len="${little_middle_len}" useMimicTag="${useMimicTag}" abd_R="${little_abd_R}" inner_R="${little_inner_R *(inner_ub - inner_lb)*pi/180}" middle_R="${little_middle_R *(middle_ub - middle_lb)*pi/180}" outer_R="${little_outer_R *(outer_ub - outer_lb)*pi/180}" />
-		<xacro:property name="tactile_mapping_file" value="../model/${tactile_mapping}.mapping.yaml"/>
-		<xacro:include filename="$(find human_hand_description)/model/${_tactileMappingToLayout[tactile_mapping]}.urdf.xacro"/>
-		<xacro:tactile_glove name="${name}" reflect="${reflect}" tactMap="${load_yaml(tactile_mapping_file)}"/>
+		<!-- TACTILE MARKERS -->
+		<xacro:property name="mapping" value="${load_yaml('../model/taxel.yaml')[tactile_mapping]}"/>
+		<xacro:include filename="$(find human_hand_description)/model/${mapping['layout']}.urdf.xacro"/>
+		<xacro:tactile_glove name="${name}" reflect="${reflect}" tactMap="${mapping}"/>
 	</xacro:macro>
 </robot>

Commit message: choose left/right hand version based on tactile_mapping

File: model/human_hand.urdf.xacro (robot description, xacro)
@@ -223,10 +223,14 @@
 	</xacro:macro>
 	<!-- HUMAN HAND MODEL -->
-	<xacro:macro name="human_hand" params="parent name useMimicTag left *origin">
+	<xacro:macro name="human_hand" params="parent name useMimicTag side:='' tactile_mapping:='' *origin">
+		<xacro:if value="${tactile_mapping not in ['', '-']}">
+			<xacro:property name="mapping" value="${load_yaml('../model/taxel.yaml')[tactile_mapping]}"/>
+			<!-- if side is not yet specified, try to fetch it from the mapping -->
+			<xacro:if value="${side not in ['left', 'right']}">
+				<xacro:property name="side" value="${mapping.get('handedness','right')}"/>
+			</xacro:if>
+		</xacro:if>
 		<!-- left/right hand model-->
-		<xacro:property name="reflect" value="1" />
-		<xacro:if value="${left}">
-			<xacro:property name="reflect" value="-1" />
-		</xacro:if>
+		<xacro:property name="reflect" value="${dict(right=1, left=-1)[side]}" />
 		<!-- PALM -->
 		<joint name="${name}_palm_joint" type="fixed" >
@@ -262,7 +266,8 @@
 		<xacro:finger parent="${name}_palm_link" parent_name="${name}" prefix="${name}_" name="little" reflect="${reflect}" position="${-0.04175*reflect} -0.003 0.079" orientation="0 0 0" proximal_len="${little_proximal_len}" middle_len="${little_middle_len}" useMimicTag="${useMimicTag}" abd_R="${little_abd_R}" inner_R="${little_inner_R *(inner_ub - inner_lb)*pi/180}" middle_R="${little_middle_R *(middle_ub - middle_lb)*pi/180}" outer_R="${little_outer_R *(outer_ub - outer_lb)*pi/180}" />
 		<!-- TACTILE MARKERS -->
-		<xacro:property name="mapping" value="${load_yaml('../model/taxel.yaml')[tactile_mapping]}"/>
-		<xacro:include filename="$(find human_hand_description)/model/${mapping['layout']}.urdf.xacro"/>
-		<xacro:tactile_glove name="${name}" reflect="${reflect}" tactMap="${mapping}"/>
+		<xacro:if value="${tactile_mapping not in ['', '-']}">
+			<xacro:include filename="$(find human_hand_description)/model/${mapping['layout']}.urdf.xacro"/>
+			<xacro:tactile_glove name="${name}" reflect="${reflect}" tactMap="${mapping}"/>
+		</xacro:if>
 	</xacro:macro>
 </robot>

File: robots/human_hand.urdf.xacro (robot description, xacro)
@@ -1,11 +1,12 @@
 <?xml version="1.0"?>
 <robot xmlns:xacro="http://www.ros.org/wiki/xacro" name="human_hand">
-	<xacro:arg name="left_hand" default="false"/>
+	<!-- side can be left | right | '' | '-' (meaning, fetch from mapping) -->
+	<xacro:arg name="side" default=""/>
 	<xacro:arg name="use_mimic_tag" default="false"/>
 	<xacro:arg name="tactile_mapping" default="P3r"/>
-	<xacro:property name="tactile_mapping" value="$(arg tactile_mapping)"/>
 	<xacro:include filename="$(find human_hand_description)/model/human_hand.urdf.xacro"/>
 	<link name="world"/>
-	<xacro:human_hand parent="world" name="human_hand_right" left="$(arg left_hand)" useMimicTag="$(arg use_mimic_tag)" >
+	<xacro:human_hand parent="world" name="human_hand$(arg side)" side="$(arg side)"
+	                  tactile_mapping="$(arg tactile_mapping)" useMimicTag="$(arg use_mimic_tag)">
 		<origin xyz="0 0 0" rpy="0 0 0"/>
 	</xacro:human_hand>

Commit message: Handle non existing taxeldata file

File: model/human_hand.urdf.xacro (robot description, xacro)
@@ -114,5 +114,8 @@
 			</xacro:if>
 			<xacro:property name="layout" value="${mapping.get('layout','L3')}"/>
-			<xacro:property name="taxel_data" value="${load_yaml('../model/'+layout+side+'.yaml')}"/>
+			<xacro:property name="taxeldata_file" value="${mapping.get('taxeldata_file','../model/'+layout+side+'.yaml')}"/>
+			<xacro:if value="${taxeldata_file not in ['', '-']}">
+				<xacro:property name="taxel_data" value="${load_yaml(taxeldata_file)}"/>
+			</xacro:if>
 		</xacro:if>
 		<!-- left/right hand model-->
