Commit message: fixed tactile marker description in urdf
Use a single generic tactile_markers.urdf.xacro instead of L[123].urdf.xacro
Adapted channel to "tactile glove" (after change in TactileGlove repo)
Handling of different taxel layouts by tactMap.get('xxx', -1), merged taxel names from all layouts.
Handle availability of tactile data description yamls (tactData -> None).

File: model/human_hand.urdf.xacro (robot description, xacro)
@@ -107,12 +107,15 @@
 		<xacro:property name="synergies" value="${properties['synergies']}"/>
 		<!-- load taxel mapping -->
+		<xacro:property name="mapping" value="${None}"/>
 		<xacro:if value="${tactile_mapping not in ['', '-']}">
 			<xacro:property name="mapping" value="${load_yaml('../model/taxel.yaml')[tactile_mapping]}"/>
-			<!-- if side is not yet specified, try to fetch it from the mapping -->
+			<!-- if side is not yet specified, try to fetch it from the tactile_mapping dictionary -->
 			<xacro:if value="${side not in ['left', 'right']}">
 				<xacro:property name="side" value="${mapping.get('handedness','right')}"/>
 			</xacro:if>
-			<xacro:property name="layout" value="${mapping.get('layout','L3')}"/>
+			<xacro:property name="layout" value="${mapping['layout']}"/>
 			<xacro:property name="taxeldata_file" value="${mapping.get('taxeldata_file','../model/'+layout+side+'.yaml')}"/>
+			<!-- load taxeldata dictionary (positions + orientations) of taxel normals from file if available, else None -->
+			<xacro:property name="taxel_data" value="${None}"/>
 			<xacro:if value="${taxeldata_file not in ['', '-']}">
 				<xacro:property name="taxel_data" value="${load_yaml(taxeldata_file)}"/>
@@ -167,12 +170,7 @@
 		</xacro:finger>
 		<!-- TACTILE MARKERS -->
-		<xacro:if value="${tactile_mapping not in ['', '-']}">
-			<xacro:include filename="$(find human_hand_description)/model/${mapping['layout']}.urdf.xacro"/>
-			<xacro:if value="${taxel_data is not None}">
-				<xacro:tactile_glove prefix="${prefix}" reflect="${reflect}" tactMap="${mapping}" tactData="${taxel_data}"/>
-			</xacro:if>
-			<xacro:unless value="${taxel_data is not None}">
-				<xacro:tactile_glove prefix="${prefix}" reflect="${reflect}" tactMap="${mapping}"/>
-			</xacro:unless>
+		<xacro:if value="${mapping is not None}">
+			<xacro:include filename="$(find human_hand_description)/model/tactile_markers.urdf.xacro"/>
+			<xacro:tactile_glove prefix="${prefix}" reflect="${reflect}" tactMap="${mapping}" tactData="${taxel_data}"/>
 		</xacro:if>
 	</xacro:macro>

File: model/tactile_markers.urdf.xacro (robot description, xacro)
@@ -1,19 +1,33 @@
 <?xml version="1.0"?>
 <robot name="tactile_glove_markers" xmlns:xacro="http://www.ros.org/wiki/xacro">
-	<xacro:macro name="taxel" params="prefix:=^ mesh idx">
+	<xacro:macro name="taxel" params="prefix:=^ layout:=^ tactData:=^ reflect:=^ mesh idx">
+		<!-- only consider this, if taxel idx exists -->
 		<xacro:if value="${idx >= 0}">
-			<taxel idx="${idx}">
-				<geometry>
-					<mesh filename="package://human_hand_description/model/meshes/taxels/L1/${mesh}.stl"
-					      scale="${0.00101*reflect} 0.00101 0.00101"/>
-				</geometry>
-			</taxel>
+			<xacro:if value="${tactData is not None}" >
+				<taxel idx="${idx}"
+				       xyz="${' '.join([str(v) for v in tactData['positions'][mesh]])}"
+				       rpy="${' '.join([str(v) for v in tactData['orientations'][mesh]])}">
+					<geometry>
+						<mesh filename="package://human_hand_description/model/meshes/taxels/${layout}/${mesh}.stl"
+						      scale="${0.00101*reflect} 0.00101 0.00101"/>
+					</geometry>
+				</taxel>
+			</xacro:if>
+			<xacro:unless value="${tactData is not None}" >
+				<taxel idx="${idx}">
+					<geometry>
+						<mesh filename="package://human_hand_description/model/meshes/taxels/${layout}/${mesh}.stl"
+									scale="${0.00101*reflect} 0.00101 0.00101"/>
+					</geometry>
+				</taxel>
+			</xacro:unless>
 		</xacro:if>
 	</xacro:macro>
-	<xacro:macro name="tactile_glove_finger" params="prefix:=^ finger tactMap:=^">
+	<xacro:macro name="tactile_glove_finger" params="prefix:=^ finger tactMap:=^ tactData:=^|'-'">
+		<xacro:property name="layout" value="${tactMap['layout']}"/>
 		<xacro:property name="F" value="${finger[0]}"/>
 		<sensor name="${prefix}${finger}_distal" update_rate="100" group="distal">
 			<parent link="${finger}_distal_link"/>
-			<tactile channel="tactile">
+			<tactile channel="tactile glove">
 				<xacro:taxel mesh="${F}dd" idx="${tactMap.get(F+'dd', -1)}"/>
 				<xacro:taxel mesh="${F}do" idx="${tactMap.get(F+'do', -1)}"/>
@@ -24,5 +38,5 @@
 		<sensor name="${prefix}${finger}_middle" update_rate="100" group="middle">
 			<parent link="${finger}_middle_link"/>
-			<tactile channel="tactile">
+			<tactile channel="tactile glove">
 				<xacro:taxel mesh="${F}mo" idx="${tactMap.get(F+'mo', -1)}"/>
 				<xacro:taxel mesh="${F}mm" idx="${tactMap.get(F+'mm', -1)}"/>
@@ -32,5 +46,5 @@
 		<sensor name="${prefix}${finger}_proximal" update_rate="100" group="proximal">
 			<parent link="${finger}_proximal_link"/>
-			<tactile channel="tactile">
+			<tactile channel="tactile glove">
 				<xacro:taxel mesh="${F}p" idx="${tactMap.get(F+'p', -1)}"/>
 				<xacro:taxel mesh="${F}pi" idx="${tactMap.get(F+'pi', -1)}"/>
@@ -39,5 +53,5 @@
 		</sensor>
 	</xacro:macro>
-	<xacro:macro name="tactile_glove" params="prefix reflect:=1 tactMap">
+	<xacro:macro name="tactile_glove" params="prefix reflect:=1 tactMap tactData">
 		<xacro:tactile_glove_finger finger="index"/>
 		<xacro:tactile_glove_finger finger="middle"/>
@@ -47,7 +61,9 @@
 		<sensor name="thumb_base" update_rate="100" group="proximal">
 			<parent link="${prefix}thumb_proximal_link"/>
-			<tactile channel="tactile">
+			<tactile channel="tactile glove">
 				<xacro:taxel mesh="ptmp2" idx="${tactMap.get('ptop', -1)}"/>
+				<xacro:taxel mesh="ptmp2" idx="${tactMap.get('ptmp', -1)}"/>
 				<xacro:taxel mesh="ptmd2" idx="${tactMap.get('ptod', -1)}"/>
+				<xacro:taxel mesh="ptmd2" idx="${tactMap.get('ptmd', -1)}"/>
 				<xacro:taxel mesh="ptip2" idx="${tactMap.get('ptip', -1)}"/>
 				<xacro:taxel mesh="ptid2" idx="${tactMap.get('ptid', -1)}"/>
@@ -56,6 +72,7 @@
 		<sensor name="palm" update_rate="100" group="palm">
 			<parent link="${prefix}palm_link"/>
-			<tactile channel="tactile">
+			<tactile channel="tactile glove">
 				<xacro:taxel mesh="pdlo" idx="${tactMap.get('po', -1)}"/>
+				<xacro:taxel mesh="pdlo" idx="${tactMap.get('pdlo', -1)}"/>
 				<xacro:taxel mesh="pdl" idx="${tactMap.get('pdl', -1)}"/>
 				<xacro:taxel mesh="pdr" idx="${tactMap.get('pdr', -1)}"/>
@@ -64,4 +81,5 @@
 				<xacro:taxel mesh="pdii" idx="${tactMap.get('pdii', -1)}"/>
 				<xacro:taxel mesh="pco" idx="${tactMap.get('po', -1)}"/>
+				<xacro:taxel mesh="pco" idx="${tactMap.get('pco', -1)}"/>
 				<xacro:taxel mesh="pcmp" idx="${tactMap.get('pcmp', -1)}"/>
 				<xacro:taxel mesh="pcmd" idx="${tactMap.get('pcmd', -1)}"/>
@@ -69,8 +87,11 @@
 				<xacro:taxel mesh="pcim" idx="${tactMap.get('pcim', -1)}"/>
 				<xacro:taxel mesh="pcid" idx="${tactMap.get('pcid', -1)}"/>
+				<xacro:taxel mesh="pi" idx="${tactMap.get('pi', -1)}"/>
 				<xacro:taxel mesh="ptop" idx="${tactMap.get('ptop', -1)}"/>
 				<xacro:taxel mesh="ptod" idx="${tactMap.get('ptod', -1)}"/>
 				<xacro:taxel mesh="ptmp" idx="${tactMap.get('ptop', -1)}"/>
+				<xacro:taxel mesh="ptmp" idx="${tactMap.get('ptmp', -1)}"/>
 				<xacro:taxel mesh="ptmd" idx="${tactMap.get('ptod', -1)}"/>
+				<xacro:taxel mesh="ptmd" idx="${tactMap.get('ptmd', -1)}"/>
 				<xacro:taxel mesh="ptip" idx="${tactMap.get('ptip', -1)}"/>
 				<xacro:taxel mesh="ptid" idx="${tactMap.get('ptid', -1)}"/>

Commit message: cleanup prefix use
xacro: distinguish between link_prefix and joint_prefix
- link_prefix: needed to have multiple hands within the same TF tree
  Instead of modifying the robot_description,
  one can also use tf_prefix parameter for robot_state_publisher
- joint_prefix: needed to have multiple hands within the same robot description

File: model/human_hand.urdf.xacro (robot description, xacro)
@@ -11,11 +11,12 @@
 	<!-- a segment is composed of a joint and the attached link -->
 	<xacro:macro name="xacro:segment"
-	             params="prefix:=^|'' finger:=^ joint link parent reflect:=^ *origin *axis
+	             params="link_prefix:=^|'' joint_prefix:=^|''
+	                     finger:=^ joint link parent reflect:=^ *origin *axis
 	                     synergy_weight:=None mesh:=1 use_synergy:=^">
 		<xacro:property name="props" value="${joint_props[finger][joint]}"/>
-		<joint name="${prefix}${finger}_${joint}_joint" type="revolute">
+		<joint name="${joint_prefix}${finger}_${joint}_joint" type="revolute">
 			<xacro:insert_block name="origin"/>
-			<parent link="${parent}"/>
-			<child link="${prefix}${finger}_${link}_link"/>
+			<parent link="${link_prefix}${parent}"/>
+			<child link="${link_prefix}${finger}_${link}_link"/>
 			<xacro:insert_block name="axis"/>
 			<limit lower="${props['bounds'][0]*pi/180}" upper="${props['bounds'][1]*pi/180}"
@@ -30,5 +31,5 @@
 			</xacro:if>
 		</joint>
-		<link name="${prefix}${finger}_${link}_link">
+		<link name="${link_prefix}${finger}_${link}_link">
 			<xacro:if value="${mesh != 0}">
 				<visual>
@@ -47,6 +48,6 @@
 	<!-- FINGER MODEL -->
 	<xacro:macro name="finger"
-	             params="parent prefix:=^ finger reflect:=^ *origin
-	                     joint_props:=${properties['joints']}">
+	             params="parent link_prefix:=^|'' joint_prefix:=^|''
+	                     finger reflect:=^ *origin joint_props:=${properties['joints']}">
 		<xacro:property name="proximal_len" value="${properties['link_lengths'][finger]['proximal']}"/>
 		<xacro:property name="middle_len" value="${properties['link_lengths'][finger]['middle']}"/>
@@ -57,15 +58,15 @@
 		</xacro:segment>
 		<!-- PROXIMAL PHALANGE -->
-		<xacro:segment joint="proximal" link="proximal" parent="${prefix}${finger}_knuckle_link">
+		<xacro:segment joint="proximal" link="proximal" parent="${finger}_knuckle_link">
 			<origin xyz="0 0 0" rpy="0 0 0"/>
 			<axis xyz="1 0 0" />
 		</xacro:segment>
 		<!-- MIDDLE PHALANGE -->
-		<xacro:segment joint="middle" link="middle" parent="${prefix}${finger}_proximal_link">
+		<xacro:segment joint="middle" link="middle" parent="${finger}_proximal_link">
 			<origin xyz="0 0 ${proximal_len}" rpy="0 0 0"/>
 			<axis xyz="1 0 0" />
 		</xacro:segment>
 		<!-- DISTAL PHALANGE -->
-		<xacro:segment joint="distal" link="distal" parent="${prefix}${finger}_middle_link">
+		<xacro:segment joint="distal" link="distal" parent="${finger}_middle_link">
 			<origin xyz="0 0 ${middle_len}" rpy="0 0 0"/>
 			<axis xyz="1 0 0" />
@@ -74,6 +75,6 @@
 	<!-- THUMB MODEL -->
 	<xacro:macro name="thumb"
-	             params="parent prefix:=^ finger:='thumb' reflect:=^ *origin
-	                     joint_props:=${properties['joints']}">
+	             params="parent link_prefix:=^|'' joint_prefix:=^|''
+	                     finger:='thumb' reflect:=^ *origin joint_props:=${properties['joints']}">
 		<xacro:property name="proximal_len" value="${properties['link_lengths'][finger]['proximal']}"/>
 		<xacro:property name="middle_len" value="${properties['link_lengths'][finger]['middle']}"/>
@@ -85,15 +86,15 @@
 		</xacro:segment>
 		<!-- PROXIMAL PHALANGE -->
-		<xacro:segment joint="proximal" link="proximal" parent="${prefix}${finger}_knuckle_link">
+		<xacro:segment joint="proximal" link="proximal" parent="${finger}_knuckle_link">
 			<origin xyz="0 0 0" rpy="0 0 0" />
 			<axis xyz="0 ${-1*reflect} 0" />
 		</xacro:segment>
 		<!-- MIDDLE PHALANGE -->
-		<xacro:segment joint="middle" link="middle" parent="${prefix}${finger}_proximal_link">
+		<xacro:segment joint="middle" link="middle" parent="${finger}_proximal_link">
 			<origin xyz="0 0 ${proximal_len}" rpy="0 0 0"/>
 			<axis xyz="0 ${-1*reflect} 0" />
 		</xacro:segment>
 		<!-- DISTAL PHALANGE -->
-		<xacro:segment joint="distal" link="distal" parent="${prefix}${finger}_middle_link">
+		<xacro:segment joint="distal" link="distal" parent="${finger}_middle_link">
 			<origin xyz="0 0 ${middle_len}" rpy="0 0 0"/>
 			<axis xyz="0 ${-1*reflect} 0" />
@@ -102,5 +103,6 @@
 	<!-- HUMAN HAND MODEL -->
 	<xacro:macro name="human_hand"
-	             params="parent prefix:='' use_synergy side:='' tactile_mapping:='' *origin">
+	             params="parent link_prefix:=^|'' joint_prefix:=^|''
+	                     use_synergy side:='' tactile_mapping:='' *origin">
 		<!-- load kinematics properties -->
 		<xacro:property name="properties" value="${load_yaml('../model/properties.yaml')}"/>
@@ -125,10 +127,10 @@
 		<xacro:property name="reflect" value="${dict(right=1, left=-1)[side]}" />
 		<!-- PALM -->
-		<joint name="${prefix}palm_joint" type="fixed" >
+		<joint name="${joint_prefix}palm_joint" type="fixed" >
 			<xacro:insert_block name="origin"/>
 			<parent link="${parent}" />
-			<child link="${prefix}palm_link" />
+			<child link="${link_prefix}palm_link" />
 		</joint>
-		<link name="${prefix}palm_link">
+		<link name="${link_prefix}palm_link">
 			<visual>
 				<geometry>
@@ -140,9 +142,9 @@
 		</link>
 		<xacro:if value="${use_synergy}">
-			<xacro:property name="synergy_joint" value="${prefix}synergy_joint"/>
+			<xacro:property name="synergy_joint" value="${joint_prefix}synergy_joint"/>
 			<!-- SYNERGY JOINT -->
 			<joint name="${synergy_joint}" type="revolute">
-				<parent link="${prefix}palm_link" />
-				<child link="${prefix}dummy_synergy_link"/>
+				<parent link="${link_prefix}palm_link" />
+				<child link="${link_prefix}dummy_synergy_link"/>
 				<axis xyz="0 0 1" />
 				<xacro:property name="props" value="${properties['joints']['synergy']}"/>
@@ -151,20 +153,20 @@
 				<dynamics damping="${props['damping']}" friction="${props['friction']}"/>
 			</joint>
-			<link name="${prefix}dummy_synergy_link"/>
+			<link name="${link_prefix}dummy_synergy_link"/>
 		</xacro:if>
 		<!-- THUMB AND FINGERS -->
-		<xacro:thumb parent="${prefix}palm_link" finger="thumb">
+		<xacro:thumb parent="palm_link" finger="thumb">
 			<origin xyz="${0.02475*reflect} -0.0125 0.0125" rpy="0.0 ${0.6240*reflect} 0"/>
 		</xacro:thumb>
-		<xacro:finger parent="${prefix}palm_link" finger="index">
+		<xacro:finger parent="palm_link" finger="index">
 			<origin xyz="${0.02175*reflect} -0.002 0.099" rpy="0 0 0"/>
 		</xacro:finger>
-		<xacro:finger parent="${prefix}palm_link" finger="middle">
+		<xacro:finger parent="palm_link" finger="middle">
 			<origin xyz="${-0.002*reflect} 0.0015 0.0955" rpy="0 0 0"/>
 		</xacro:finger>
-		<xacro:finger parent="${prefix}palm_link" finger="ring">
+		<xacro:finger parent="palm_link" finger="ring">
 			<origin xyz="${-0.02225*reflect} 0.0010 0.090" rpy="0 0 0"/>
 		</xacro:finger>
-		<xacro:finger parent="${prefix}palm_link" finger="little">
+		<xacro:finger parent="palm_link" finger="little">
 			<origin xyz="${-0.04175*reflect} -0.003 0.079" rpy="0 0 0"/>
 		</xacro:finger>
@@ -172,5 +174,6 @@
 		<xacro:if value="${mapping is not None}">
 			<xacro:include filename="$(find human_hand_description)/model/tactile_markers.urdf.xacro"/>
-			<xacro:tactile_glove prefix="${prefix}" reflect="${reflect}" tactMap="${mapping}" tactData="${taxel_data}"/>
+			<xacro:tactile_glove prefix="${link_prefix}" reflect="${reflect}"
+			                     tactMap="${mapping}" tactData="${taxel_data}"/>
 		</xacro:if>
 	</xacro:macro>

File: model/tactile_markers.urdf.xacro (robot description, xacro)
@@ -24,5 +24,6 @@
 		</xacro:if>
 	</xacro:macro>
-	<xacro:macro name="tactile_glove_finger" params="prefix:=^ finger tactMap:=^ tactData:=^|'-'">
+	<xacro:macro name="tactile_glove_finger"
+	             params="prefix:=^ finger tactMap:=^ tactData:=^|'-'">
 		<xacro:property name="layout" value="${tactMap['layout']}"/>
 		<xacro:property name="F" value="${finger[0]}"/>

File: robots/human_hand.urdf.xacro (robot description, xacro)
@@ -2,5 +2,9 @@
 <robot xmlns:xacro="http://www.ros.org/wiki/xacro" name="human_hand">
 	<!-- side can be left | right | '' | '-' (meaning, fetch from mapping) -->
-	<xacro:arg name="prefix" default=""/>
+	<xacro:arg name="prefix" default=""/> <!-- prefix serves as default for link_prefix -->
+	<!-- link prefix is needed for multiple hands within the TF tree -->
+	<xacro:arg name="link_prefix" default="$(arg prefix)"/>
+	<!-- joint_prefix is only needed when combining multiple hands into a single robot -->
+	<xacro:arg name="joint_prefix" default=""/>
 	<xacro:arg name="side" default=""/>
 	<xacro:arg name="use_synergy" default="false"/>
@@ -9,5 +13,6 @@
 	<link name="$(arg prefix)glove_base"/>
 	<xacro:property name="side" value="$(arg side)"/>
-	<xacro:human_hand parent="$(arg prefix)glove_base" prefix="$(arg prefix)"
+	<xacro:human_hand parent="$(arg prefix)glove_base"
+	                  link_prefix="$(arg link_prefix)" joint_prefix="$(arg joint_prefix)"
 	                  side="$(arg side)" use_synergy="$(arg use_synergy)"
 	                  tactile_mapping="$(arg tactile_mapping)">

Commit message: Added a parameter to modify the default tactile channel if needed

File: model/human_hand.urdf.xacro (robot description, xacro)
@@ -104,5 +104,5 @@
 	<xacro:macro name="human_hand"
 	             params="parent link_prefix:=^|'' joint_prefix:=^|''
-	                     use_synergy side:='' tactile_mapping:='' *origin">
+	                     use_synergy side:='' tactile_mapping:='' tactile_channel:='tactile glove' *origin">
 		<!-- load kinematics properties -->
 		<xacro:property name="properties" value="${load_yaml('../model/properties.yaml')}"/>
@@ -175,5 +175,5 @@
 			<xacro:include filename="$(find human_hand_description)/model/tactile_markers.urdf.xacro"/>
 			<xacro:tactile_glove prefix="${link_prefix}" reflect="${reflect}"
-			                     tactMap="${mapping}" tactData="${taxel_data}"/>
+			                     tactMap="${mapping}" tactData="${taxel_data}" channel="${tactile_channel}"/>
 		</xacro:if>
 	</xacro:macro>

File: model/tactile_markers.urdf.xacro (robot description, xacro)
@@ -25,10 +25,10 @@
 	</xacro:macro>
 	<xacro:macro name="tactile_glove_finger"
-	             params="prefix:=^ finger tactMap:=^ tactData:=^|'-'">
+	             params="prefix:=^ finger tactMap:=^ tactData:=^|'-' channel:=^|'tactile glove'">
 		<xacro:property name="layout" value="${tactMap['layout']}"/>
 		<xacro:property name="F" value="${finger[0]}"/>
 		<sensor name="${prefix}${finger}_distal" update_rate="100" group="distal">
 			<parent link="${prefix}${finger}_distal_link"/>
-			<tactile channel="tactile glove">
+			<tactile channel="${channel}">
 				<xacro:taxel mesh="${F}dd" idx="${tactMap.get(F+'dd', -1)}"/>
 				<xacro:taxel mesh="${F}do" idx="${tactMap.get(F+'do', -1)}"/>
@@ -39,5 +39,5 @@
 		<sensor name="${prefix}${finger}_middle" update_rate="100" group="middle">
 			<parent link="${prefix}${finger}_middle_link"/>
-			<tactile channel="tactile glove">
+			<tactile channel="${channel}">
 				<xacro:taxel mesh="${F}mo" idx="${tactMap.get(F+'mo', -1)}"/>
 				<xacro:taxel mesh="${F}mm" idx="${tactMap.get(F+'mm', -1)}"/>
@@ -47,5 +47,5 @@
 		<sensor name="${prefix}${finger}_proximal" update_rate="100" group="proximal">
 			<parent link="${prefix}${finger}_proximal_link"/>
-			<tactile channel="tactile glove">
+			<tactile channel="${channel}">
 				<xacro:taxel mesh="${F}p" idx="${tactMap.get(F+'p', -1)}"/>
 				<xacro:taxel mesh="${F}pi" idx="${tactMap.get(F+'pi', -1)}"/>
@@ -54,5 +54,5 @@
 		</sensor>
 	</xacro:macro>
-	<xacro:macro name="tactile_glove" params="prefix reflect:=1 tactMap tactData">
+	<xacro:macro name="tactile_glove" params="prefix reflect:=1 tactMap tactData channel:='tactile glove'">
 		<xacro:tactile_glove_finger finger="index"/>
 		<xacro:tactile_glove_finger finger="middle"/>
@@ -62,5 +62,5 @@
 		<sensor name="${prefix}thumb_base" update_rate="100" group="proximal">
 			<parent link="${prefix}thumb_proximal_link"/>
-			<tactile channel="tactile glove">
+			<tactile channel="${channel}">
 				<xacro:taxel mesh="ptmp2" idx="${tactMap.get('ptop', -1)}"/>
 				<xacro:taxel mesh="ptmp2" idx="${tactMap.get('ptmp', -1)}"/>
@@ -73,5 +73,5 @@
 		<sensor name="${prefix}palm" update_rate="100" group="palm">
 			<parent link="${prefix}palm_link"/>
-			<tactile channel="tactile glove">
+			<tactile channel="${channel}">
 				<xacro:taxel mesh="pdlo" idx="${tactMap.get('po', -1)}"/>
 				<xacro:taxel mesh="pdlo" idx="${tactMap.get('pdlo', -1)}"/>

File: robots/human_hand.urdf.xacro (robot description, xacro)
@@ -10,4 +10,5 @@
 	<xacro:arg name="use_synergy" default="false"/>
 	<xacro:arg name="tactile_mapping" default=""/>
+	<xacro:arg name="tactile_channel" default="tactile glove"/>
 	<xacro:include filename="../model/human_hand.urdf.xacro"/>
 	<link name="$(arg prefix)glove_base"/>
@@ -16,5 +17,6 @@
 	                  link_prefix="$(arg link_prefix)" joint_prefix="$(arg joint_prefix)"
 	                  side="$(arg side)" use_synergy="$(arg use_synergy)"
-	                  tactile_mapping="$(arg tactile_mapping)">
+	                  tactile_mapping="$(arg tactile_mapping)"
+	                  tactile_channel="'$(arg tactile_channel)'">
 		<origin xyz="0 0 0" rpy="0 0 0"/>
 	</xacro:human_hand>
