Commit message: Added support for scaling the hand down

File: model/human_hand.urdf.xacro (robot description, xacro)
@@ -13,5 +13,6 @@
 	             params="link_prefix:=^|'' joint_prefix:=^|''
 	                     finger:=^ joint link parent reflect:=^ *origin *axis
-	                     synergy_weight:=None mesh:=1 use_synergy:=^">
+	                     synergy_weight:=None mesh:=1 use_synergy:=^
+	                     scale_factor:=^|1.0">
 		<xacro:property name="props" value="${joint_props[finger][joint]}"/>
 		<joint name="${joint_prefix}${finger}_${joint}_joint" type="revolute">
@@ -39,5 +40,5 @@
 						</xacro:if>
 						<mesh filename="package://human_hand_description/model/meshes/${mesh}.stl"
-						      scale="${0.001*reflect} 0.001 .001"/>
+						      scale="${scale_factor*0.001*reflect} ${scale_factor*0.001} ${scale_factor*0.001}"/>
 					</geometry>
 					<material name="HumanHand/Skin" />
@@ -64,10 +65,10 @@
 		<!-- MIDDLE PHALANGE -->
 		<xacro:segment joint="middle" link="middle" parent="${finger}_proximal_link">
-			<origin xyz="0 0 ${proximal_len}" rpy="0 0 0"/>
+			<origin xyz="0 0 ${proximal_len*scale_factor}" rpy="0 0 0"/>
 			<axis xyz="1 0 0" />
 		</xacro:segment>
 		<!-- DISTAL PHALANGE -->
 		<xacro:segment joint="distal" link="distal" parent="${finger}_middle_link">
-			<origin xyz="0 0 ${middle_len}" rpy="0 0 0"/>
+			<origin xyz="0 0 ${middle_len*scale_factor}" rpy="0 0 0"/>
 			<axis xyz="1 0 0" />
 		</xacro:segment>
@@ -92,10 +93,10 @@
 		<!-- MIDDLE PHALANGE -->
 		<xacro:segment joint="middle" link="middle" parent="${finger}_proximal_link">
-			<origin xyz="0 0 ${proximal_len}" rpy="0 0 0"/>
+			<origin xyz="0 0 ${proximal_len*scale_factor}" rpy="0 0 0"/>
 			<axis xyz="0 ${-1*reflect} 0" />
 		</xacro:segment>
 		<!-- DISTAL PHALANGE -->
 		<xacro:segment joint="distal" link="distal" parent="${finger}_middle_link">
-			<origin xyz="0 0 ${middle_len}" rpy="0 0 0"/>
+			<origin xyz="0 0 ${middle_len*scale_factor}" rpy="0 0 0"/>
 			<axis xyz="0 ${-1*reflect} 0" />
 		</xacro:segment>
@@ -103,9 +104,10 @@
 	<!-- HUMAN HAND MODEL -->
 	<xacro:macro name="human_hand"
-	             params="parent link_prefix:=^|'' joint_prefix:=^|''
+	             params="parent link_prefix:=^|'' joint_prefix:=^|'' scale:=1.0
 	                     use_synergy side:='' tactile_mapping:='' tactile_channel:='tactile glove' *origin">
 		<!-- load kinematics properties -->
 		<xacro:property name="properties" value="${load_yaml('../model/properties.yaml')}"/>
 		<xacro:property name="synergies" value="${properties['synergies']}"/>
+		<xacro:property name="scale_factor" value="${scale}"/>
 		<!-- load taxel mapping -->
 		<xacro:property name="mapping" value="${None}"/>
@@ -136,5 +138,5 @@
 				<geometry>
 					<mesh filename="package://human_hand_description/model/meshes/palm.stl"
-					      scale=" ${.001*reflect} .001 .001" />
+					      scale="${scale_factor*0.001*reflect} ${scale_factor*0.001} ${scale_factor*0.001}" />
 				</geometry>
 				<material name="HumanHand/Skin" />
@@ -157,22 +159,22 @@
 		<!-- THUMB AND FINGERS -->
 		<xacro:thumb parent="palm_link" finger="thumb">
-			<origin xyz="${0.02475*reflect} -0.0125 0.0125" rpy="0.0 ${0.6240*reflect} 0"/>
+			<origin xyz="${0.02475*reflect*scale_factor} ${-0.0125*scale_factor} ${0.0125*scale_factor}" rpy="0.0 ${0.6240*reflect} 0"/>
 		</xacro:thumb>
 		<xacro:finger parent="palm_link" finger="index">
-			<origin xyz="${0.02175*reflect} -0.002 0.099" rpy="0 0 0"/>
+			<origin xyz="${0.02175*reflect*scale_factor} ${-0.002*scale_factor} ${0.099*scale_factor}" rpy="0 0 0"/>
 		</xacro:finger>
 		<xacro:finger parent="palm_link" finger="middle">
-			<origin xyz="${-0.002*reflect} 0.0015 0.0955" rpy="0 0 0"/>
+			<origin xyz="${-0.002*reflect*scale_factor} ${0.0015*scale_factor} ${0.0955*scale_factor}" rpy="0 0 0"/>
 		</xacro:finger>
 		<xacro:finger parent="palm_link" finger="ring">
-			<origin xyz="${-0.02225*reflect} 0.0010 0.090" rpy="0 0 0"/>
+			<origin xyz="${-0.02225*reflect*scale_factor} ${0.0010*scale_factor} ${0.090*scale_factor}" rpy="0 0 0"/>
 		</xacro:finger>
 		<xacro:finger parent="palm_link" finger="little">
-			<origin xyz="${-0.04175*reflect} -0.003 0.079" rpy="0 0 0"/>
+			<origin xyz="${-0.04175*reflect*scale_factor} ${-0.003*scale_factor} ${0.079*scale_factor}" rpy="0 0 0"/>
 		</xacro:finger>
 		<!-- TACTILE MARKERS -->
 		<xacro:if value="${mapping is not None}">
 			<xacro:include filename="$(find human_hand_description)/model/tactile_markers.urdf.xacro"/>
-			<xacro:tactile_glove prefix="${link_prefix}" reflect="${reflect}"
+			<xacro:tactile_glove prefix="${link_prefix}" reflect="${reflect}" scale_factor="${scale}"
 			                     tactMap="${mapping}" tactData="${taxel_data}" channel="${tactile_channel}"/>
 		</xacro:if>

File: model/tactile_markers.urdf.xacro (robot description, xacro)
@@ -1,5 +1,5 @@
 <?xml version="1.0"?>
 <robot name="tactile_glove_markers" xmlns:xacro="http://www.ros.org/wiki/xacro">
-	<xacro:macro name="taxel" params="prefix:=^ layout:=^ tactData:=^ reflect:=^ mesh idx">
+	<xacro:macro name="taxel" params="prefix:=^ layout:=^ tactData:=^ reflect:=^ scale_factor:=^|1.0 mesh idx" >
 		<!-- only consider this, if taxel idx exists -->
 		<xacro:if value="${idx >= 0}">
@@ -10,5 +10,5 @@
 					<geometry>
 						<mesh filename="package://human_hand_description/model/meshes/taxels/${layout}/${mesh}.stl"
-						      scale="${0.00101*reflect} 0.00101 0.00101"/>
+						      scale="${0.00101*reflect*scale_factor} ${0.00101*scale_factor} ${0.00101*scale_factor}"/>
 					</geometry>
 				</taxel>
@@ -18,5 +18,5 @@
 					<geometry>
 						<mesh filename="package://human_hand_description/model/meshes/taxels/${layout}/${mesh}.stl"
-									scale="${0.00101*reflect} 0.00101 0.00101"/>
+									scale="${0.00101*reflect*scale_factor} ${0.00101*scale_factor} ${0.00101*scale_factor}"/>
 					</geometry>
 				</taxel>
@@ -54,5 +54,5 @@
 		</sensor>
 	</xacro:macro>
-	<xacro:macro name="tactile_glove" params="prefix reflect:=1 tactMap tactData channel:='tactile glove'">
+	<xacro:macro name="tactile_glove" params="prefix reflect:=1 scale_factor:=1.0 tactMap tactData channel:='tactile glove'">
 		<xacro:tactile_glove_finger finger="index"/>
 		<xacro:tactile_glove_finger finger="middle"/>

File: robots/human_hand.urdf.xacro (robot description, xacro)
@@ -7,4 +7,5 @@
 	<!-- joint_prefix is only needed when combining multiple hands into a single robot -->
 	<xacro:arg name="joint_prefix" default=""/>
+	<xacro:arg name="scale" default="1.0"/>
 	<xacro:arg name="side" default=""/>
 	<xacro:arg name="use_synergy" default="false"/>
@@ -16,4 +17,5 @@
 	<xacro:human_hand parent="$(arg prefix)glove_base"
 	                  link_prefix="$(arg link_prefix)" joint_prefix="$(arg joint_prefix)"
+	                  scale="$(arg scale)"
 	                  side="$(arg side)" use_synergy="$(arg use_synergy)"
 	                  tactile_mapping="$(arg tactile_mapping)"

Commit message: Use package find instead of relative path to allow re-use from external packages

File: model/human_hand.urdf.xacro (robot description, xacro)
@@ -107,5 +107,6 @@
 	                     use_synergy side:='' tactile_mapping:='' tactile_channel:='tactile glove' *origin">
 		<!-- load kinematics properties -->
-		<xacro:property name="properties" value="${load_yaml('../model/properties.yaml')}"/>
+		<xacro:property name="package" value="$(find human_hand_description)"/>
+		<xacro:property name="properties" value="${load_yaml(package + '/model/properties.yaml')}"/>
 		<xacro:property name="synergies" value="${properties['synergies']}"/>
 		<xacro:property name="scale_factor" value="${scale}"/>
@@ -113,5 +114,5 @@
 		<xacro:property name="mapping" value="${None}"/>
 		<xacro:if value="${tactile_mapping not in ['', '-']}">
-			<xacro:property name="mapping" value="${load_yaml('../model/taxel.yaml')[tactile_mapping]}"/>
+			<xacro:property name="mapping" value="${load_yaml(package + '/model/taxel.yaml')[tactile_mapping]}"/>
 			<!-- if side is not yet specified, try to fetch it from the tactile_mapping dictionary -->
 			<xacro:if value="${side not in ['left', 'right']}">
@@ -119,5 +120,5 @@
 			</xacro:if>
 			<xacro:property name="layout" value="${mapping['layout']}"/>
-			<xacro:property name="taxeldata_file" value="${mapping.get('taxeldata_file','../model/'+layout+side+'.yaml')}"/>
+			<xacro:property name="taxeldata_file" value="${mapping.get('taxeldata_file',package + '/model/'+layout+side+'.yaml')}"/>
 			<!-- load taxeldata dictionary (positions + orientations) of taxel normals from file if available, else None -->
 			<xacro:property name="taxel_data" value="${None}"/>

Commit message: Fix missing xacro namespace prefixes

File: model/human_hand.urdf.xacro (robot description, xacro)
@@ -10,5 +10,5 @@
 	<xacro:include filename="$(find human_hand_description)/model/materials.urdf.xacro"/>
 	<!-- a segment is composed of a joint and the attached link -->
-	<xacro:macro name="xacro:segment"
+	<xacro:macro name="segment"
 	             params="link_prefix:=^|'' joint_prefix:=^|''
 	                     finger:=^ joint link parent reflect:=^ *origin *axis

Commit message: load_yaml -> xacro.load_yaml

File: model/human_hand.urdf.xacro (robot description, xacro)
@@ -108,5 +108,5 @@
 		<!-- load kinematics properties -->
 		<xacro:property name="package" value="$(find human_hand_description)"/>
-		<xacro:property name="properties" value="${load_yaml(package + '/model/properties.yaml')}"/>
+		<xacro:property name="properties" value="${xacro.load_yaml(package + '/model/properties.yaml')}" />
 		<xacro:property name="synergies" value="${properties['synergies']}"/>
 		<xacro:property name="scale_factor" value="${scale}"/>
@@ -114,5 +114,5 @@
 		<xacro:property name="mapping" value="${None}"/>
 		<xacro:if value="${tactile_mapping not in ['', '-']}">
-			<xacro:property name="mapping" value="${load_yaml(package + '/model/taxel.yaml')[tactile_mapping]}"/>
+			<xacro:property name="mapping" value="${xacro.load_yaml(package + '/model/taxel.yaml')[tactile_mapping]}" />
 			<!-- if side is not yet specified, try to fetch it from the tactile_mapping dictionary -->
 			<xacro:if value="${side not in ['left', 'right']}">
@@ -129,5 +129,5 @@
 			<xacro:property name="taxel_data" value="${None}"/>
 			<xacro:if value="${taxeldata_file not in ['', '-']}">
-				<xacro:property name="taxel_data" value="${load_yaml(taxeldata_file)}"/>
+				<xacro:property name="taxel_data" value="${xacro.load_yaml(taxeldata_file)}" />
 			</xacro:if>
 		</xacro:if>

Commit message: Added support for passing mapping and property file path

File: model/human_hand.urdf.xacro (robot description, xacro)
@@ -105,14 +105,26 @@
 	<xacro:macro name="human_hand"
 	             params="parent link_prefix:=^|'' joint_prefix:=^|'' scale:=1.0
-	                     use_synergy side:='' tactile_mapping:='' tactile_channel:='tactile glove' *origin">
-		<!-- load kinematics properties -->
+	                     use_synergy side:='' property_file:=^|'' mapping_file:=^|'' tactile_mapping:=''
+	                     tactile_channel:='tactile glove' *origin">
 		<xacro:property name="package" value="$(find human_hand_description)"/>
-		<xacro:property name="properties" value="${xacro.load_yaml(package + '/model/properties.yaml')}" />
+		<!-- load kinematics properties from file if given or from default file -->
+		<xacro:if value="${property_file in ['', '-']}">
+			<xacro:property name="properties" value="${xacro.load_yaml(package + '/model/properties.yaml')}" />
+		</xacro:if>
+		<xacro:unless value="${property_file in ['', '-']}">
+			<xacro:property name="properties" value="${xacro.load_yaml(property_file)}" />
+		</xacro:unless>
+		<!-- load or read other properties -->
 		<xacro:property name="synergies" value="${properties['synergies']}"/>
 		<xacro:property name="scale_factor" value="${scale}"/>
-		<!-- load taxel mapping -->
+		<!-- if desired, load taxel mapping from file if given or from default file -->
 		<xacro:property name="mapping" value="${None}"/>
 		<xacro:if value="${tactile_mapping not in ['', '-']}">
-			<xacro:property name="mapping" value="${xacro.load_yaml(package + '/model/taxel.yaml')[tactile_mapping]}" />
+			<xacro:if value="${mapping_file in ['', '-']}">
+				<xacro:property name="mapping" value="${xacro.load_yaml(package + '/model/taxel.yaml')[tactile_mapping]}"/>
+			</xacro:if>
+			<xacro:unless value="${mapping_file in ['', '-']}">
+				<xacro:property name="mapping" value="${xacro.load_yaml(mapping_file)[tactile_mapping]}" />
+			</xacro:unless>
 			<!-- if side is not yet specified, try to fetch it from the tactile_mapping dictionary -->
 			<xacro:if value="${side not in ['left', 'right']}">

File: robots/human_hand.urdf.xacro (robot description, xacro)
@@ -12,4 +12,6 @@
 	<xacro:arg name="tactile_mapping" default=""/>
 	<xacro:arg name="tactile_channel" default="tactile glove"/>
+	<xacro:arg name="mapping_file" default=""/>
+	<xacro:arg name="property_file" default=""/>
 	<xacro:include filename="../model/human_hand.urdf.xacro"/>
 	<link name="$(arg prefix)glove_base"/>
@@ -20,5 +22,7 @@
 	                  side="$(arg side)" use_synergy="$(arg use_synergy)"
 	                  tactile_mapping="$(arg tactile_mapping)"
-	                  tactile_channel="'$(arg tactile_channel)'">
+	                  tactile_channel="'$(arg tactile_channel)'"
+	                  mapping_file="$(arg mapping_file)"
+	                  property_file="$(arg property_file)">
 		<origin xyz="0 0 0" rpy="0 0 0"/>
 	</xacro:human_hand>

Commit message: Added support for passing mapping and property file path

File: model/human_hand.urdf.xacro (robot description, xacro)
@@ -1,4 +1,6 @@
 <?xml version="1.0"?>
 <robot xmlns:xacro="http://www.ros.org/wiki/xacro">
+	<xacro:arg name="property_file" default="$(find human_hand_description)/model/properties.yaml"/>
+	<xacro:arg name="mapping_file" default="$(find human_hand_description)/model/taxel.yaml"/>
 	<!--
 	    HUMAN HAND MODEL v 0.1
@@ -108,5 +110,5 @@
 		<!-- load kinematics properties -->
 		<xacro:property name="package" value="$(find human_hand_description)"/>
-		<xacro:property name="properties" value="${xacro.load_yaml(package + '/model/properties.yaml')}" />
+		<xacro:property name="properties" value="${xacro.load_yaml(xacro.arg('property_file'))}" />
 		<xacro:property name="synergies" value="${properties['synergies']}"/>
 		<xacro:property name="scale_factor" value="${scale}"/>
@@ -114,5 +116,5 @@
 		<xacro:property name="mapping" value="${None}"/>
 		<xacro:if value="${tactile_mapping not in ['', '-']}">
-			<xacro:property name="mapping" value="${xacro.load_yaml(package + '/model/taxel.yaml')[tactile_mapping]}" />
+			<xacro:property name="mapping" value="${xacro.load_yaml(xacro.arg('mapping_file'))[tactile_mapping]}" />
 			<!-- if side is not yet specified, try to fetch it from the tactile_mapping dictionary -->
 			<xacro:if value="${side not in ['left', 'right']}">

File: robots/human_hand.urdf.xacro (robot description, xacro)
@@ -1,4 +1,6 @@
 <?xml version="1.0"?>
 <robot xmlns:xacro="http://www.ros.org/wiki/xacro" name="human_hand">
+	<xacro:arg name="property_file" default="$(find human_hand_description)/model/properties.yaml"/>
+	<xacro:arg name="mapping_file" default="$(find human_hand_description)/model/taxel.yaml"/>
 	<!-- side can be left | right | '' | '-' (meaning, fetch from mapping) -->
 	<xacro:arg name="prefix" default=""/> <!-- prefix serves as default for link_prefix -->
